File: culturit_tx.kicad_sch (KiCad schematic)
At the start: 0 parts

Commit message: 2022-08-08
Other:
- sheet Power ports: added VDRAIN; removed none
- sheet USB Connector ports: added USB_DN, USB_DP, VBAT_MON, VBAT_MON_EN, VDRAIN; removed none

Commit message: 2022-08-09
Other:
- sheet MDBT50Q ports: added AIN2_XDK, AIN3_XDK, CS, GPIO0, GPIO1, GPIO2/INT1, GPIO3/INT2, GPIO4, GPIO5, GPIO_EXT1_XDK, GPIO_EXT2_XDK, IOXP_INT, MCU_LED_B, MCU_LED_G, MCU_LED_R, MCU_RESET, PROM_RW, PS_EN1, PS_EN2, PlugDet, SCK/SCL, SCL0, SDA0, SDI/SDA, SDO, SPI0_CS, SPI0_MISO, SPI0_MOSI, SPI0_SCK, SWDCLK, SWDIO, SWDO, SWITCH1, SWITCH2, USBdata_N, USBdata_P, VBAT_MON, VBAT_MOT_EN, VDD_SEL; removed none
- sheet Power ports: added PS_EN1, PS_EN2, UVL_RST, VDD_SEL; removed none

Commit message: 2022-08-10
Parts:
- added TP1, TP10, TP11, TP12, TP14, TP15, TP2, TP3, TP4, TP5, TP9: TestPoint, TestPoint:TestPoint_Pad_D2.5mm, symbol Connector:TestPoint
- added TP13, TP6, TP7, TP8: TestPoint, TestPoint:TestPoint_Pad_D4.0mm, symbol Connector:TestPoint
Connections:
- new net BHI260AP/B260_TP1: TP1.1
- new net BHI260AP/B260_TP10: TP10.1
- new net BHI260AP/B260_TP11: TP11.1
- new net BHI260AP/B260_TP12: TP12.1
- new net BHI260AP/B260_TP13: TP13.1
- new net BHI260AP/B260_TP14: TP14.1
- new net BHI260AP/B260_TP15: TP15.1
- new net BHI260AP/B260_TP2: TP2.1
- new net BHI260AP/B260_TP3: TP3.1
- new net BHI260AP/B260_TP4: TP4.1
- new net BHI260AP/B260_TP5: TP5.1
- new net BHI260AP/B260_TP6: TP6.1
- new net BHI260AP/B260_TP7: TP7.1
- new net BHI260AP/B260_TP8: TP8.1
- new net BHI260AP/B260_TP9: TP9.1
Other:
- sheet BHI260AP ports: added B260_TP1, B260_TP10, B260_TP11, B260_TP12, B260_TP13, B260_TP14, B260_TP15, B260_TP2, B260_TP3, B260_TP4, B260_TP5, B260_TP6, B260_TP7, B260_TP8, B260_TP9, CS, GPIO0, GPIO1, GPIO2/INT, GPIO3/INT2, GPIO5, PROM_RW, SCK/SCL, SDI/SDA, SDO; removed none
- sheet MDBT50Q ports: added none; removed AIN2_XDK, AIN3_XDK, GPIO4, GPIO_EXT1_XDK, GPIO_EXT2_XDK, IOXP_INT, MCU_LED_B, MCU_LED_G, MCU_LED_R, MCU_RESET, PlugDet, SCL0, SDA0, SPI0_CS, SPI0_MISO, SPI0_MOSI, SPI0_SCK, SWDCLK, SWDIO, SWDO, SWITCH1, SWITCH2

Commit message: 2022-08-25
Other:
- sheet MDBT50Q ports: added none; removed VBAT_MON, VBAT_MOT_EN, VDD_SEL
- sheet USB Connector ports: added BATT_SCL, BATT_SDA, BIN, GPOUT; removed VBAT_MON, VBAT_MON_EN, VDRAIN

Commit message: 2022-08-26
Other:
- sheet BHI260AP ports: added QSPI_CLK, QSPI_CSN, QSPI_D0, QSPI_D1; removed none
- sheet MDBT50Q ports: added SCL0, SDA0, SPI0_CS, SPI0_MISO, SPI0_MOSI, SPI0_SCK, VBAT_MON, VBAT_MOT_EN; removed none
- sheet Power ports: added LDO_ON, ON_MONITOR; removed PS_EN1, PS_EN2, UVL_RST, VDD_SEL, VDRAIN

Commit message: 2022-08-29
Parts:
- removed TP1, TP10, TP11, TP12, TP14, TP15, TP2, TP3, TP4, TP5, TP9: TestPoint, TestPoint:TestPoint_Pad_D2.5mm, symbol Connector:TestPoint
- removed TP13, TP6, TP7, TP8: TestPoint, TestPoint:TestPoint_Pad_D4.0mm, symbol Connector:TestPoint
- added J1: SWD, symbol Connector_Generic:Conn_01x04
Connections:
- new net +3V3: J1.1 (Pin_1)
- new net Earth: J1.4 (Pin_4)
- new net MDBT50Q/SWDCLK: J1.3 (Pin_3)
- new net MDBT50Q/SWDIO: J1.2 (Pin_2)
Other:
- sheet BHI260AP ports: added APP_SPI_CS, APP_SPI_MISO, APP_SPI_MOSI, APP_SPI_SCK, BHI2x_JTAG_CLK, BHI2x_JTAG_DIO, GPIO2/INT1; removed B260_TP1, B260_TP10, B260_TP11, B260_TP12, B260_TP13, B260_TP14, B260_TP15, B260_TP2, B260_TP3, B260_TP4, B260_TP5, B260_TP6, B260_TP7, B260_TP8, B260_TP9, CS, GPIO0, GPIO1, GPIO2/INT, GPIO5, PROM_RW, QSPI_CLK, QSPI_CSN, QSPI_D0, QSPI_D1, SCK/SCL, SDI/SDA, SDO
- sheet MDBT50Q ports: added IMU_INT1, IMU_INT2, IMU_SPI_CS, IMU_SPI_MISO, IMU_SPI_MOSI, IMU_SPI_SCK, LDO_ON, ON_MONITOR, SWDCLK, SWDIO, SWDO; removed CS, GPIO0, GPIO1, GPIO2/INT1, GPIO3/INT2, GPIO5, PROM_RW, PS_EN1, PS_EN2, SCK/SCL, SCL0, SDA0, SDI/SDA, SDO, SPI0_CS, SPI0_MISO, SPI0_MOSI, SPI0_SCK, VBAT_MON, VBAT_MOT_EN
- company: (none) -> donnyunn@gmail.com
- title: (none) -> culturit_tx
