File: culturit_tx.kicad_sch (KiCad schematic)
At the start: 1 part, among them J1 SWD

Commit message: 2022-09-07
Other:
- sheet BHI260AP ports: added BNO_NRST, HIRQ, HOST_CS, HOST_MISO, HOST_MOSI, HOST_SCK, MCSB4; removed APP_SPI_CS, APP_SPI_MISO, APP_SPI_MOSI, APP_SPI_SCK, BHI2x_JTAG_CLK, BHI2x_JTAG_DIO, GPIO2/INT1, GPIO3/INT2, RESETN
- title: culturit_tx -> culturit_tx (BHI)
Changed lines of the file:
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@@
   (paper "A4")
   (title_block
-    (title "culturit_tx")
-    (date "2022-08-29")
+    (title "culturit_tx (BHI)")
+    (date "2022-09-06")
     (company "donnyunn@gmail.com")
   )
@@
       (effects (font (size 1.27 1.27)) (justify left top))
     )
-    (pin "APP_SPI_MOSI" input (at 203.2 63.5 180)
+    (pin "HOST_SCK" input (at 203.2 68.58 180)
       (effects (font (size 1.27 1.27)) (justify left))
     )
-    (pin "GPIO2{slash}INT1" input (at 203.2 55.88 180)
+    (pin "HOST_MISO" input (at 203.2 66.04 180)
       (effects (font (size 1.27 1.27)) (justify left))
     )
-    (pin "APP_SPI_MISO" input (at 203.2 66.04 180)
+    (pin "HOST_CS" input (at 203.2 60.96 180)
       (effects (font (size 1.27 1.27)) (justify left))
     )
-    (pin "APP_SPI_SCK" input (at 203.2 68.58 180)
+    (pin "BNO_NRST" input (at 203.2 71.12 180)
       (effects (font (size 1.27 1.27)) (justify left))
     )
-    (pin "GPIO3{slash}INT2" input (at 203.2 58.42 180)
+    (pin "HOST_MOSI" input (at 203.2 63.5 180)
       (effects (font (size 1.27 1.27)) (justify left))
     )
-    (pin "BHI2x_JTAG_CLK" input (at 241.3 55.88 0)
-      (effects (font (size 1.27 1.27)) (justify right))
-    )
-    (pin "BHI2x_JTAG_DIO" input (at 241.3 58.42 0)
-      (effects (font (size 1.27 1.27)) (justify right))
-    )
-    (pin "APP_SPI_CS" input (at 203.2 60.96 180)
+    (pin "HIRQ" input (at 203.2 55.88 180)
       (effects (font (size 1.27 1.27)) (justify left))
     )
-    (pin "RESETN" input (at 203.2 71.12 180)
+    (pin "MCSB4" input (at 203.2 58.42 180)
       (effects (font (size 1.27 1.27)) (justify left))
     )

Commit message: 2022-09-14
Parts:
- J1: footprint (none) -> Local_devices:SWD_port
Other:
- sheet BHI260AP ports: added none; removed BNO_NRST, HIRQ, HOST_CS, HOST_MISO, HOST_MOSI, HOST_SCK, MCSB4
Changed lines of the file:
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@@
     (property "Reference" "J1" (id 0) (at 184.15 120.65 0))
     (property "Value" "SWD" (id 1) (at 184.15 123.19 0))
-    (property "Footprint" "" (id 2) (at 184.15 129.54 0)
+    (property "Footprint" "Local_devices:SWD_port" (id 2) (at 184.15 129.54 0)
       (effects (font (size 1.27 1.27)) hide)
     )
@@
       (effects (font (size 1.27 1.27)) (justify left top))
     )
-    (pin "HOST_SCK" input (at 203.2 68.58 180)
-      (effects (font (size 1.27 1.27)) (justify left))
-    )
-    (pin "HOST_MISO" input (at 203.2 66.04 180)
-      (effects (font (size 1.27 1.27)) (justify left))
-    )
-    (pin "HOST_CS" input (at 203.2 60.96 180)
-      (effects (font (size 1.27 1.27)) (justify left))
-    )
-    (pin "BNO_NRST" input (at 203.2 71.12 180)
-      (effects (font (size 1.27 1.27)) (justify left))
-    )
-    (pin "HOST_MOSI" input (at 203.2 63.5 180)
-      (effects (font (size 1.27 1.27)) (justify left))
-    )
-    (pin "HIRQ" input (at 203.2 55.88 180)
-      (effects (font (size 1.27 1.27)) (justify left))
-    )
-    (pin "MCSB4" input (at 203.2 58.42 180)
-      (effects (font (size 1.27 1.27)) (justify left))
-    )
   )
   (sheet (at 114.3 38.1) (size 50.8 101.6) (fields_autoplaced)
@@
       (effects (font (size 1.27 1.27)) (justify left))
     )
-    (pin "BNO_WAKE" input (at 165.1 58.42 0)
+    (pin "BNO_WAKE" input (at 165.1 50.8 0)
       (effects (font (size 1.27 1.27)) (justify right))
     )
@@
       (effects (font (size 1.27 1.27)) (justify right))
     )
-    (pin "BNO_NRST" input (at 165.1 71.12 0)
+    (pin "BNO_NRST" input (at 165.1 53.34 0)
       (effects (font (size 1.27 1.27)) (justify right))
     )
@@
       (effects (font (size 1.27 1.27)) (justify right))
     )
-    (pin "BNO_BOOTN" input (at 165.1 73.66 0)
+    (pin "BNO_BOOTN" input (at 165.1 58.42 0)
       (effects (font (size 1.27 1.27)) (justify right))
     )
@@
     )
     (path "/ec86ed94-250f-4411-abc1-430cd40d9990/02a074d6-2998-4cf4-ad15-d28b418572f3"
-      (reference "#PWR?") (unit 1) (value "+1V8") (footprint "")
+      (reference "#PWR0101") (unit 1) (value "+1V8") (footprint "")
     )
     (path "/ec86ed94-250f-4411-abc1-430cd40d9990/9426da45-0082-44a3-97e1-64809d6c1b25"
-      (reference "#PWR?") (unit 1) (value "+1V8") (footprint "")
+      (reference "#PWR0102") (unit 1) (value "+1V8") (footprint "")
     )
     (path "/ec86ed94-250f-4411-abc1-430cd40d9990/6683a9dc-555d-4067-9470-1d5c0e641769"
@@
     )
     (path "/ec86ed94-250f-4411-abc1-430cd40d9990/3c7b59f8-157a-48d0-bcbd-1b5daab963d2"
-      (reference "FB1") (unit 1) (value "MMZ1005Y121CT000") (footprint "")
+      (reference "FB1") (unit 1) (value "MMZ1005Y121CT000") (footprint "Inductor_SMD:L_0402_1005Metric")
     )
     (path "/f3f07d98-b780-4b2e-a979-4057042f4915/3e9fae16-d7fb-42c3-aba6-9b15173e5aa1"
-      (reference "FB2") (unit 1) (value "MMZ1005Y121CT000") (footprint "")
+      (reference "FB2") (unit 1) (value "MMZ1005Y121CT000") (footprint "Inductor_SMD:L_0402_1005Metric")
     )
     (path "/5c1238b7-e2aa-494e-b35e-8b4315319494"
-      (reference "J1") (unit 1) (value "SWD") (footprint "")
+      (reference "J1") (unit 1) (value "SWD") (footprint "Local_devices:SWD_port")
     )
     (path "/ec86ed94-250f-4411-abc1-430cd40d9990/464199a5-5226-467c-98b4-1521b44fe720"

Commit message: 2022-10-13
Other:
- sheet BHI260AP ports: added GPIO_MCSB4, HOST_CS, HOST_INT, HOST_MISO, HOST_MOSI, HOST_NRST, HOST_SCK; removed none
- sheet MDBT50Q ports: added GPIO_MCSB4, HOST_NRST; removed BNO_BOOTN, BNO_NRST, BNO_WAKE
Changed lines of the file:
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@@
   (title_block
     (title "culturit_tx (BHI)")
-    (date "2022-09-06")
+    (date "2022-10-13")
+    (rev "v0.6")
     (company "donnyunn@gmail.com")
   )
@@
     (stroke (width 0) (type default) (color 0 0 0 0))
   )
+  (wire (pts (xy 165.1 53.34) (xy 203.2 53.34))
+    (stroke (width 0) (type default) (color 0 0 0 0))
+  )
   (wire (pts (xy 76.2 43.18) (xy 114.3 43.18))
     (stroke (width 0) (type default) (color 0 0 0 0))
@@
   )
   (wire (pts (xy 76.2 50.8) (xy 114.3 50.8))
-    (stroke (width 0) (type default) (color 0 0 0 0))
-  )
-  (wire (pts (xy 165.1 71.12) (xy 203.2 71.12))
     (stroke (width 0) (type default) (color 0 0 0 0))
   )
@@
       (effects (font (size 1.27 1.27)) (justify left top))
     )
+    (pin "HOST_CS" input (at 203.2 60.96 180)
+      (effects (font (size 1.27 1.27)) (justify left))
+    )
+    (pin "HOST_MISO" input (at 203.2 66.04 180)
+      (effects (font (size 1.27 1.27)) (justify left))
+    )
+    (pin "HOST_SCK" input (at 203.2 68.58 180)
+      (effects (font (size 1.27 1.27)) (justify left))
+    )
+    (pin "HOST_MOSI" input (at 203.2 63.5 180)
+      (effects (font (size 1.27 1.27)) (justify left))
+    )
+    (pin "HOST_INT" input (at 203.2 55.88 180)
+      (effects (font (size 1.27 1.27)) (justify left))
+    )
+    (pin "GPIO_MCSB4" input (at 203.2 58.42 180)
+      (effects (font (size 1.27 1.27)) (justify left))
+    )
+    (pin "HOST_NRST" input (at 203.2 53.34 180)
+      (effects (font (size 1.27 1.27)) (justify left))
+    )
   )
   (sheet (at 114.3 38.1) (size 50.8 101.6) (fields_autoplaced)
@@
       (effects (font (size 1.27 1.27)) (justify left))
     )
-    (pin "BNO_WAKE" input (at 165.1 50.8 0)
-      (effects (font (size 1.27 1.27)) (justify right))
-    )
     (pin "HOST_CSN" input (at 165.1 60.96 0)
       (effects (font (size 1.27 1.27)) (justify right))
@@
       (effects (font (size 1.27 1.27)) (justify right))
     )
-    (pin "BNO_NRST" input (at 165.1 53.34 0)
+    (pin "HOST_NRST" input (at 165.1 53.34 0)
       (effects (font (size 1.27 1.27)) (justify right))
     )
@@
       (effects (font (size 1.27 1.27)) (justify right))
     )
-    (pin "BNO_BOOTN" input (at 165.1 58.42 0)
+    (pin "GPIO_MCSB4" input (at 165.1 58.42 0)
       (effects (font (size 1.27 1.27)) (justify right))
     )
@@
       (reference "#PWR030") (unit 1) (value "Earth") (footprint "")
     )
+    (path "/cc5876ad-d1e1-4601-a6b1-2ecc2cb597c8/1910d10c-2f2b-41e6-a094-077a72888d75"
+      (reference "#PWR031") (unit 1) (value "Earth") (footprint "")
+    )
+    (path "/cc5876ad-d1e1-4601-a6b1-2ecc2cb597c8/995129a8-eb04-40ef-a6a5-8d49feef1722"
+      (reference "#PWR032") (unit 1) (value "Earth") (footprint "")
+    )
     (path "/cc5876ad-d1e1-4601-a6b1-2ecc2cb597c8/e1341a4d-89a3-451f-9240-dd68e2a3b4eb"
       (reference "#PWR033") (unit 1) (value "Earth") (footprint "")
@@
       (reference "#PWR041") (unit 1) (value "+3V3") (footprint "")
     )
-    (path "/cc5876ad-d1e1-4601-a6b1-2ecc2cb597c8/8245a6c4-2bea-4b4c-b988-2130d2ead7d0"
-      (reference "#PWR042") (unit 1) (value "Earth") (footprint "")
+    (path "/cc5876ad-d1e1-4601-a6b1-2ecc2cb597c8/c621f4c9-1d6e-4143-a9c7-68425d26ac6d"
+      (reference "#PWR042") (unit 1) (value "+1V8") (footprint "")
     )
     (path "/cc5876ad-d1e1-4601-a6b1-2ecc2cb597c8/a24cf183-b318-48c4-b9d7-269fa86ce7d7"
       (reference "#PWR043") (unit 1) (value "+3V3") (footprint "")
     )
-    (path "/cc5876ad-d1e1-4601-a6b1-2ecc2cb597c8/917f56fc-c5d9-4117-bbad-99832aee860e"
+    (path "/cc5876ad-d1e1-4601-a6b1-2ecc2cb597c8/c6389d47-fe9e-42be-a2cc-093c9133faf3"
       (reference "#PWR044") (unit 1) (value "Earth") (footprint "")
-    )
-    (path "/cc5876ad-d1e1-4601-a6b1-2ecc2cb597c8/b90dc511-0fe6-4d20-b9f2-88469902bb27"
-      (reference "#PWR045") (unit 1) (value "+1V8") (footprint "")
-    )
-    (path "/cc5876ad-d1e1-4601-a6b1-2ecc2cb597c8/76ace861-d81c-42c2-986e-c00645775667"
-      (reference "#PWR046") (unit 1) (value "Earth") (footprint "")
     )
     (path "/9e0f1fe0-2fcc-4e96-84c9-b35726e658d5/6a2d09e5-ec58-4b41-bdc9-36b85e62f156"
@@
       (reference "#PWR060") (unit 1) (value "+1V8") (footprint "")
     )
-    (path "/9e0f1fe0-2fcc-4e96-84c9-b35726e658d5/79b5c970-2cd5-4423-9515-9f446add76d7"
-      (reference "#PWR061") (unit 1) (value "Earth") (footprint "")
-    )
     (path "/9e0f1fe0-2fcc-4e96-84c9-b35726e658d5/234e9f06-346b-4583-9ea1-9f6976070a6d"
       (reference "#PWR062") (unit 1) (value "Earth") (footprint "")
@@
       (reference "#PWR065") (unit 1) (value "Earth") (footprint "")
     )
-    (path "/9e0f1fe0-2fcc-4e96-84c9-b35726e658d5/03b5cee1-f5b5-4354-95b7-8e7c66e802a1"
-      (reference "#PWR066") (unit 1) (value "Earth") (footprint "")
-    )
     (path "/9e0f1fe0-2fcc-4e96-84c9-b35726e658d5/49572224-7634-4fe2-8497-a622b87c27d2"
       (reference "#PWR067") (unit 1) (value "+1V8") (footprint "")
@@
       (reference "#PWR069") (unit 1) (value "Earth") (footprint "")
     )
-    (path "/9e0f1fe0-2fcc-4e96-84c9-b35726e658d5/1241a013-55ba-4076-ada4-33b69f5685ea"
-      (reference "#PWR070") (unit 1) (value "+1V8") (footprint "")
-    )
-    (path "/9e0f1fe0-2fcc-4e96-84c9-b35726e658d5/2fbe0c76-0e2d-4b2f-a15f-1a87fe25b80a"
-      (reference "#PWR071") (unit 1) (value "Earth") (footprint "")
-    )
     (path "/ec86ed94-250f-4411-abc1-430cd40d9990/02a074d6-2998-4cf4-ad15-d28b418572f3"
       (reference "#PWR0101") (unit 1) (value "+1V8") (footprint "")
@@
       (reference "C13") (unit 1) (value "22uF/2012") (footprint "Capacitor_SMD:C_0805_2012Metric")
     )
-    (path "/cc5876ad-d1e1-4601-a6b1-2ecc2cb597c8/03bd3033-bed0-469a-a7b3-322c062fc30b"
+    (path "/cc5876ad-d1e1-4601-a6b1-2ecc2cb597c8/4a82fbb4-4f86-44b0-a57a-8df7352281e3"
+      (reference "C14") (unit 1) (value "12pF") (footprint "Capacitor_SMD:C_0402_1005Metric")
+    )
+    (path "/cc5876ad-d1e1-4601-a6b1-2ecc2cb597c8/eeb6afd2-3b0a-4904-a170-3386013ab6c9"
+      (reference "C15") (unit 1) (value "12pF") (footprint "Capacitor_SMD:C_0402_1005Metric")
+    )
+    (path "/cc5876ad-d1e1-4601-a6b1-2ecc2cb597c8/e9743ca3-cd15-4f97-98b3-4b31791015d4"
       (reference "C16") (unit 1) (value "100nF") (footprint "Capacitor_SMD:C_0402_1005Metric")
     )
@@
       (reference "C22") (unit 1) (value "100nF") (footprint "Capacitor_SMD:C_0402_1005Metric")
     )
-    (path "/9e0f1fe0-2fcc-4e96-84c9-b35726e658d5/1fea0e4e-9984-463b-b7eb-1f362f486d63"
-      (reference "C23") (unit 1) (value "100nF") (footprint "Capacitor_SMD:C_0402_1005Metric")
-    )
     (path "/ec86ed94-250f-4411-abc1-430cd40d9990/d4f4bd35-b969-4251-9057-212d1361b823"
       (reference "CN1") (unit 1) (value "2.54 X 2P") (footprint "Connector_PinHeader_2.54mm:PinHeader_1x02_P2.54mm_Vertical")
@@
     )
     (path "/f3f07d98-b780-4b2e-a979-4057042f4915/7eab498a-be0f-4f22-8536-fe996ac90f55"
-      (reference "Q1") (unit 1) (value "MMBT2222LT1G") (footprint "Local_devices:SOT23")
+      (reference "Q1") (unit 1) (value "MMBT3904,215") (footprint "Local_devices:SOT23")
     )
     (path "/f3f07d98-b780-4b2e-a979-4057042f4915/75689cf3-e1b7-4aa1-8672-1630f048e618"
-      (reference "Q2") (unit 1) (value "FDN340P") (footprint "Local_devices:SOT23")
+      (reference "Q2") (unit 1) (value "AO3401A") (footprint "Local_devices:SOT23")
     )
     (path "/f3f07d98-b780-4b2e-a979-4057042f4915/0d6bd594-5b69-407a-bb90-3d11f16fdf66"
-      (reference "Q3") (unit 1) (value "MMBT2222LT1G") (footprint "Local_devices:SOT23")
+      (reference "Q3") (unit 1) (value "MMBT3904,215") (footprint "Local_devices:SOT23")
     )
     (path "/ec86ed94-250f-4411-abc1-430cd40d9990/7da91088-fbab-45de-9fdf-cc77b6a21e7c"
@@
       (reference "U5") (unit 1) (value "MDBT50Q-1M") (footprint "Local_devices:MDBT50Q-1M")
     )
-    (path "/cc5876ad-d1e1-4601-a6b1-2ecc2cb597c8/7adefd7f-8646-4a16-9ff5-193e4be36f90"
-      (reference "U6") (unit 1) (value "W25Q32JWZPIQ") (footprint "Local_devices:SON127P600X500X80-9N-D")
+    (path "/cc5876ad-d1e1-4601-a6b1-2ecc2cb597c8/69e48c34-a2bd-49ef-a70b-68ca40a1bb8c"
+      (reference "U6") (unit 1) (value "MX25R6435FM2IH0") (footprint "Package_SO:SOP-8_5.28x5.23mm_P1.27mm")
     )
     (path "/9e0f1fe0-2fcc-4e96-84c9-b35726e658d5/f631a7a3-ad7d-4556-8d3b-b269f1165b54"
       (reference "U7") (unit 1) (value "BHI260AP") (footprint "Local_devices:BHI260AP")
     )
-    (path "/9e0f1fe0-2fcc-4e96-84c9-b35726e658d5/65d4d345-3e0c-4f4b-b0ff-858c30fd3f03"
-      (reference "U8") (unit 1) (value "W25Q32JWZPIQ") (footprint "Local_devices:SON127P600X500X80-9N-D")
-    )
     (path "/9e0f1fe0-2fcc-4e96-84c9-b35726e658d5/9d2de40e-a037-4cf1-9781-261567f558b4"
       (reference "U9") (unit 1) (value "BMM150") (footprint "Package_CSP:WLCSP-12_1.56x1.56mm_P0.4mm")
     )
-  )
+    (path "/cc5876ad-d1e1-4601-a6b1-2ecc2cb597c8/75d99a53-b183-484d-ba22-112c672e0acc"
+      (reference "Y1") (unit 1) (value "32.768MHz") (footprint "Crystal:Crystal_SMD_2012-2Pin_2.0x1.2mm")
+    )
+  )
