File: culturit_tx.kicad_sch (KiCad schematic)
At the start: 1 part, among them J1 SWD

Commit message: bno085 branch
Other:
- removed sheet BHI260AP

Commit message: 2022-09-05
Other:
- added sheet BNO085 (bno085.kicad_sch)
- sheet MDBT50Q ports: added IMU_BOOTN, IMU_NRST, IMU_WAKE; removed none
- title: culturit_tx -> culturit_tx (BNO)
Changed lines of the file:
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@@
   (paper "A4")
   (title_block
-    (title "culturit_tx")
-    (date "2022-08-29")
+    (title "culturit_tx (BNO)")
+    (date "2022-09-05")
     (company "donnyunn@gmail.com")
   )
+  (wire (pts (xy 165.1 58.42) (xy 212.09 58.42))
+    (stroke (width 0) (type default) (color 0 0 0 0))
+  )
+  (wire (pts (xy 165.1 50.8) (xy 212.09 50.8))
+    (stroke (width 0) (type default) (color 0 0 0 0))
+  )
   (wire (pts (xy 165.1 129.54) (xy 179.07 129.54))
     (stroke (width 0) (type default) (color 0 0 0 0))
@@
     (stroke (width 0) (type default) (color 0 0 0 0))
   )
+  (wire (pts (xy 165.1 68.58) (xy 212.09 68.58))
+    (stroke (width 0) (type default) (color 0 0 0 0))
+  )
   (wire (pts (xy 76.2 80.01) (xy 114.3 80.01))
     (stroke (width 0) (type default) (color 0 0 0 0))
@@
     (stroke (width 0) (type default) (color 0 0 0 0))
   )
+  (wire (pts (xy 165.1 63.5) (xy 212.09 63.5))
+    (stroke (width 0) (type default) (color 0 0 0 0))
+  )
+  (wire (pts (xy 165.1 60.96) (xy 212.09 60.96))
+    (stroke (width 0) (type default) (color 0 0 0 0))
+  )
   (wire (pts (xy 76.2 43.18) (xy 114.3 43.18))
     (stroke (width 0) (type default) (color 0 0 0 0))
@@
     (stroke (width 0) (type default) (color 0 0 0 0))
   )
+  (wire (pts (xy 165.1 55.88) (xy 212.09 55.88))
+    (stroke (width 0) (type default) (color 0 0 0 0))
+  )
+  (wire (pts (xy 165.1 66.04) (xy 212.09 66.04))
+    (stroke (width 0) (type default) (color 0 0 0 0))
+  )
   (wire (pts (xy 176.53 124.46) (xy 176.53 127))
     (stroke (width 0) (type default) (color 0 0 0 0))
   )
   (wire (pts (xy 165.1 132.08) (xy 179.07 132.08))
+    (stroke (width 0) (type default) (color 0 0 0 0))
+  )
+  (wire (pts (xy 165.1 53.34) (xy 212.09 53.34))
     (stroke (width 0) (type default) (color 0 0 0 0))
   )
@@
     (pin "1")
   )
+  (sheet (at 212.09 38.1) (size 48.26 68.58) (fields_autoplaced)
+    (stroke (width 0.1524) (type solid) (color 0 0 0 0))
+    (fill (color 0 0 0 0.0000))
+    (property "Sheet name" "BNO085" (id 0) (at 212.09 37.3884 0)
+      (effects (font (size 1.27 1.27)) (justify left bottom))
+    )
+    (property "Sheet file" "bno085.kicad_sch" (id 1) (at 212.09 107.2646 0)
+      (effects (font (size 1.27 1.27)) (justify left top))
+    )
+    (pin "HOST_INTN" input (at 212.09 55.88 180)
+      (effects (font (size 1.27 1.27)) (justify left))
+    )
+    (pin "BNO_BOOTN" input (at 212.09 58.42 180)
+      (effects (font (size 1.27 1.27)) (justify left))
+    )
+    (pin "BNO_NRST" input (at 212.09 53.34 180)
+      (effects (font (size 1.27 1.27)) (justify left))
+    )
+    (pin "HOST_MISO" input (at 212.09 66.04 180)
+      (effects (font (size 1.27 1.27)) (justify left))
+    )
+    (pin "HOST_SCLK" input (at 212.09 68.58 180)
+      (effects (font (size 1.27 1.27)) (justify left))
+    )
+    (pin "HOST_CSN" input (at 212.09 60.96 180)
+      (effects (font (size 1.27 1.27)) (justify left))
+    )
+    (pin "HOST_MOSI" input (at 212.09 63.5 180)
+      (effects (font (size 1.27 1.27)) (justify left))
+    )
+    (pin "BNO_WAKE" input (at 212.09 50.8 180)
+      (effects (font (size 1.27 1.27)) (justify left))
+    )
+  )
   (sheet (at 114.3 38.1) (size 50.8 101.6) (fields_autoplaced)
     (stroke (width 0.1524) (type solid) (color 0 0 0 0))
@@
       (effects (font (size 1.27 1.27)) (justify right))
     )
-    (pin "IMU_INT2" input (at 165.1 58.42 0)
+    (pin "IMU_INT2" input (at 165.1 45.72 0)
+      (effects (font (size 1.27 1.27)) (justify right))
+    )
+    (pin "IMU_NRST" input (at 165.1 53.34 0)
+      (effects (font (size 1.27 1.27)) (justify right))
+    )
+    (pin "IMU_BOOTN" input (at 165.1 58.42 0)
+      (effects (font (size 1.27 1.27)) (justify right))
+    )
+    (pin "IMU_WAKE" input (at 165.1 50.8 0)
       (effects (font (size 1.27 1.27)) (justify right))
     )
@@
     (path "/f3f07d98-b780-4b2e-a979-4057042f4915" (page "3"))
     (path "/cc5876ad-d1e1-4601-a6b1-2ecc2cb597c8" (page "4"))
+    (path "/3239e741-4b5a-4ced-814a-c8e2e717eeba" (page "5"))
   )
   (symbol_instances
@@
       (reference "#PWR048") (unit 1) (value "Earth") (footprint "")
     )
+    (path "/3239e741-4b5a-4ced-814a-c8e2e717eeba/0047b95d-43f5-41af-859d-bfaaded1df49"
+      (reference "#PWR049") (unit 1) (value "+3V3") (footprint "")
+    )
+    (path "/3239e741-4b5a-4ced-814a-c8e2e717eeba/4401399e-2514-4494-8982-665deedb2a7f"
+      (reference "#PWR050") (unit 1) (value "Earth") (footprint "")
+    )
+    (path "/3239e741-4b5a-4ced-814a-c8e2e717eeba/4fd82b7c-c427-47aa-b046-8afe8180c2ea"
+      (reference "#PWR051") (unit 1) (value "Earth") (footprint "")
+    )
+    (path "/3239e741-4b5a-4ced-814a-c8e2e717eeba/a1818ce4-3b7a-4f8b-a229-4f0fdd8fa1ea"
+      (reference "#PWR052") (unit 1) (value "Earth") (footprint "")
+    )
+    (path "/3239e741-4b5a-4ced-814a-c8e2e717eeba/6fa24cf6-3558-4e7b-b5e9-c0b221042a58"
+      (reference "#PWR053") (unit 1) (value "+3V3") (footprint "")
+    )
+    (path "/3239e741-4b5a-4ced-814a-c8e2e717eeba/a2f553d7-6fab-4e5f-9980-3d30da6e00f2"
+      (reference "#PWR054") (unit 1) (value "Earth") (footprint "")
+    )
+    (path "/3239e741-4b5a-4ced-814a-c8e2e717eeba/185a50fc-15d6-4702-a918-8d30259e52fd"
+      (reference "#PWR055") (unit 1) (value "Earth") (footprint "")
+    )
+    (path "/3239e741-4b5a-4ced-814a-c8e2e717eeba/362ee88c-cb87-46f7-8f17-7db72b89177c"
+      (reference "#PWR056") (unit 1) (value "Earth") (footprint "")
+    )
+    (path "/3239e741-4b5a-4ced-814a-c8e2e717eeba/6ba6642e-92e6-4e79-900c-4e0372d61996"
+      (reference "#PWR057") (unit 1) (value "+3V3") (footprint "")
+    )
     (path "/ec86ed94-250f-4411-abc1-430cd40d9990/6683a9dc-555d-4067-9470-1d5c0e641769"
       (reference "C1") (unit 1) (value "1nF(1812),X7R,2kV") (footprint "Capacitor_SMD:C_1812_4532Metric")
@@
       (reference "C16") (unit 1) (value "100nF") (footprint "Capacitor_SMD:C_0402_1005Metric")
     )
+    (path "/3239e741-4b5a-4ced-814a-c8e2e717eeba/9fd2982d-800f-43ee-9447-01a541277e6e"
+      (reference "C17") (unit 1) (value "10nF") (footprint "Capacitor_SMD:C_0402_1005Metric")
+    )
+    (path "/3239e741-4b5a-4ced-814a-c8e2e717eeba/b5a98b14-ac33-4b29-bdea-cb2914481017"
+      (reference "C18") (unit 1) (value "100nF") (footprint "Capacitor_SMD:C_0402_1005Metric")
+    )
+    (path "/3239e741-4b5a-4ced-814a-c8e2e717eeba/bd03ae52-5463-49e4-8965-5b05e1087339"
+      (reference "C19") (unit 1) (value "10nF") (footprint "Capacitor_SMD:C_0402_1005Metric")
+    )
+    (path "/3239e741-4b5a-4ced-814a-c8e2e717eeba/ca62fe8d-2298-4051-8051-8274c6ab13f6"
+      (reference "C20") (unit 1) (value "100nF") (footprint "Capacitor_SMD:C_0402_1005Metric")
+    )
     (path "/ec86ed94-250f-4411-abc1-430cd40d9990/d4f4bd35-b969-4251-9057-212d1361b823"
       (reference "CN1") (unit 1) (value "2.54 X 2P") (footprint "Connector_PinHeader_2.54mm:PinHeader_1x02_P2.54mm_Vertical")
@@
       (reference "L1") (unit 1) (value "1uH/2012") (footprint "Inductor_SMD:L_0805_2012Metric")
     )
+    (path "/3239e741-4b5a-4ced-814a-c8e2e717eeba/a8e2d67f-04d0-456c-8de7-2bc3cc77afb8"
+      (reference "L2") (unit 1) (value "BLM15AG121SN1D") (footprint "Inductor_SMD:L_0402_1005Metric")
+    )
     (path "/ec86ed94-250f-4411-abc1-430cd40d9990/f6a46e04-f017-4718-a608-8f8fe24e892b"
       (reference "LED1") (unit 1) (value "APHHS1005SURCK") (footprint "Local_devices:LEDC1005X50N")
@@
       (reference "R28") (unit 1) (value "33") (footprint "Resistor_SMD:R_0402_1005Metric")
     )
+    (path "/3239e741-4b5a-4ced-814a-c8e2e717eeba/fb4b4b89-7e17-476e-b47b-80412b47a44f"
+      (reference "R29") (unit 1) (value "10k") (footprint "Resistor_SMD:R_0402_1005Metric")
+    )
+    (path "/3239e741-4b5a-4ced-814a-c8e2e717eeba/70addd95-f8e4-4a5d-aa5f-b159d88e8151"
+      (reference "R30") (unit 1) (value "10k") (footprint "Resistor_SMD:R_0402_1005Metric")
+    )
+    (path "/3239e741-4b5a-4ced-814a-c8e2e717eeba/18065ee2-99d3-42aa-86cb-ec0ff1dd0730"
+      (reference "R31") (unit 1) (value "10k") (footprint "Resistor_SMD:R_0402_1005Metric")
+    )
     (path "/f3f07d98-b780-4b2e-a979-4057042f4915/9a1aa609-89db-4acb-9b44-be898f41298f"
       (reference "S1") (unit 1) (value "SKSCLDE010") (footprint "Local_devices:SKSCLDE010")
@@
       (reference "U7") (unit 1) (value "DS28E05R+T") (footprint "Local_devices:SOT95P237X112-3N")
     )
+    (path "/3239e741-4b5a-4ced-814a-c8e2e717eeba/16490ab6-a8cc-429e-b52a-a1aa84365b4f"
+      (reference "U8") (unit 1) (value "BNO055") (footprint "Package_LGA:LGA-28_5.2x3.8mm_P0.5mm")
+    )
     (path "/cc5876ad-d1e1-4601-a6b1-2ecc2cb597c8/1cd31147-141a-4208-877f-1fc358e9bf62"

Commit message: 2022-09-06 1
Other:
- sheet MDBT50Q ports: added BATT_SCL, BATT_SDA, BIN, BNO_BOOTN, BNO_NRST, BNO_WAKE, GPOUT, HOST_CSN, HOST_INTN, HOST_MISO, HOST_MOSI, HOST_SCLK; removed IMU_BOOTN, IMU_INT1, IMU_INT2, IMU_NRST, IMU_SPI_CS, IMU_SPI_MISO, IMU_SPI_MOSI, IMU_SPI_SCK, IMU_WAKE
Changed lines of the file:
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@@
   (title_block
     (title "culturit_tx (BNO)")
-    (date "2022-09-05")
+    (date "2022-09-06")
     (company "donnyunn@gmail.com")
   )
@@
     (stroke (width 0) (type default) (color 0 0 0 0))
   )
+  (wire (pts (xy 76.2 58.42) (xy 114.3 58.42))
+    (stroke (width 0) (type default) (color 0 0 0 0))
+  )
   (wire (pts (xy 165.1 50.8) (xy 212.09 50.8))
     (stroke (width 0) (type default) (color 0 0 0 0))
@@
     (stroke (width 0) (type default) (color 0 0 0 0))
   )
+  (wire (pts (xy 76.2 53.34) (xy 114.3 53.34))
+    (stroke (width 0) (type default) (color 0 0 0 0))
+  )
+  (wire (pts (xy 76.2 55.88) (xy 114.3 55.88))
+    (stroke (width 0) (type default) (color 0 0 0 0))
+  )
   (wire (pts (xy 165.1 55.88) (xy 212.09 55.88))
     (stroke (width 0) (type default) (color 0 0 0 0))
@@
   )
   (wire (pts (xy 165.1 132.08) (xy 179.07 132.08))
+    (stroke (width 0) (type default) (color 0 0 0 0))
+  )
+  (wire (pts (xy 76.2 50.8) (xy 114.3 50.8))
     (stroke (width 0) (type default) (color 0 0 0 0))
   )
@@
       (effects (font (size 1.27 1.27)) (justify right))
     )
-    (pin "IMU_SPI_MOSI" input (at 165.1 63.5 0)
-      (effects (font (size 1.27 1.27)) (justify right))
-    )
-    (pin "IMU_SPI_SCK" input (at 165.1 68.58 0)
-      (effects (font (size 1.27 1.27)) (justify right))
-    )
-    (pin "IMU_SPI_CS" input (at 165.1 60.96 0)
-      (effects (font (size 1.27 1.27)) (justify right))
-    )
-    (pin "IMU_INT1" input (at 165.1 55.88 0)
-      (effects (font (size 1.27 1.27)) (justify right))
-    )
     (pin "ON_MONITOR" input (at 114.3 80.01 180)
       (effects (font (size 1.27 1.27)) (justify left))
@@
       (effects (font (size 1.27 1.27)) (justify left))
     )
-    (pin "IMU_SPI_MISO" input (at 165.1 66.04 0)
-      (effects (font (size 1.27 1.27)) (justify right))
-    )
-    (pin "IMU_INT2" input (at 165.1 45.72 0)
-      (effects (font (size 1.27 1.27)) (justify right))
-    )
-    (pin "IMU_NRST" input (at 165.1 53.34 0)
-      (effects (font (size 1.27 1.27)) (justify right))
-    )
-    (pin "IMU_BOOTN" input (at 165.1 58.42 0)
-      (effects (font (size 1.27 1.27)) (justify right))
-    )
-    (pin "IMU_WAKE" input (at 165.1 50.8 0)
+    (pin "BNO_BOOTN" input (at 165.1 58.42 0)
+      (effects (font (size 1.27 1.27)) (justify right))
+    )
+    (pin "GPOUT" input (at 114.3 50.8 180)
+      (effects (font (size 1.27 1.27)) (justify left))
+    )
+    (pin "BATT_SDA" input (at 114.3 55.88 180)
+      (effects (font (size 1.27 1.27)) (justify left))
+    )
+    (pin "BIN" input (at 114.3 58.42 180)
+      (effects (font (size 1.27 1.27)) (justify left))
+    )
+    (pin "BATT_SCL" input (at 114.3 53.34 180)
+      (effects (font (size 1.27 1.27)) (justify left))
+    )
+    (pin "BNO_WAKE" input (at 165.1 50.8 0)
+      (effects (font (size 1.27 1.27)) (justify right))
+    )
+    (pin "HOST_INTN" input (at 165.1 55.88 0)
+      (effects (font (size 1.27 1.27)) (justify right))
+    )
+    (pin "BNO_NRST" input (at 165.1 53.34 0)
+      (effects (font (size 1.27 1.27)) (justify right))
+    )
+    (pin "HOST_CSN" input (at 165.1 60.96 0)
+      (effects (font (size 1.27 1.27)) (justify right))
+    )
+    (pin "HOST_MISO" input (at 165.1 66.04 0)
+      (effects (font (size 1.27 1.27)) (justify right))
+    )
+    (pin "HOST_SCLK" input (at 165.1 68.58 0)
+      (effects (font (size 1.27 1.27)) (justify right))
+    )
+    (pin "HOST_MOSI" input (at 165.1 63.5 0)
       (effects (font (size 1.27 1.27)) (justify right))
     )
@@
       (reference "#PWR032") (unit 1) (value "Earth") (footprint "")
     )
-    (path "/cc5876ad-d1e1-4601-a6b1-2ecc2cb597c8/f877faf9-0eab-420b-b800-0e93d2fbdd52"
-      (reference "#PWR033") (unit 1) (value "+1V8") (footprint "")
-    )
     (path "/cc5876ad-d1e1-4601-a6b1-2ecc2cb597c8/e1341a4d-89a3-451f-9240-dd68e2a3b4eb"
       (reference "#PWR034") (unit 1) (value "Earth") (footprint "")
@@
       (reference "#PWR045") (unit 1) (value "Earth") (footprint "")
     )
-    (path "/cc5876ad-d1e1-4601-a6b1-2ecc2cb597c8/3e09d247-64e6-43e2-9176-a61ebbf3c7ee"
-      (reference "#PWR046") (unit 1) (value "Earth") (footprint "")
-    )
     (path "/cc5876ad-d1e1-4601-a6b1-2ecc2cb597c8/b90dc511-0fe6-4d20-b9f2-88469902bb27"
       (reference "#PWR047") (unit 1) (value "+1V8") (footprint "")
@@
       (reference "R21") (unit 1) (value "100k") (footprint "Resistor_SMD:R_0402_1005Metric")
     )
-    (path "/cc5876ad-d1e1-4601-a6b1-2ecc2cb597c8/19763e9e-c103-4514-a6a0-857ac5a974d2"
-      (reference "R22") (unit 1) (value "4.7k") (footprint "Resistor_SMD:R_0402_1005Metric")
-    )
     (path "/cc5876ad-d1e1-4601-a6b1-2ecc2cb597c8/96ff75a6-a528-4cbc-96d5-3779595982fc"
       (reference "R23") (unit 1) (value "0") (footprint "Resistor_SMD:R_0402_1005Metric")
@@
       (reference "U6") (unit 1) (value "W25Q32JWZPIQ") (footprint "Local_devices:SON127P600X500X80-9N-D")
     )
-    (path "/cc5876ad-d1e1-4601-a6b1-2ecc2cb597c8/a947e12c-d9e7-40da-8240-d060c7c763b9"
-      (reference "U7") (unit 1) (value "DS28E05R+T") (footprint "Local_devices:SOT95P237X112-3N")
-    )
     (path "/3239e741-4b5a-4ced-814a-c8e2e717eeba/16490ab6-a8cc-429e-b52a-a1aa84365b4f"

Commit message: 2022-09-07
Parts:
- J1: footprint (none) -> Local_devices:SWD_port

Commit message: 2022-11-01
Parts:
- J1: footprint Local_devices:SWD_port -> Connector_PinHeader_2.54mm:PinHeader_1x04_P2.54mm_Vertical
Changed lines of the file:
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@@
     (property "Reference" "J1" (id 0) (at 184.15 120.65 0))
     (property "Value" "SWD" (id 1) (at 184.15 123.19 0))
-    (property "Footprint" "Local_devices:SWD_port" (id 2) (at 184.15 129.54 0)
+    (property "Footprint" "Connector_PinHeader_2.54mm:PinHeader_1x04_P2.54mm_Vertical" (id 2) (at 184.15 129.54 0)
       (effects (font (size 1.27 1.27)) hide)
     )
@@
       (reference "#PWR018") (unit 1) (value "Earth") (footprint "")
     )
-    (path "/f3f07d98-b780-4b2e-a979-4057042f4915/fcaa0254-0b64-48ae-9076-13e485360de7"
-      (reference "#PWR019") (unit 1) (value "Earth") (footprint "")
-    )
     (path "/f3f07d98-b780-4b2e-a979-4057042f4915/8d2cbeca-98c3-4c5a-80cd-32821493c0ef"
       (reference "#PWR020") (unit 1) (value "Earth") (footprint "")
@@
       (reference "#PWR0103") (unit 1) (value "+1V8") (footprint "")
     )
+    (path "/ec86ed94-250f-4411-abc1-430cd40d9990/046aed05-0ce6-4756-863a-5d9c77b2210a"
+      (reference "#PWR0104") (unit 1) (value "Earth") (footprint "")
+    )
+    (path "/ec86ed94-250f-4411-abc1-430cd40d9990/08121723-6b7f-472e-89db-8f92654a9b38"
+      (reference "#PWR0105") (unit 1) (value "Earth") (footprint "")
+    )
+    (path "/ec86ed94-250f-4411-abc1-430cd40d9990/52df4a80-7a40-4368-9492-e15f8272b675"
+      (reference "#PWR0106") (unit 1) (value "Earth") (footprint "")
+    )
     (path "/ec86ed94-250f-4411-abc1-430cd40d9990/6683a9dc-555d-4067-9470-1d5c0e641769"
       (reference "C1") (unit 1) (value "4.7nF/1608") (footprint "Capacitor_SMD:C_0603_1608Metric")
@@
     )
     (path "/cc5876ad-d1e1-4601-a6b1-2ecc2cb597c8/468d7804-3cf9-4408-8db6-bbaf9907b1d6"
-      (reference "C14") (unit 1) (value "10uF") (footprint "Capacitor_SMD:C_0603_1608Metric")
+      (reference "C14") (unit 1) (value "10uF/1608") (footprint "Capacitor_SMD:C_0603_1608Metric")
     )
     (path "/cc5876ad-d1e1-4601-a6b1-2ecc2cb597c8/13f4a429-0dce-40ec-bfd3-0e5f7b5d0fd3"
-      (reference "C15") (unit 1) (value "12pF") (footprint "Capacitor_SMD:C_0402_1005Metric")
+      (reference "C15") (unit 1) (value "12pF/1005") (footprint "Capacitor_SMD:C_0402_1005Metric")
     )
     (path "/cc5876ad-d1e1-4601-a6b1-2ecc2cb597c8/03bd3033-bed0-469a-a7b3-322c062fc30b"
@@
     )
     (path "/cc5876ad-d1e1-4601-a6b1-2ecc2cb597c8/ebf5b1d8-f6be-4ebd-8d37-017f06517d7d"
-      (reference "C17") (unit 1) (value "12pF") (footprint "Capacitor_SMD:C_0402_1005Metric")
+      (reference "C17") (unit 1) (value "12pF/1005") (footprint "Capacitor_SMD:C_0402_1005Metric")
     )
     (path "/3239e741-4b5a-4ced-814a-c8e2e717eeba/ca62fe8d-2298-4051-8051-8274c6ab13f6"
@@
     )
     (path "/5c1238b7-e2aa-494e-b35e-8b4315319494"
-      (reference "J1") (unit 1) (value "SWD") (footprint "Local_devices:SWD_port")
-    )
-    (path "/ec86ed94-250f-4411-abc1-430cd40d9990/464199a5-5226-467c-98b4-1521b44fe720"
-      (reference "J2") (unit 1) (value "USB4105-GF-A") (footprint "Local_devices:GCT_USB4105-GF-A")
+      (reference "J1") (unit 1) (value "SWD") (footprint "Connector_PinHeader_2.54mm:PinHeader_1x04_P2.54mm_Vertical")
+    )
+    (path "/ec86ed94-250f-4411-abc1-430cd40d9990/13e08d0d-104f-4744-8227-1f734080597b"
+      (reference "J2") (unit 1) (value "USB4110-GF-A") (footprint "Local_devices:USB4110GFA")
     )
     (path "/f3f07d98-b780-4b2e-a979-4057042f4915/07ee436e-ef79-4678-a8d1-13bfa8fddcaf"
@@
     )
     (path "/cc5876ad-d1e1-4601-a6b1-2ecc2cb597c8/5963b6c5-f3cb-49fd-ac85-679b8e253913"
-      (reference "R25") (unit 1) (value "100") (footprint "Resistor_SMD:R_0402_1005Metric")
+      (reference "R25") (unit 1) (value "470") (footprint "Resistor_SMD:R_0402_1005Metric")
     )
     (path "/cc5876ad-d1e1-4601-a6b1-2ecc2cb597c8/5b9b5412-616d-47e7-83ab-c4fe2afcb587"
-      (reference "R26") (unit 1) (value "100") (footprint "Resistor_SMD:R_0402_1005Metric")
+      (reference "R26") (unit 1) (value "470") (footprint "Resistor_SMD:R_0402_1005Metric")
     )
     (path "/cc5876ad-d1e1-4601-a6b1-2ecc2cb597c8/55305c6e-b793-48dc-8ef7-99ff50b78fff"
-      (reference "R27") (unit 1) (value "100") (footprint "Resistor_SMD:R_0402_1005Metric")
+      (reference "R27") (unit 1) (value "470") (footprint "Resistor_SMD:R_0402_1005Metric")
     )
     (path "/3239e741-4b5a-4ced-814a-c8e2e717eeba/fb4b4b89-7e17-476e-b47b-80412b47a44f"
@@
       (reference "S1") (unit 1) (value "SKSCLDE010") (footprint "Local_devices:SKSCLDE010")
     )
-    (path "/cc5876ad-d1e1-4601-a6b1-2ecc2cb597c8/262866ed-31a4-4089-a60f-b327a8954020"
-      (reference "S2") (unit 1) (value "SKSCLDE010") (footprint "Local_devices:SKSCLDE010")
+    (path "/cc5876ad-d1e1-4601-a6b1-2ecc2cb597c8/95a8d439-85c8-43d7-9cc0-0e8513c56a4f"
+      (reference "S2") (unit 1) (value "Reset") (footprint "Button_Switch_SMD:SW_SPST_B3U-1000P")
     )
     (path "/ec86ed94-250f-4411-abc1-430cd40d9990/bb76d75f-466d-4cf3-8d59-4a8a674c52d1"
