File: 02_Culturit_Tx_Power.kicad_sch (KiCad schematic)
At the start: 0 parts

Commit message: 2022-08-08
Parts:
- added C10, C7, C9: 2.2uF(2012), Capacitor_SMD:C_0805_2012Metric, symbol Device:C
- added C12: 4.7uF(2012), Capacitor_SMD:C_0805_2012Metric, symbol Device:C
- added C13: 120pF, Capacitor_SMD:C_0402_1005Metric, symbol Device:C
- added C14, C15: 10uF(2012), Capacitor_SMD:C_0805_2012Metric, symbol Device:C
- added C16, C17, C18, C20, C21, C22: 100nF, Capacitor_SMD:C_0402_1005Metric, symbol Device:C
- added C19, C23: 1uF(1608), Capacitor_SMD:C_0603_1608Metric, symbol Device:C
- added D4, D5: SMAJ7.0A, Diode_SMD:D_SMA, symbol Device:D_Schottky
- added L2: 470nH, Inductor_SMD:L_0805_2012Metric, symbol Device:L
- added R16: 0, Resistor_SMD:R_0402_1005Metric, symbol Device:R
- added R17: 1k, Resistor_SMD:R_0402_1005Metric, symbol Device:R
- added R18: 200k, Resistor_SMD:R_0402_1005Metric, symbol Device:R
- added R19: 100k, Resistor_SMD:R_0402_1005Metric, symbol Device:R
- added R20, R22: 100, Resistor_SMD:R_0402_1005Metric, symbol Device:R
- added R21, R23: 1.91k, Resistor_SMD:R_0402_1005Metric, symbol Device:R
- added U10, U12: TPS22916CNYFPT, Local_devices:BGA4C40P2X2_78X78X50, symbol TPS22916CNYFPT:TPS22916CNYFPT
- added U11, U9: SN74AUP2G08RSER, Local_devices:RSE0008A, symbol SN74AUP2G08RSER:SN74AUP2G08RSER
- added U5: TPS3839A09DBZR, Package_TO_SOT_SMD:SOT-23, symbol Power_Supervisor:TPS3839DBZ
- added U7: LP5907QMFX-2.8Q1, Local_devices:SOT95P280X145-5N, symbol LP5907QMFX-2.8Q1:LP5907QMFX-2.8Q1
- added U8: TPS6282618DMQR, Local_devices:TPS6282618DMQR, symbol TPS6282618DMQR:TPS6282618DMQR
Connections:
- new net: R18.2, R19.1, U8.3 (FB)
- new net: C22.1, D5.2 (A), R23.1, U12.B2 (ON)
- new net: D5.1 (K), R22.1, R23.2
- new net: C7.2, R16.1, R17.2, U5.3 (VDD)
- new net: D4.1 (K), R20.1, R21.2
- new net: R20.2, U11.1 (1Y)
- new net: R22.2, U11.5 (2Y)
- new net: U11.7 (1A), U9.1 (1Y)
- new net: C18.1, D4.2 (A), R21.1, U10.B2 (ON)
- new net: L2.1, U8.5 (SW)
- new net +1V8: C13.2, C14.2, C15.2, C17.2, C19.1, C20.2, L2.2, R18.1, U10.A2 (VIN), U11.8 (VCC), U9.8 (VCC)
- new net +2V8: C10.2, C23.1, U12.A2 (VIN), U7.5 (OUT)
- new net Earth: C10.1, C12.1, C13.1, C14.1, C15.1, C16.2, C17.1, C18.2, C19.2, C20.1, C21.2, C22.2, C23.2, C7.1, C9.1, R19.2, U10.B1 (GND), U11.2 (2B), U11.3 (2A), U11.4 (GND), U12.B1 (GND), U5.1 (GND), U7.2 (GND), U8.4 (GND), U9.2 (2B), U9.3 (2A), U9.4 (GND)
- new net PS_EN1: U11.6 (1B)
- new net UVL_RST: R16.2, U5.2 (~{RESET}), U7.3 (EN)
- new net VDD: C16.1, C21.1, U10.A1 (VOUT), U12.A1 (VOUT)
- new net VDD_SEL: U9.6 (1B), U9.7 (1A)
- new net VDRAIN: C12.2, C9.2, R17.1, U7.1 (IN), U8.1 (EN), U8.6 (VIN)

Commit message: 2022-08-09
Parts:
- added C11: 1uF(1608), Capacitor_SMD:C_0603_1608Metric, symbol Device:C
- added C8: 100nF, Capacitor_SMD:C_0402_1005Metric, symbol Device:C
- added U6: TPS22916CNYFPT, Local_devices:BGA4C40P2X2_78X78X50, symbol TPS22916CNYFPT:TPS22916CNYFPT
Connections:
- net +1V8: now also C11.1, U6.A1 (VOUT)
- net Earth: now also C11.2, C8.2, U6.B1 (GND)
- new net PS_EN2: U6.B2 (ON)
- new net VDDIO: C8.1, U6.A2 (VIN)

Commit message: 2022-08-11 2
Parts:
- C10, C7, C9: MPN (none) -> CC0805KKX7R8BB225
- C11, C19, C23: MPN (none) -> CC0603KRX7R8BB105
- C12: MPN (none) -> CC0805KKX5R8BB475
- C13: MPN (none) -> 0402CG121J500NT
- C14, C15: MPN (none) -> CC0805ZKY5V6BB106
- C16, C17, C18, C20, C21, C22, C8: MPN (none) -> CC0402KRX7R7BB104
- R16: MPN (none) -> 0402WGF0000TCE
- R17: MPN (none) -> 0402WGJ0102TCE
- R18: MPN (none) -> RTT022003FTH
- R19: MPN (none) -> RC0402FR-07100KL
- R20, R22: MPN (none) -> 0402WGF1000TCE
- R21, R23: MPN (none) -> 0402WGF1911TCE
- U10, U12, U6: MPN (none) -> TPS22916CNYFPT
- U11, U9: MPN (none) -> SN74AUP2G08RSER
- U5: MPN (none) -> TPS3839A09DBZR
- U7: MPN (none) -> LP5907QMFX-2.8Q1
- U8: MPN (none) -> TPS6282618DMQR
Changed lines of the file:
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@@
+      (effects (font (size 1.27 1.27)) hide)
+    )
+    (property "MPN" "RTT022003FTH" (id 4) (at 124.46 100.33 0)
       (effects (font (size 1.27 1.27)) hide)
     )
@@
       (effects (font (size 1.27 1.27)) hide)
     )
+    (property "MPN" "CC0805KKX7R8BB225" (id 4) (at 38.1 74.93 0)
+      (effects (font (size 1.27 1.27)) hide)
+    )
     (pin "1")
     (pin "2")
@@
     )
     (property "Datasheet" "~" (id 3) (at 78.74 158.75 0)
+      (effects (font (size 1.27 1.27)) hide)
+    )
+    (property "MPN" "CC0402KRX7R7BB104" (id 4) (at 78.74 158.75 0)
       (effects (font (size 1.27 1.27)) hide)
     )
@@
       (effects (font (size 1.27 1.27)) hide)
     )
+    (property "MPN" "0402WGF1911TCE" (id 4) (at 140.97 152.4 0)
+      (effects (font (size 1.27 1.27)) hide)
+    )
     (pin "1")
     (pin "2")
@@
       (effects (font (size 1.27 1.27)) hide)
     )
+    (property "MPN" "TPS3839A09DBZR" (id 4) (at 55.88 45.72 0)
+      (effects (font (size 1.27 1.27)) hide)
+    )
     (pin "1")
     (pin "2")
@@
     )
     (property "Datasheet" "~" (id 3) (at 48.26 46.99 0)
+      (effects (font (size 1.27 1.27)) hide)
+    )
+    (property "MPN" "CC0805KKX7R8BB225" (id 4) (at 48.26 46.99 0)
       (effects (font (size 1.27 1.27)) hide)
     )
@@
       (effects (font (size 1.27 1.27)) hide)
     )
+    (property "MPN" "0402WGJ0102TCE" (id 4) (at 41.91 38.1 0)
+      (effects (font (size 1.27 1.27)) hide)
+    )
     (pin "1")
     (pin "2")
@@
     )
     (property "Datasheet" "~" (id 3) (at 232.41 151.13 0)
+      (effects (font (size 1.27 1.27)) hide)
+    )
+    (property "MPN" "CC0603KRX7R8BB105" (id 4) (at 232.41 151.13 0)
       (effects (font (size 1.27 1.27)) hide)
     )
@@
     )
     (property "Datasheet" "~" (id 3) (at 93.98 74.93 0)
+      (effects (font (size 1.27 1.27)) hide)
+    )
+    (property "MPN" "CC0805KKX7R8BB225" (id 4) (at 93.98 74.93 0)
       (effects (font (size 1.27 1.27)) hide)
     )
@@
     (property "Manufacturer_Part_Number" "TPS22916CNYFPT" (id 9) (at 191.77 134.62 0)
       (effects (font (size 1.27 1.27)) (justify left) hide)
+    )
+    (property "MPN" "TPS22916CNYFPT" (id 10) (at 215.9 149.86 0)
+      (effects (font (size 1.27 1.27)) hide)
     )
     (pin "A1")
@@
       (effects (font (size 1.27 1.27)) hide)
     )
+    (property "MPN" "	CC0805ZKY5V6BB106" (id 4) (at 109.22 100.33 0)
+      (effects (font (size 1.27 1.27)) hide)
+    )
     (pin "1")
     (pin "2")
@@
       (effects (font (size 1.27 1.27)) hide)
     )
+    (property "MPN" "0402CG121J500NT" (id 4) (at 134.62 100.33 0)
+      (effects (font (size 1.27 1.27)) hide)
+    )
     (pin "1")
     (pin "2")
@@
     )
     (property "Datasheet" "~" (id 3) (at 220.98 67.31 0)
+      (effects (font (size 1.27 1.27)) hide)
+    )
+    (property "MPN" "CC0402KRX7R7BB104" (id 4) (at 220.98 67.31 0)
       (effects (font (size 1.27 1.27)) hide)
     )
@@
     (property "Manufacturer_Part_Number" "TPS22916CNYFPT" (id 9) (at 191.77 45.72 0)
       (effects (font (size 1.27 1.27)) (justify left) hide)
+    )
+    (property "MPN" "TPS22916CNYFPT" (id 10) (at 215.9 60.96 0)
+      (effects (font (size 1.27 1.27)) hide)
     )
     (pin "A1")
@@
       (effects (font (size 1.27 1.27)) hide)
     )
+    (property "MPN" "CC0402KRX7R7BB104" (id 4) (at 149.86 158.75 0)
+      (effects (font (size 1.27 1.27)) hide)
+    )
     (pin "1")
     (pin "2")
@@
       (effects (font (size 1.27 1.27)) hide)
     )
+    (property "MPN" "RC0402FR-07100KL" (id 4) (at 124.46 107.95 0)
+      (effects (font (size 1.27 1.27)) hide)
+    )
     (pin "1")
     (pin "2")
@@
       (effects (font (size 1.27 1.27)) (justify left) hide)
     )
+    (property "MPN" "LP5907QMFX-2.8Q1" (id 10) (at 60.96 68.58 0)
+      (effects (font (size 1.27 1.27)) hide)
+    )
     (pin "1")
     (pin "2")
@@
       (effects (font (size 1.27 1.27)) hide)
     )
+    (property "MPN" "CC0402KRX7R7BB104" (id 4) (at 220.98 153.67 0)
+      (effects (font (size 1.27 1.27)) hide)
+    )
     (pin "1")
     (pin "2")
@@
     )
     (property "Datasheet" "~" (id 3) (at 232.41 67.31 0)
+      (effects (font (size 1.27 1.27)) hide)
+    )
+    (property "MPN" "CC0603KRX7R8BB105" (id 4) (at 232.41 67.31 0)
       (effects (font (size 1.27 1.27)) hide)
     )
@@
       (effects (font (size 1.27 1.27)) hide)
     )
+    (property "MPN" "0402WGF1000TCE" (id 4) (at 128.27 127 0)
+      (effects (font (size 1.27 1.27)) hide)
+    )
     (pin "1")
     (pin "2")
@@
     (property "Manufacturer_Part_Number" "SN74AUP2G08RSER" (id 9) (at 82.55 139.7 0)
       (effects (font (size 1.27 1.27)) (justify left) hide)
+    )
+    (property "MPN" "SN74AUP2G08RSER" (id 10) (at 104.14 147.32 0)
+      (effects (font (size 1.27 1.27)) hide)
     )
     (pin "1")
@@
       (effects (font (size 1.27 1.27)) hide)
     )
+    (property "MPN" "CC0603KRX7R8BB105" (id 4) (at 232.41 125.73 0)
+      (effects (font (size 1.27 1.27)) hide)
+    )
     (pin "1")
     (pin "2")
@@
     )
     (property "Datasheet" "~" (id 3) (at 149.86 133.35 0)
+      (effects (font (size 1.27 1.27)) hide)
+    )
+    (property "MPN" "CC0402KRX7R7BB104" (id 4) (at 149.86 133.35 0)
       (effects (font (size 1.27 1.27)) hide)
     )
@@
       (effects (font (size 1.27 1.27)) hide)
     )
+    (property "MPN" "CC0805KKX5R8BB475" (id 4) (at 38.1 97.79 0)
+      (effects (font (size 1.27 1.27)) hide)
+    )
     (pin "1")
     (pin "2")
@@
     (property "Manufacturer_Part_Number" "TPS22916CNYFPT" (id 9) (at 191.77 109.22 0)
       (effects (font (size 1.27 1.27)) (justify left) hide)
+    )
+    (property "MPN" "TPS22916CNYFPT" (id 10) (at 215.9 124.46 0)
+      (effects (font (size 1.27 1.27)) hide)
     )
     (pin "A1")
@@
       (effects (font (size 1.27 1.27)) hide)
     )
+    (property "MPN" "0402WGF1911TCE" (id 4) (at 140.97 127 0)
+      (effects (font (size 1.27 1.27)) hide)
+    )
     (pin "1")
     (pin "2")
@@
     (property "Manufacturer_Part_Number" "TPS6282618DMQR" (id 9) (at 82.55 111.76 0)
       (effects (font (size 1.27 1.27)) (justify left) hide)
+    )
+    (property "MPN" "TPS6282618DMQR" (id 10) (at 60.96 96.52 0)
+      (effects (font (size 1.27 1.27)) hide)
     )
     (pin "1")
@@
       (effects (font (size 1.27 1.27)) hide)
     )
+    (property "MPN" "0402WGF0000TCE" (id 4) (at 59.69 33.02 0)
+      (effects (font (size 1.27 1.27)) hide)
+    )
     (pin "1")
     (pin "2")
@@
       (effects (font (size 1.27 1.27)) hide)
     )
+    (property "MPN" "CC0402KRX7R7BB104" (id 4) (at 220.98 128.27 0)
+      (effects (font (size 1.27 1.27)) hide)
+    )
     (pin "1")
     (pin "2")
@@
     )
     (property "Datasheet" "~" (id 3) (at 104.14 100.33 0)
+      (effects (font (size 1.27 1.27)) hide)
+    )
+    (property "MPN" "	CC0805ZKY5V6BB106" (id 4) (at 104.14 100.33 0)
       (effects (font (size 1.27 1.27)) hide)
     )
@@
       (effects (font (size 1.27 1.27)) hide)
     )
+    (property "MPN" "0402WGF1000TCE" (id 4) (at 128.27 152.4 0)
+      (effects (font (size 1.27 1.27)) hide)
+    )
     (pin "1")
     (pin "2")
@@
     )
     (property "Datasheet" "~" (id 3) (at 38.1 158.75 0)
+      (effects (font (size 1.27 1.27)) hide)
+    )
+    (property "MPN" "CC0402KRX7R7BB104" (id 4) (at 38.1 158.75 0)
       (effects (font (size 1.27 1.27)) hide)
     )
@@
       (effects (font (size 1.27 1.27)) (justify left) hide)
     )
-    (pin "1")
+    (property "MPN" "SN74AUP2G08RSER" (id 10) (at 63.5 147.32 0)
+      (effects (font (size 1.27 1.27)) hide)
+    )
+    (pin "1")

Commit message: 2022-08-16
Connections:
- net +1V8: now also U6.A2 (VIN); no longer U6.A1 (VOUT)
- net Earth: no longer C13.1
- net UVL_RST: now also U8.1 (EN)
- net VDDIO: now also U6.A1 (VOUT); no longer U6.A2 (VIN)
- net VDRAIN: no longer U8.1 (EN)
- net at R18.2, R19.1, U8.3 (FB): now also C13.1
Changed lines of the file:
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@@
 (kicad_sch (version 20211123) (generator eeschema)
   (paper "A4")
-  (junction (at 60.96 91.44) (diameter 0) (color 0 0 0 0)
+  (title_block
+    (date "2022-08-16")
   )
   (junction (at 134.62 127) (diameter 0) (color 0 0 0 0)
@@
   (junction (at 124.46 93.98) (diameter 0) (color 0 0 0 0)
   )
-  (junction (at 232.41 60.96) (diameter 0) (color 0 0 0 0)
-  )
   (junction (at 33.02 38.1) (diameter 0) (color 0 0 0 0)
   )
@@
   (junction (at 232.41 147.32) (diameter 0) (color 0 0 0 0)
   )
-  (junction (at 220.98 58.42) (diameter 0) (color 0 0 0 0)
-  )
   (junction (at 220.98 149.86) (diameter 0) (color 0 0 0 0)
   )
@@
   (junction (at 104.14 93.98) (diameter 0) (color 0 0 0 0)
   )
+  (junction (at 232.41 58.42) (diameter 0) (color 0 0 0 0)
+  )
   (junction (at 38.1 91.44) (diameter 0) (color 0 0 0 0)
   )
@@
   (junction (at 232.41 121.92) (diameter 0) (color 0 0 0 0)
   )
+  (junction (at 220.98 60.96) (diameter 0) (color 0 0 0 0)
+  )
   (junction (at 93.98 71.12) (diameter 0) (color 0 0 0 0)
   )
@@
     (stroke (width 0) (type default) (color 0 0 0 0))
   )
-  (wire (pts (xy 232.41 55.88) (xy 232.41 60.96))
-    (stroke (width 0) (type default) (color 0 0 0 0))
-  )
   (wire (pts (xy 114.3 152.4) (xy 114.3 172.72))
     (stroke (width 0) (type default) (color 0 0 0 0))
@@
     (stroke (width 0) (type default) (color 0 0 0 0))
   )
-  (wire (pts (xy 215.9 60.96) (xy 232.41 60.96))
-    (stroke (width 0) (type default) (color 0 0 0 0))
-  )
   (wire (pts (xy 144.78 147.32) (xy 149.86 147.32))
     (stroke (width 0) (type default) (color 0 0 0 0))
@@
     (stroke (width 0) (type default) (color 0 0 0 0))
   )
-  (wire (pts (xy 220.98 58.42) (xy 215.9 58.42))
+  (wire (pts (xy 124.46 104.14) (xy 134.62 104.14))
     (stroke (width 0) (type default) (color 0 0 0 0))
   )
@@
     (stroke (width 0) (type default) (color 0 0 0 0))
   )
-  (wire (pts (xy 220.98 55.88) (xy 220.98 58.42))
+  (wire (pts (xy 220.98 55.88) (xy 220.98 60.96))
     (stroke (width 0) (type default) (color 0 0 0 0))
   )
@@
     (stroke (width 0) (type default) (color 0 0 0 0))
   )
-  (wire (pts (xy 220.98 58.42) (xy 220.98 63.5))
-    (stroke (width 0) (type default) (color 0 0 0 0))
-  )
   (wire (pts (xy 137.16 147.32) (xy 134.62 147.32))
     (stroke (width 0) (type default) (color 0 0 0 0))
@@
     (stroke (width 0) (type default) (color 0 0 0 0))
   )
+  (wire (pts (xy 232.41 58.42) (xy 232.41 63.5))
+    (stroke (width 0) (type default) (color 0 0 0 0))
+  )
   (wire (pts (xy 86.36 99.06) (xy 91.44 99.06))
     (stroke (width 0) (type default) (color 0 0 0 0))
@@
     (stroke (width 0) (type default) (color 0 0 0 0))
   )
+  (wire (pts (xy 215.9 58.42) (xy 232.41 58.42))
+    (stroke (width 0) (type default) (color 0 0 0 0))
+  )
   (wire (pts (xy 104.14 93.98) (xy 104.14 96.52))
     (stroke (width 0) (type default) (color 0 0 0 0))
@@
     (stroke (width 0) (type default) (color 0 0 0 0))
   )
+  (wire (pts (xy 215.9 60.96) (xy 220.98 60.96))
+    (stroke (width 0) (type default) (color 0 0 0 0))
+  )
   (wire (pts (xy 104.14 127) (xy 104.14 142.24))
     (stroke (width 0) (type default) (color 0 0 0 0))
@@
     (stroke (width 0) (type default) (color 0 0 0 0))
   )
+  (wire (pts (xy 220.98 60.96) (xy 220.98 63.5))
+    (stroke (width 0) (type default) (color 0 0 0 0))
+  )
   (wire (pts (xy 165.1 152.4) (xy 165.1 147.32))
     (stroke (width 0) (type default) (color 0 0 0 0))
@@
     (stroke (width 0) (type default) (color 0 0 0 0))
   )
-  (wire (pts (xy 60.96 91.44) (xy 88.9 91.44))
-    (stroke (width 0) (type default) (color 0 0 0 0))
-  )
-  (wire (pts (xy 38.1 91.44) (xy 60.96 91.44))
+  (wire (pts (xy 38.1 91.44) (xy 88.9 91.44))
     (stroke (width 0) (type default) (color 0 0 0 0))
   )
@@
     (stroke (width 0) (type default) (color 0 0 0 0))
   )
-  (wire (pts (xy 60.96 91.44) (xy 60.96 96.52))
-    (stroke (width 0) (type default) (color 0 0 0 0))
-  )
   (wire (pts (xy 53.34 33.02) (xy 53.34 38.1))
     (stroke (width 0) (type default) (color 0 0 0 0))
@@
     (stroke (width 0) (type default) (color 0 0 0 0))
   )
-  (wire (pts (xy 232.41 60.96) (xy 232.41 63.5))
+  (wire (pts (xy 232.41 55.88) (xy 232.41 58.42))
     (stroke (width 0) (type default) (color 0 0 0 0))
   )
@@
   (hierarchical_label "UVL_RST" (shape input) (at 60.96 78.74 0)
     (effects (font (size 1.27 1.27)) (justify left))
+  )
+  (hierarchical_label "UVL_RST" (shape input) (at 60.96 96.52 180)
+    (effects (font (size 1.27 1.27)) (justify right))
   )
   (hierarchical_label "PS_EN1" (shape input) (at 78.74 144.78 180)
@@
       (effects (font (size 1.27 1.27)) hide)
     )
-    (pin "1")
-  )
-  (symbol (lib_id "power:Earth") (at 134.62 104.14 0) (unit 1)
-    (in_bom yes) (on_board yes) (fields_autoplaced)
-    (property "Reference" "#PWR0125" (id 0) (at 134.62 110.49 0)
-      (effects (font (size 1.27 1.27)) hide)
-    )
-    (property "Value" "Earth" (id 1) (at 134.62 107.95 0)
-      (effects (font (size 1.27 1.27)) hide)
-    )
-    (property "Footprint" "" (id 2) (at 134.62 104.14 0)
-      (effects (font (size 1.27 1.27)) hide)
-    )
-    (property "Datasheet" "~" (id 3) (at 134.62 104.14 0)
-      (effects (font (size 1.27 1.27)) hide)
-    )

Commit message: 2022-08-26
Parts:
- removed C12: 4.7uF(2012), Capacitor_SMD:C_0805_2012Metric, symbol Device:C
- removed C13: 120pF, Capacitor_SMD:C_0402_1005Metric, symbol Device:C
- removed C14, C15: 10uF(2012), Capacitor_SMD:C_0805_2012Metric, symbol Device:C
- removed C16, C17, C18, C20, C21, C22, C8: 100nF, Capacitor_SMD:C_0402_1005Metric, symbol Device:C
- removed C19, C23: 1uF(1608), Capacitor_SMD:C_0603_1608Metric, symbol Device:C
- removed D4, D5: SMAJ7.0A, Diode_SMD:D_SMA, symbol Device:D_Schottky
- removed L2: 470nH, Inductor_SMD:L_0805_2012Metric, symbol Device:L
- removed R20, R22: 100, Resistor_SMD:R_0402_1005Metric, symbol Device:R
- removed R21, R23: 1.91k, Resistor_SMD:R_0402_1005Metric, symbol Device:R
- removed U10, U12, U6: TPS22916CNYFPT, Local_devices:BGA4C40P2X2_78X78X50, symbol TPS22916CNYFPT:TPS22916CNYFPT
- removed U11, U9: SN74AUP2G08RSER, Local_devices:RSE0008A, symbol SN74AUP2G08RSER:SN74AUP2G08RSER
- removed U5: TPS3839A09DBZR, Package_TO_SOT_SMD:SOT-23, symbol Power_Supervisor:TPS3839DBZ
- removed U7: LP5907QMFX-2.8Q1, Local_devices:SOT95P280X145-5N, symbol LP5907QMFX-2.8Q1:LP5907QMFX-2.8Q1
- removed U8: TPS6282618DMQR, Local_devices:TPS6282618DMQR, symbol TPS6282618DMQR:TPS6282618DMQR
- added C11: 1uF(1608), Capacitor_SMD:C_0603_1608Metric, symbol Device:C
- added C6: 10nF, Capacitor_SMD:C_0402_1005Metric, symbol Device:C
- added D1: MMBD4148, Local_devices:SOT23, symbol MMBD4148:MMBD4148
- added FB2: MMZ1005Y121CT000, symbol Device:FerriteBead
- added Q1, Q3: MMBT2222LT1G, Local_devices:SOT23, symbol Device:Q_NPN_BEC
- added Q2: FDN340P, Local_devices:SOT23, symbol Device:Q_NMOS_GSD
- added R10, R12: 10k, Resistor_SMD:R_0402_1005Metric, symbol Device:R
- added R11, R13: 20k, Resistor_SMD:R_0402_1005Metric, symbol Device:R
- added R15: 1k, Resistor_SMD:R_0402_1005Metric, symbol Device:R
- added S1: SKSCLDE010, Local_devices:SKSCLDE010, symbol SKSCLDE010:SKSCLDE010
- added U3: TCR3UG33A,LF, Local_devices:BGA4N35P2X2_64X64X33, symbol TCR3UG33A_LF:TCR3UG33A,LF
- C10, C7: value 2.2uF(2012) -> 10nF; footprint Capacitor_SMD:C_0805_2012Metric -> Capacitor_SMD:C_0402_1005Metric; MPN CC0805KKX7R8BB225 -> CC0402KRX7R9BB103
- C9: value 2.2uF(2012) -> 100nF; footprint Capacitor_SMD:C_0805_2012Metric -> Capacitor_SMD:C_0402_1005Metric; MPN CC0805KKX7R8BB225 -> CC0402KRX7R7BB104
- R16: value 0 -> 1k; MPN 0402WGF0000TCE -> RC0402FR-071KL
- R17: value 1k -> 100k; MPN 0402WGJ0102TCE -> RC0402FR-07100KL
- R18: value 200k -> 1k; MPN RTT022003FTH -> RC0402FR-071KL
- renumbered C11 to C8, R19 to R14
Connections:
- net +2V8 is gone; now on net Earth: C10.2
- net Earth: now also C7.2, C9.2, C11.2, C6.2, Q1.2 (E), Q3.2 (E), R11.2, R13.2, U3.B2 (GND); no longer C10.1, C7.1, C9.1, R14.2
- net at R18.2: now also R17.2, Q3.1 (B); no longer R14.1
- net +1V8 renamed LDO_ON
- net LDO_ON: no longer C8.1
- net UVL_RST: no longer names the net of R16.2
- net UVL_RST: now also R14.2, Q2.1 (G), R15.2
- net VDRAIN: no longer names the net of R17.1
- net VDRAIN: now also Q2.2 (S), U3.A1 (VIN), U3.B1 (CTRL); no longer C9.2
- new net: Q3.3 (C), R16.1
- new net: C6.1, D1.2, R10.1, S1.3, S1.4
- new net: Q1.1 (B), R12.2, R13.1
- new net: Q1.3 (C), R15.1
- new net: D1.3, R12.1
- new net +3V3: C11.1, C7.1, FB2.2, U3.A2 (VOUT)
- new net ON_MONITOR: R10.2, R11.1
- new net VDD_BNO: C10.1, C9.1, FB2.1
- new net VSYS: C8.1, Q2.3 (D), R14.1, S1.1, S1.2
- no-connect marks 0 -> 1
Other:
- moved on the sheet: C8, R14

Commit message: 2022-08-29
Parts:
- added C11: 4.7uF/1608, Capacitor_SMD:C_0603_1608Metric, symbol Device:C
- added C13: 22uF/2012, Capacitor_SMD:C_0805_2012Metric, symbol Device:C
- added L1: 1uH/2012, Inductor_SMD:L_0805_2012Metric, symbol Device:L
- added R19: 499k, Resistor_SMD:R_0402_1005Metric, symbol Device:R
- added R20: 200k, Resistor_SMD:R_0402_1005Metric, symbol Device:R
- added R21: 100k, Resistor_SMD:R_0402_1005Metric, symbol Device:R
- added U3: TPS62A01ADRLR, Local_devices:SOTFL50P160X60-6N, symbol TPS62A01ADRLR:TPS62A01ADRLR
- renumbered C11 to C12, U3 to U4
Connections:
- net Earth: now also C11.2, C13.2, R21.1, U3.1 (GND)
- net at Q2.2 (S), R17.1, U4.A1 (VIN)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: now also C11.1, R19.1, U3.3 (VIN), U3.4 (EN)
- new net: L1.1, U3.2 (SW)
- new net: R20.1, R21.2, U3.5 (FB)
- new net: R19.2, U3.6 (PG)
- new net +1V8: C13.1, L1.2, R20.2
Other:
- moved on the sheet: C10, C12, C6, C7, C8, C9, D1, FB2, Q1, Q2, Q3, R10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
