File: 02_Culturit_Tx_Power.kicad_sch (KiCad schematic)
At the start: 29 parts, among them Q1 MMBT2222LT1G, Q2 FDN340P, Q3 MMBT2222LT1G, U3 TPS62A01ADRLR, U4 TCR3UG33A,LF

Commit message: 2022-09-14
Parts:
- FB2: footprint (none) -> Inductor_SMD:L_0402_1005Metric
Changed lines of the file:
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@@
     (property "Reference" "FB2" (id 0) (at 111.8108 111.76 90))
     (property "Value" "MMZ1005Y121CT000" (id 1) (at 111.8108 114.3 90))
-    (property "Footprint" "" (id 2) (at 111.76 117.602 90)
+    (property "Footprint" "Inductor_SMD:L_0402_1005Metric" (id 2) (at 111.76 117.602 90)
       (effects (font (size 1.27 1.27)) hide)
     )

Commit message: 2022-10-13
Parts:
- L1: MPN LQM21PN1R0MGHD -> DFE201210U-1R0M=P2
- Q1, Q3: value MMBT2222LT1G -> MMBT3904,215; MPN MMBT2222LT1G -> MMBT3904,215
- Q2: value FDN340P -> AO3401A; MPN FDN340P -> AO3401A
- R10, R12: MPN RC0402JR-07910KR -> RC0402JR-0710KL
- U4: MPN (none) -> TCR3UG33A,LF
Changed lines of the file:
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@@
   (paper "A4")
   (title_block
-    (date "2022-09-06")
+    (date "2022-10-13")
   )
   (junction (at 165.1 59.69) (diameter 0) (color 0 0 0 0)
@@
       (effects (font (size 1.27 1.27)) hide)
     )
-    (property "Datasheet" "~" (id 3) (at 215.9 123.19 0)
-      (effects (font (size 1.27 1.27)) hide)
-    )
-    (property "MPN" "LQM21PN1R0MGHD" (id 4) (at 215.9 123.19 90)
+    (property "Datasheet" "https://cn.mouser.com/ProductDetail/Murata-Electronics/DFE201210U-1R0M%3dP2?qs=AQlKX63v8RtVAgMsjSbz6w%3D%3D" (id 3) (at 215.9 123.19 0)
+      (effects (font (size 1.27 1.27)) hide)
+    )
+    (property "MPN" "DFE201210U-1R0M=P2" (id 4) (at 215.9 123.19 90)
       (effects (font (size 1.27 1.27)) hide)
     )
@@
       (effects (font (size 1.27 1.27)) (justify left))
     )
-    (property "Value" "MMBT2222LT1G" (id 1) (at 148.59 80.01 0)
+    (property "Value" "MMBT3904,215" (id 1) (at 148.59 80.01 0)
       (effects (font (size 1.27 1.27)) (justify right))
     )
@@
       (effects (font (size 1.27 1.27)) hide)
     )
-    (property "Datasheet" "https://www.mouser.kr/datasheet/2/308/MMBT2222LT1_D-1811600.pdf" (id 3) (at 148.59 82.55 0)
-      (effects (font (size 1.27 1.27)) hide)
-    )
-    (property "MPN" "MMBT2222LT1G" (id 4) (at 148.59 82.55 0)
+    (property "Datasheet" "https://cn.mouser.com/ProductDetail/Nexperia/MMBT3904215?qs=LOCUfHb8d9s%2FW6hzAJGDbw%3D%3D" (id 3) (at 148.59 82.55 0)
+      (effects (font (size 1.27 1.27)) hide)
+    )
+    (property "MPN" "MMBT3904,215" (id 4) (at 148.59 82.55 0)
       (effects (font (size 1.27 1.27)) hide)
     )
@@
       (effects (font (size 1.27 1.27)) (justify left) hide)
     )
-    (property "Datasheet" "" (id 3) (at 224.79 105.41 0)
+    (property "Datasheet" "https://cn.mouser.com/ProductDetail/Texas-Instruments/TPS62A01ADRLR?qs=tlsG%2FOw5FFjxQ1CGo801Kw%3D%3D" (id 3) (at 224.79 105.41 0)
       (effects (font (size 1.27 1.27)) (justify left) hide)
     )
@@
       (effects (font (size 1.27 1.27)) (justify left bottom) hide)
     )
-    (property "Datasheet" "" (id 3) (at 215.9 62.23 0)
+    (property "Datasheet" "https://cn.mouser.com/ProductDetail/Toshiba/TCR3UG33ALF?qs=0lQeLiL1qyaZy60Q7HF0yg%3D%3D" (id 3) (at 215.9 62.23 0)
       (effects (font (size 1.27 1.27)) (justify left bottom) hide)
     )
@@
     (property "MAXIMUM_PACKAGE_HEIGHT" "0.33mm" (id 7) (at 215.9 62.23 0)
       (effects (font (size 1.27 1.27)) (justify left bottom) hide)
+    )
+    (property "MPN" "TCR3UG33A,LF" (id 8) (at 215.9 62.23 0)
+      (effects (font (size 1.27 1.27)) hide)
     )
     (pin "A1")
@@
       (effects (font (size 1.27 1.27)) hide)
     )
-    (property "Datasheet" "https://product.tdk.com/en/system/files?file=dam/doc/product/emc/emc/beads/catalog/beads_commercial_signal_mmz1005_en.pdf" (id 3) (at 111.76 119.38 0)
+    (property "Datasheet" "https://cn.mouser.com/ProductDetail/TDK/MMZ1005Y121CT000?qs=sGAEpiMZZMukHu%252BjC5l7YXmIAtxpPm1GtwNJ54RkjIo%3D" (id 3) (at 111.76 119.38 0)
       (effects (font (size 1.27 1.27)) hide)
     )
@@
       (effects (font (size 1.27 1.27)) hide)
     )
-    (property "MPN" "RC0402JR-07910KR" (id 4) (at 63.5 95.25 0)
+    (property "MPN" "RC0402JR-0710KL" (id 4) (at 63.5 95.25 0)
       (effects (font (size 1.27 1.27)) hide)
     )
@@
     (in_bom yes) (on_board yes) (fields_autoplaced)
     (property "Reference" "Q2" (id 0) (at 127 52.07 90))
-    (property "Value" "FDN340P" (id 1) (at 127 54.61 90))
+    (property "Value" "AO3401A" (id 1) (at 127 54.61 90))
     (property "Footprint" "Local_devices:SOT23" (id 2) (at 124.46 57.15 0)
       (effects (font (size 1.27 1.27)) hide)
@@
       (effects (font (size 1.27 1.27)) hide)
     )
-    (property "MPN" "FDN340P" (id 4) (at 127 62.23 90)
+    (property "MPN" "AO3401A" (id 4) (at 127 62.23 90)
       (effects (font (size 1.27 1.27)) hide)
     )
@@
       (effects (font (size 1.27 1.27)) (justify left))
     )
-    (property "Value" "MMBT2222LT1G" (id 1) (at 129.54 83.8199 0)
+    (property "Value" "MMBT3904,215" (id 1) (at 129.54 83.8199 0)
       (effects (font (size 1.27 1.27)) (justify left))
     )
@@
       (effects (font (size 1.27 1.27)) hide)
     )
-    (property "Datasheet" "https://www.mouser.kr/datasheet/2/308/MMBT2222LT1_D-1811600.pdf" (id 3) (at 124.46 82.55 0)
-      (effects (font (size 1.27 1.27)) hide)
-    )
-    (property "MPN" "MMBT2222LT1G" (id 4) (at 124.46 82.55 0)
+    (property "Datasheet" "https://cn.mouser.com/ProductDetail/Nexperia/MMBT3904215?qs=LOCUfHb8d9s%2FW6hzAJGDbw%3D%3D" (id 3) (at 124.46 82.55 0)
+      (effects (font (size 1.27 1.27)) hide)
+    )
+    (property "MPN" "MMBT3904,215" (id 4) (at 124.46 82.55 0)
       (effects (font (size 1.27 1.27)) hide)
     )
@@
       (effects (font (size 1.27 1.27)) hide)
     )
-    (property "MPN" "RC0402JR-07910KR" (id 4) (at 105.41 82.55 0)
+    (property "MPN" "RC0402JR-0710KL" (id 4) (at 105.41 82.55 0)
       (effects (font (size 1.27 1.27)) hide)
     )
@@
       (effects (font (size 1.27 1.27)) (justify left bottom) hide)
     )
-    (property "Datasheet" "https://file.elecfans.com/web1/M00/B8/ED/o4YBAF6BmEGAH9mVAAh24-M3Ykk719.pdf?filename=SKSCLDE010-ALPS.pdf" (id 3) (at 55.88 91.44 0)
+    (property "Datasheet" "https://cn.mouser.com/ProductDetail/Alps-Alpine/SKSCLDE010?qs=6EGMNY9ZYDQWpz3nhZNkIQ%3D%3D" (id 3) (at 55.88 91.44 0)
       (effects (font (size 1.27 1.27)) (justify left bottom) hide)
     )
@@
       (effects (font (size 1.27 1.27)) (justify left bottom) hide)
     )
-    (property "Datasheet" "https://www.onsemi.com/pdf/datasheet/mmbd4148se-d.pdf" (id 3) (at 88.9 88.9 0)
+    (property "Datasheet" "https://cn.mouser.com/ProductDetail/onsemi-Fairchild/MMBD4148CC?qs=E58pcOqB2RLfMqQ5hwAraQ%3D%3D" (id 3) (at 88.9 88.9 0)
       (effects (font (size 1.27 1.27)) (justify left bottom) hide)
     )
