File: 02_Culturit_Tx_Power.kicad_sch (KiCad schematic)
At the start: 29 parts, among them Q1 MMBT2222LT1G, Q2 FDN340P, Q3 MMBT2222LT1G, U3 TPS62A01ADRLR, U4 TCR3UG33A,LF

Commit message: 2022-09-07
Parts:
- FB2: footprint (none) -> Inductor_SMD:L_0402_1005Metric
- U4: MPN (none) -> TCR3UG33A,LF
Changed lines of the file:
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@@
       (effects (font (size 1.27 1.27)) (justify left bottom) hide)
+    )
+    (property "MPN" "TCR3UG33A,LF" (id 8) (at 215.9 62.23 0)
+      (effects (font (size 1.27 1.27)) hide)
     )
     (pin "A1")
@@
     (property "Reference" "FB2" (id 0) (at 111.8108 111.76 90))
     (property "Value" "MMZ1005Y121CT000" (id 1) (at 111.8108 114.3 90))
-    (property "Footprint" "" (id 2) (at 111.76 117.602 90)
+    (property "Footprint" "Inductor_SMD:L_0402_1005Metric" (id 2) (at 111.76 117.602 90)
       (effects (font (size 1.27 1.27)) hide)
     )

Commit message: 2022-10-27
Parts:
- removed Q2: FDN340P, Local_devices:SOT23, symbol Device:Q_NMOS_GSD
- added Q2: Q_PMOS_GSD, Package_TO_SOT_SMD:SOT-23, symbol Device:Q_PMOS_GSD
Connections:
- net VSYS: now also Q2.2 (S)
- net at C11.1, R17.1, R19.1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: now also Q2.3 (D)
- net at R14.2, R15.2, R16.2: now also Q2.1 (G)
Changed lines of the file:
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@@
     (pin "2")
-  )
-  (symbol (lib_id "Device:Q_NMOS_GSD") (at 127 62.23 90) (unit 1)
-    (in_bom yes) (on_board yes) (fields_autoplaced)
-    (property "Reference" "Q2" (id 0) (at 127 52.07 90))
-    (property "Value" "FDN340P" (id 1) (at 127 54.61 90))
-    (property "Footprint" "Local_devices:SOT23" (id 2) (at 124.46 57.15 0)
-      (effects (font (size 1.27 1.27)) hide)
-    )
-    (property "Datasheet" "https://statics3.seeedstudio.com/fusion/opl/datasheet/305030026.pdf" (id 3) (at 127 62.23 0)
-      (effects (font (size 1.27 1.27)) hide)
-    )
-    (property "MPN" "FDN340P" (id 4) (at 127 62.23 90)
-      (effects (font (size 1.27 1.27)) hide)
-    )
-    (pin "1")
-    (pin "2")
-    (pin "3")
   )
   (symbol (lib_id "Device:C") (at 241.3 63.5 0) (mirror y) (unit 1)
@@
     (pin "2")
   )
+  (symbol (lib_id "Device:Q_PMOS_GSD") (at 127 62.23 270) (mirror x) (unit 1)
+    (in_bom yes) (on_board yes) (fields_autoplaced)
+    (property "Reference" "Q2" (id 0) (at 127 52.07 90))
+    (property "Value" "Q_PMOS_GSD" (id 1) (at 127 54.61 90))
+    (property "Footprint" "Package_TO_SOT_SMD:SOT-23" (id 2) (at 129.54 57.15 0)
+      (effects (font (size 1.27 1.27)) hide)
+    )
+    (property "Datasheet" "~" (id 3) (at 127 62.23 0)
+      (effects (font (size 1.27 1.27)) hide)
+    )
+    (property "MPN" "FDN352AP" (id 4) (at 127 62.23 90)
+      (effects (font (size 1.27 1.27)) hide)
+    )
+    (pin "1")
+    (pin "2")
+    (pin "3")
+  )
   (symbol (lib_id "power:Earth") (at 73.66 106.68 0) (unit 1)

Commit message: 2022-10-30
Parts:
- removed D1: MMBD4148, Local_devices:SOT23, symbol MMBD4148:MMBD4148
- removed Q1, Q3: MMBT2222LT1G, Local_devices:SOT23, symbol Device:Q_NPN_BEC
- removed R12: 10k, Resistor_SMD:R_0402_1005Metric, symbol Device:R
- removed R13: 20k, Resistor_SMD:R_0402_1005Metric, symbol Device:R
- removed R15, R16: 1k, Resistor_SMD:R_0402_1005Metric, symbol Device:R
- removed U4: TCR3UG33A,LF, Local_devices:BGA4N35P2X2_64X64X33, symbol TCR3UG33A_LF:TCR3UG33A,LF
- added Q1, Q3: FDV303N, Package_TO_SOT_SMD:SOT-23, symbol Device:Q_NMOS_GSD
- added U4: MIC5317-3.3YM5-TR, Local_devices:SOT95P280X145-5N, symbol MIC5317-3.3YM5-TR:MIC5317-3.3YM5-TR
- Q2: value Q_PMOS_GSD -> FDN352AP
- R11: value 20k -> 33k; MPN RC0402FR-0720KL -> RC0402FR-0733KL
- R18: value 1k -> 10k; MPN RC0402FR-071KL -> RC0402FR-0710KL
Connections:
- net +3V3: now also U4.5 (VOUT)
- net Earth: now also C6.1, R10.1, R18.2, S1.3, S1.4, Q1.1 (G), Q1.2 (S), Q3.2 (S), U4.2 (GND)
- net LDO_ON: now also R17.2, Q3.1 (G)
- net at C11.1, Q2.3 (D), R17.1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: now also U4.1 (VIN), U4.3 (EN)
- net at Q2.1 (G), R14.2: now also Q1.3 (D), Q3.3 (D)
- no-connect marks 1 -> 0
Other:
- moved on the sheet: R18

Commit message: 2022-11-01
Parts:
- L1: MPN LQM21PN1R0MGHD -> LQM21PN1R0MGHL
Connections:
- net Earth: no longer C6.1, Q1.1 (G), R10.1, S1.3, S1.4
- new net: C6.1, Q1.1 (G), R10.1, S1.3, S1.4
Changed lines of the file:
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@@
   (junction (at 241.3 59.69) (diameter 0) (color 0 0 0 0)
   )
-  (junction (at 111.76 82.55) (diameter 0) (color 0 0 0 0)
-  )
   (junction (at 198.12 59.69) (diameter 0) (color 0 0 0 0)
   )
@@
     (stroke (width 0) (type default) (color 0 0 0 0))
   )
-  (wire (pts (xy 96.52 82.55) (xy 111.76 82.55))
-    (stroke (width 0) (type default) (color 0 0 0 0))
-  )
   (wire (pts (xy 73.66 91.44) (xy 63.5 91.44))
     (stroke (width 0) (type default) (color 0 0 0 0))
@@
     (stroke (width 0) (type default) (color 0 0 0 0))
   )
-  (wire (pts (xy 111.76 82.55) (xy 119.38 82.55))
+  (wire (pts (xy 96.52 82.55) (xy 119.38 82.55))
     (stroke (width 0) (type default) (color 0 0 0 0))
   )
@@
   )
   (wire (pts (xy 203.2 107.95) (xy 200.66 107.95))
-    (stroke (width 0) (type default) (color 0 0 0 0))
-  )
-  (wire (pts (xy 111.76 82.55) (xy 111.76 92.71))
     (stroke (width 0) (type default) (color 0 0 0 0))
   )
@@
       (effects (font (size 1.27 1.27)) hide)
     )
-    (property "MPN" "LQM21PN1R0MGHD" (id 4) (at 215.9 123.19 90)
+    (property "MPN" "LQM21PN1R0MGHL" (id 4) (at 215.9 123.19 90)
       (effects (font (size 1.27 1.27)) hide)
     )
@@
     (pin "2")
   )
-  (symbol (lib_id "power:Earth") (at 111.76 92.71 0) (unit 1)
-    (in_bom yes) (on_board yes) (fields_autoplaced)
-    (property "Reference" "#PWR019" (id 0) (at 111.76 99.06 0)
-      (effects (font (size 1.27 1.27)) hide)
-    )
-    (property "Value" "Earth" (id 1) (at 111.76 96.52 0)
-      (effects (font (size 1.27 1.27)) hide)
-    )
-    (property "Footprint" "" (id 2) (at 111.76 92.71 0)
-      (effects (font (size 1.27 1.27)) hide)
-    )
-    (property "Datasheet" "~" (id 3) (at 111.76 92.71 0)
-      (effects (font (size 1.27 1.27)) hide)
-    )
-    (pin "1")
-  )
   (symbol (lib_id "power:Earth") (at 133.35 129.54 0) (unit 1)
