File: 03_Curturit_Tx_MDBT.kicad_sch (KiCad schematic)
At the start: 1 part, among them U13 MDBT50Q-1M

Commit message: 2022-08-08
Connections:
- net Earth: now reaches U13.1 (GND_1)
- net Earth: now also U13.15 (GND_3), U13.2 (GND_2), U13.33 (GND_4), U13.55 (GND_5)
- net +1V8: now reaches U13.28 (VDD)
- net +1V8: now also U13.30 (VDDH)
- net VUSB: now reaches U13.32 (VBUS)
Other:
- moved on the sheet: U13

Commit message: 2022-08-09
Parts:
- added C24: 100pF, Capacitor_SMD:C_0402_1005Metric, symbol Device:C
- added C25, C26: 12pF, Capacitor_SMD:C_0402_1005Metric, symbol Device:C
- added J3: FTR-105-02-L-D, Connector_PinHeader_1.27mm:PinHeader_2x05_P1.27mm_Vertical_SMD, symbol Connector_Generic:Conn_02x05_Odd_Even
- added LED3: IN-P32TATRGB, Local_devices:INP32TATRGB, symbol IN-P32TATRGB:IN-P32TATRGB
- added R24, R29, R30: 4.7k, Resistor_SMD:R_0402_1005Metric, symbol Device:R
- added R25, R26: 0, Resistor_SMD:R_0402_1005Metric, symbol Device:R
- added R32: 100, Resistor_SMD:R_0402_1005Metric, symbol Device:R
- added R33, R35: NC, Resistor_SMD:R_0402_1005Metric, symbol Device:R
- added R34, R36: 33, Resistor_SMD:R_0402_1005Metric, symbol Device:R
- added R37, R38: 360, Resistor_SMD:R_0402_1005Metric, symbol Device:R
- added SW2, SW3: EVQ-P7J01P, Local_devices:EVQP7J01P, symbol Switch:SW_MEC_5E
- added Y1: 32.768kHz, Crystal:Crystal_SMD_3215-2Pin_3.2x1.5mm, symbol Device:Crystal
Connections:
- net +1V8: now also C24.1, J3.1 (Pin_1), R24.1, R29.2, R30.2, R33.2, R35.2
- net AIN2_XDK: now also U13.20 (P0.04)
- net AIN3_XDK: now also U13.7 (P1.14)
- net CS: now also U13.48 (P0.24)
- net Earth: now also C24.2, C25.1, C26.1, J3.3 (Pin_3), J3.5 (Pin_5), J3.9 (Pin_9), R37.1, R38.1
- net GPIO0: now also U13.36 (P0.14)
- net GPIO1: now also U13.37 (P0.13)
- net GPIO2/INT1: now also U13.61 (P1.01)
- net GPIO3/INT2: now also U13.25 (P1.08)
- net GPIO4: now also U13.60 (P1.03)
- net GPIO5: now also U13.50 (P1.02)
- net GPIO_EXT1_XDK: now also U13.54 (P0.10/NFC2)
- net GPIO_EXT2_XDK: now also U13.52 (P0.09/NFC1)
- net IOXP_INT: now also U13.4 (P1.11)
- net MCU_LED_B: now also U13.29 (P0.12), R36.2
- net MCU_LED_G: now also U13.27 (P0.11), R34.2
- net MCU_LED_R: now also U13.23 (P0.07), R32.2
- net MCU_RESET: now also U13.40 (P0.18/RESET), J3.10 (Pin_10)
- net PROM_RW: now also U13.21 (P0.05), R29.1
- net PS_EN1: now also U13.9 (P0.03)
- net PS_EN2: now also U13.13 (P0.28)
- net PlugDet: now also U13.3 (P1.10)
- net SCK/SCL: now also U13.38 (P0.16)
- net SCL0: now also U13.19 (P0.26), R30.1
- net SDA0: now also U13.10 (P0.29), R24.2
- net SDI/SDA: now also U13.22 (P0.06)
- net SDO: now also U13.39 (P0.15)
- net SPI0_CS: now also U13.6 (P1.13)
- net SPI0_MISO: now also U13.14 (P0.30)
- net SPI0_MOSI: now also U13.8 (P1.15)
- net SPI0_SCK: now also U13.5 (P1.12)
- net SWDCLK: now also U13.53 (SWDCLK), J3.4 (Pin_4)
- net SWDIO: now also U13.51 (SWDIO), J3.2 (Pin_2)
- net SWDO: now also U13.47 (P1.00), J3.6 (Pin_6)
- net SWITCH1: now also U13.26 (P1.09), SW2.3 (K), SW2.4 (A)
- net SWITCH2: now also U13.49 (P0.25), SW3.3 (K), SW3.4 (A)
- net USBdata_N: now also U13.34 (D-)
- net USBdata_P: now also U13.35 (D+)
- net VBAT_MON: now also U13.12 (P0.31)
- net VBAT_MOT_EN: now also U13.11 (P0.02)
- net VDD_SEL: now also U13.16 (P0.27)
- net at U13.17 (P0.00/XL1): now also R25.2
- net at U13.18 (P0.01/XL2): now also R26.2
- new net: C26.2, R26.1, Y1.1
- new net: C25.2, R25.1, Y1.2
- new net: LED3.3 (K_GREEN), R34.1
- new net: LED3.1 (K_RED), R32.1
- new net: LED3.4 (K_BLUE), R36.1
- new net: R35.1, R37.2, SW2.1, SW2.2
- new net: R33.1, R38.2, SW3.1, SW3.2
- new net +2V8: LED3.2 (COM+)

Commit message: 2022-08-11 2
Parts:
- C24: MPN (none) -> CC0402JRNPO9BN101
- C25, C26: MPN (none) -> CC0402JRNPO9BN120
- LED3: MPN (none) -> IN-P32TATRGB
- R24, R29, R30: MPN (none) -> 0402WGJ0472TCE
- R25, R26: MPN (none) -> 0402WGF0000TCE
- R32: MPN (none) -> 0402WGF1000TCE
- R34, R36: MPN (none) -> 0402WGJ0330TCE
- R37, R38: MPN (none) -> RC0402FR-07360RL
- SW2, SW3: MPN (none) -> EVQ-P7J01P
- U13: MPN (none) -> MDBT50Q-M1V2; Manufacturer_Part_Number 113990583 -> 113990582
Changed lines of the file:
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@@
+      (effects (font (size 1.27 1.27)) hide)
+    )
+    (property "MPN" "0402WGJ0472TCE" (id 4) (at 83.82 110.49 0)
       (effects (font (size 1.27 1.27)) hide)
     )
@@
       (effects (font (size 1.27 1.27)) hide)
     )
+    (property "MPN" "0402WGJ0330TCE" (id 4) (at 77.47 157.48 0)
+      (effects (font (size 1.27 1.27)) hide)
+    )
     (pin "1")
     (pin "2")
@@
     )
     (property "Datasheet" "~" (id 3) (at 100.33 96.52 0)
+      (effects (font (size 1.27 1.27)) hide)
+    )
+    (property "MPN" "0402WGF0000TCE" (id 4) (at 100.33 96.52 0)
       (effects (font (size 1.27 1.27)) hide)
     )
@@
       (effects (font (size 1.27 1.27)) (justify left) hide)
     )
-    (property "Manufacturer_Part_Number" "113990583" (id 9) (at 163.83 68.58 0)
-      (effects (font (size 1.27 1.27)) (justify left) hide)
+    (property "Manufacturer_Part_Number" "113990582" (id 9) (at 163.83 68.58 0)
+      (effects (font (size 1.27 1.27)) (justify left) hide)
+    )
+    (property "MPN" "MDBT50Q-M1V2" (id 10) (at 124.46 53.34 0)
+      (effects (font (size 1.27 1.27)) hide)
     )
     (pin "1")
@@
       (effects (font (size 1.27 1.27)) hide)
     )
+    (property "MPN" "0402WGJ0472TCE" (id 4) (at 91.44 69.85 0)
+      (effects (font (size 1.27 1.27)) hide)
+    )
     (pin "1")
     (pin "2")
@@
       (effects (font (size 1.27 1.27)) hide)
     )
+    (property "MPN" "0402WGF1000TCE" (id 4) (at 77.47 154.94 0)
+      (effects (font (size 1.27 1.27)) hide)
+    )
     (pin "1")
     (pin "2")
@@
     )
     (property "Datasheet" "~" (id 3) (at 77.47 162.56 0)
+      (effects (font (size 1.27 1.27)) hide)
+    )
+    (property "MPN" "0402WGJ0330TCE" (id 4) (at 77.47 162.56 0)
       (effects (font (size 1.27 1.27)) hide)
     )
@@
       (effects (font (size 1.27 1.27)) hide)
     )
+    (property "MPN" "CC0402JRNPO9BN120" (id 4) (at 67.31 88.9 0)
+      (effects (font (size 1.27 1.27)) hide)
+    )
     (pin "1")
     (pin "2")
@@
     )
     (property "Datasheet" "~" (id 3) (at 106.68 168.91 0)
+      (effects (font (size 1.27 1.27)) hide)
+    )
+    (property "MPN" "RC0402FR-07360RL" (id 4) (at 106.68 168.91 0)
       (effects (font (size 1.27 1.27)) hide)
     )
@@
       (effects (font (size 1.27 1.27)) hide)
     )
+    (property "MPN" "CC0402JRNPO9BN120" (id 4) (at 67.31 96.52 0)
+      (effects (font (size 1.27 1.27)) hide)
+    )
     (pin "1")
     (pin "2")
@@
     )
     (property "Datasheet" "~" (id 3) (at 100.33 88.9 0)
+      (effects (font (size 1.27 1.27)) hide)
+    )
+    (property "MPN" "0402WGF0000TCE" (id 4) (at 100.33 88.9 0)
       (effects (font (size 1.27 1.27)) hide)
     )
@@
       (effects (font (size 1.27 1.27)) (justify left) hide)
     )
+    (property "MPN" "IN-P32TATRGB" (id 10) (at 68.58 154.94 0)
+      (effects (font (size 1.27 1.27)) hide)
+    )
     (pin "1")
     (pin "2")
@@
     )
     (property "Datasheet" "~" (id 3) (at 91.44 110.49 0)
+      (effects (font (size 1.27 1.27)) hide)
+    )
+    (property "MPN" "0402WGJ0472TCE" (id 4) (at 91.44 110.49 0)
       (effects (font (size 1.27 1.27)) hide)
     )
@@
       (effects (font (size 1.27 1.27)) hide)
     )
+    (property "MPN" "CC0402JRNPO9BN101" (id 4) (at 213.36 63.5 0)
+      (effects (font (size 1.27 1.27)) hide)
+    )
     (pin "1")
     (pin "2")
@@
     )
     (property "Datasheet" "~" (id 3) (at 144.78 168.91 0)
+      (effects (font (size 1.27 1.27)) hide)
+    )
+    (property "MPN" "RC0402FR-07360RL" (id 4) (at 144.78 168.91 0)
       (effects (font (size 1.27 1.27)) hide)
     )
@@
       (effects (font (size 1.27 1.27)) hide)
     )
+    (property "MPN" "EVQ-P7J01P" (id 4) (at 119.38 165.1 0)
+      (effects (font (size 1.27 1.27)) hide)
+    )
     (pin "1")
     (pin "2")
@@
       (effects (font (size 1.27 1.27)) hide)
     )
+    (property "MPN" "EVQ-P7J01P" (id 4) (at 157.48 165.1 0)
+      (effects (font (size 1.27 1.27)) hide)
+    )

Commit message: 2022-08-16
Parts:
- added R27: 10k, Resistor_SMD:R_0402_1005Metric, symbol Device:R
Connections:
- net +1V8: now also R27.2
- net MCU_RESET: now also R27.1
Changed lines of the file:
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@@
 (kicad_sch (version 20211123) (generator eeschema)
   (paper "A4")
+  (title_block
+    (date "2022-08-16")
+  )
   (junction (at 121.92 53.34) (diameter 0) (color 0 0 0 0)
   )
@@
   (junction (at 124.46 162.56) (diameter 0) (color 0 0 0 0)
   )
+  (junction (at 185.42 73.66) (diameter 0) (color 0 0 0 0)
+  )
   (junction (at 91.44 99.06) (diameter 0) (color 0 0 0 0)
   )
@@
     (stroke (width 0) (type default) (color 0 0 0 0))
   )
-  (wire (pts (xy 167.64 73.66) (xy 170.18 73.66))
+  (wire (pts (xy 167.64 73.66) (xy 185.42 73.66))
     (stroke (width 0) (type default) (color 0 0 0 0))
   )
@@
     (stroke (width 0) (type default) (color 0 0 0 0))
   )
+  (wire (pts (xy 190.5 78.74) (xy 185.42 78.74))
+    (stroke (width 0) (type default) (color 0 0 0 0))
+  )
   (wire (pts (xy 121.92 88.9) (xy 124.46 88.9))
     (stroke (width 0) (type default) (color 0 0 0 0))
@@
     (stroke (width 0) (type default) (color 0 0 0 0))
   )
+  (wire (pts (xy 185.42 78.74) (xy 185.42 73.66))
+    (stroke (width 0) (type default) (color 0 0 0 0))
+  )
   (wire (pts (xy 121.92 53.34) (xy 124.46 53.34))
     (stroke (width 0) (type default) (color 0 0 0 0))
   )
+  (wire (pts (xy 185.42 73.66) (xy 190.5 73.66))
+    (stroke (width 0) (type default) (color 0 0 0 0))
+  )
   (wire (pts (xy 167.64 104.14) (xy 170.18 104.14))
     (stroke (width 0) (type default) (color 0 0 0 0))
@@
     (effects (font (size 1.27 1.27)) (justify left))
   )
-  (hierarchical_label "MCU_RESET" (shape input) (at 170.18 73.66 0)
+  (hierarchical_label "MCU_RESET" (shape input) (at 190.5 73.66 0)
     (effects (font (size 1.27 1.27)) (justify left))
   )
@@
     (pin "2")
   )
+  (symbol (lib_id "Device:R") (at 194.31 78.74 90) (unit 1)
+    (in_bom yes) (on_board yes)
+    (property "Reference" "R27" (id 0) (at 191.77 76.2 90))
+    (property "Value" "10k" (id 1) (at 194.31 78.74 90))
+    (property "Footprint" "Resistor_SMD:R_0402_1005Metric" (id 2) (at 194.31 80.518 90)
+      (effects (font (size 1.27 1.27)) hide)
+    )
+    (property "Datasheet" "~" (id 3) (at 194.31 78.74 0)
+      (effects (font (size 1.27 1.27)) hide)
+    )
+    (property "MPN" "RC0402JR-0710KL" (id 4) (at 194.31 78.74 0)
+      (effects (font (size 1.27 1.27)) hide)
+    )
+    (pin "1")
+    (pin "2")
+  )
   (symbol (lib_id "power:+2V8") (at 30.48 152.4 0) (unit 1)
     (in_bom yes) (on_board yes) (fields_autoplaced)
@@
     (pin "2")
   )
+  (symbol (lib_id "power:+1V8") (at 198.12 78.74 270) (unit 1)
+    (in_bom yes) (on_board yes) (fields_autoplaced)
+    (property "Reference" "#PWR0188" (id 0) (at 194.31 78.74 0)
+      (effects (font (size 1.27 1.27)) hide)
+    )
+    (property "Value" "+1V8" (id 1) (at 201.93 78.7399 90)
+      (effects (font (size 1.27 1.27)) (justify left))
+    )
+    (property "Footprint" "" (id 2) (at 198.12 78.74 0)
+      (effects (font (size 1.27 1.27)) hide)
+    )
+    (property "Datasheet" "" (id 3) (at 198.12 78.74 0)
+      (effects (font (size 1.27 1.27)) hide)
+    )
+    (pin "1")
+  )
   (symbol (lib_id "Device:R") (at 106.68 156.21 180) (unit 1)

Commit message: 2022-08-26
Parts:
- removed C24: 100pF, Capacitor_SMD:C_0402_1005Metric, symbol Device:C
- removed J3: FTR-105-02-L-D, Connector_PinHeader_1.27mm:PinHeader_2x05_P1.27mm_Vertical_SMD, symbol Connector_Generic:Conn_02x05_Odd_Even
- removed R33, R35: NC, Resistor_SMD:R_0402_1005Metric, symbol Device:R
- removed R37, R38: 360, Resistor_SMD:R_0402_1005Metric, symbol Device:R
- removed SW2, SW3: EVQ-P7J01P, Local_devices:EVQP7J01P, symbol Switch:SW_MEC_5E
- added J2: SWD, symbol Connector_Generic:Conn_01x04
- added S2: SKSCLDE010, Local_devices:SKSCLDE010, symbol SKSCLDE010:SKSCLDE010
- renumbered C25 to C12, C26 to C13, LED3 to LED2, R29 to R19, R24 to R20, R30 to R21, R25 to R22, R26 to R23, R27 to R24, R32 to R25, R34 to R26, R36 to R27, U13 to U4
Connections:
- net +1V8: no longer R20.1, R24.2
- net Earth: now also J2.4 (Pin_4), S2.3, S2.4
- net MCU_RESET: now also S2.1, S2.2
- net SWDCLK: now also J2.3 (Pin_3)
- net SWDIO: now also J2.2 (Pin_2)
- net +2V8 renamed +3V3
- net +3V3: now also R20.1, R24.2, J2.1 (Pin_1)
- net VUSB renamed VBUS
Other:
- moved on the sheet: C12, C13, LED2, R19, R20, R21, R22, R23, R24, R25, R26, R27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

Commit message: 2022-08-29
Parts:
- removed J2: SWD, symbol Connector_Generic:Conn_01x04
- removed R20, R21: 4.7k, Resistor_SMD:R_0402_1005Metric, symbol Device:R
- added C16: 100nF, Capacitor_SMD:C_0402_1005Metric, symbol Device:C
- added U6: W25Q32JWZPIQ, Local_devices:SON127P600X500X80-9N-D, symbol W25Q32JWZPIQ:W25Q32JWZPIQ
- added U7: DS28E05R+T, Local_devices:SOT95P237X112-3N, symbol DS28E05R+T:DS28E05R+T
- renumbered C12 to C14, C13 to C15, R19 to R22, R22 to R23, R23 to R24, R24 to R25, R25 to R26, R26 to R27, R27 to R28, U4 to U5
Connections:
- net +1V8: now also C16.1, U6.8 (VCC)
- net Earth: now also C16.2, U6.4 (GND), U6.9 (EP), U7.3 (GND)
- net PROM_RW: now also U7.1 (IO)
- net AIN2_XDK: no longer names the net of U5.20 (P0.04)
- net AIN3_XDK: no longer names the net of U5.7 (P1.14)
- net CS renamed IMU_SPI_CS
- net GPIO0 renamed FLASH_D2
- net FLASH_D2: now also U6.3 (~{WP_(IO2})), U6.7 (~{HOLD_OR_}/RESET_(IO3))
- net GPIO1 renamed FLASH_D3
- net GPIO2/INT1 renamed IMU_INT1
- net GPIO3/INT2 renamed IMU_INT2
- net GPIO4: no longer names the net of U5.60 (P1.03)
- net GPIO5: no longer names the net of U5.50 (P1.02)
- net GPIO_EXT1_XDK: no longer names the net of U5.54 (P0.10/NFC2)
- net GPIO_EXT2_XDK: no longer names the net of U5.52 (P0.09/NFC1)
- net IOXP_INT: no longer names the net of U5.4 (P1.11)
- net PS_EN1 renamed LDO_ON
- net PS_EN2: no longer names the net of U5.13 (P0.28)
- net PlugDet: no longer names the net of U5.3 (P1.10)
- net SCK/SCL renamed IMU_SPI_SCK
- net SCL0: no longer names the net of U5.19 (P0.26)
- net SDA0: no longer names the net of U5.10 (P0.29)
- net SDI/SDA renamed IMU_SPI_MISO
- net SDO renamed IMU_SPI_MOSI
- net SPI0_CS renamed FLASH_SPI0_CS
- net FLASH_SPI0_CS: now also U6.1 (~{CS})
- net SPI0_MISO renamed FLASH_SPI0_MISO
- net FLASH_SPI0_MISO: now also U6.2 (DO_(IO1))
- net SPI0_MOSI renamed FLASH_SPI0_MOSI
- net FLASH_SPI0_MOSI: now also U6.5 (DI_(IO0))
- net SPI0_SCK renamed FLASH_SPI0_SCK
- net FLASH_SPI0_SCK: now also U6.6 (CLK)
- net SWITCH1: no longer names the net of U5.26 (P1.09)
- net SWITCH2: no longer names the net of U5.49 (P0.25)
- net VBAT_MON: no longer names the net of U5.12 (P0.31)
- net VBAT_MOT_EN renamed ON_MONITOR
- net VDD_SEL: no longer names the net of U5.16 (P0.27)
Other:
- moved on the sheet: C14, C15, LED2, R22, R23, R24, R25, R26, R27, R28, S2, U5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

Commit message: 2022-09-05
Connections:
- net FLASH_D2: now also U5.38 (P0.16); no longer U5.36 (P0.14)
- net FLASH_D3: now also U5.39 (P0.15); no longer U5.37 (P0.13)
- net IMU_INT1: now also U5.48 (P0.24); no longer U5.61 (P1.01)
- net IMU_INT2: now also U5.3 (P1.10); no longer U5.25 (P1.08)
- net IMU_SPI_CS: now also U5.46 (P0.22); no longer U5.48 (P0.24)
- net IMU_SPI_MISO: now also U5.43 (P0.21); no longer U5.22 (P0.06)
- net IMU_SPI_MOSI: now also U5.45 (P0.23); no longer U5.39 (P0.15)
- net IMU_SPI_SCK: now also U5.42 (P0.19); no longer U5.38 (P0.16)
- net MCU_LED_B: now also U5.4 (P1.11); no longer U5.29 (P0.12)
- net MCU_LED_R: now also U5.47 (P1.00); no longer U5.23 (P0.07)
- net ON_MONITOR: now also U5.37 (P0.13); no longer U5.11 (P0.02)
- net SWDO: now also U5.52 (P0.09/NFC1); no longer U5.47 (P1.00)
Changed lines of the file:
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@@
   (paper "A4")
   (title_block
-    (date "2022-08-26")
+    (date "2022-08-29")
   )
   (junction (at 88.9 57.15) (diameter 0) (color 0 0 0 0)
@@
     (stroke (width 0) (type default) (color 0 0 0 0))
   )
-  (wire (pts (xy 80.01 113.03) (xy 91.44 113.03))
+  (wire (pts (xy 146.05 95.25) (xy 134.62 95.25))
     (stroke (width 0) (type default) (color 0 0 0 0))
   )
@@
     (stroke (width 0) (type default) (color 0 0 0 0))
   )
-  (wire (pts (xy 80.01 128.27) (xy 91.44 128.27))
+  (wire (pts (xy 80.01 64.77) (xy 91.44 64.77))
     (stroke (width 0) (type default) (color 0 0 0 0))
   )
@@
     (effects (font (size 1.27 1.27)) (justify right bottom))
   )
-  (label "FLASH_D3" (at 134.62 69.85 0)
+  (label "FLASH_D3" (at 134.62 74.93 0)
     (effects (font (size 1.27 1.27)) (justify left bottom))
   )
@@
     (effects (font (size 1.27 1.27)) (justify left bottom))
   )
-  (label "MCU_LED_R" (at 80.01 113.03 0)
-    (effects (font (size 1.27 1.27)) (justify left bottom))
+  (label "MCU_LED_R" (at 146.05 95.25 180)
+    (effects (font (size 1.27 1.27)) (justify right bottom))
   )
   (label "FLASH_D2" (at 265.43 121.92 180)
@@
     (effects (font (size 1.27 1.27)) (justify left bottom))
   )
-  (label "MCU_LED_B" (at 80.01 128.27 0)
+  (label "MCU_LED_B" (at 80.01 64.77 0)
     (effects (font (size 1.27 1.27)) (justify left bottom))
   )
@@
     (effects (font (size 1.27 1.27)) (justify left bottom))
   )
-  (label "FLASH_D2" (at 134.62 67.31 0)
-    (effects (font (size 1.27 1.27)) (justify left bottom))
-  )
-  (hierarchical_label "IMU_INT1" (shape input) (at 134.62 130.81 0)
-    (effects (font (size 1.27 1.27)) (justify left))
-  )
-  (hierarchical_label "IMU_SPI_SCK" (shape input) (at 134.62 72.39 0)
-    (effects (font (size 1.27 1.27)) (justify left))
-  )
-  (hierarchical_label "IMU_INT2" (shape input) (at 91.44 118.11 180)
+  (label "FLASH_D2" (at 134.62 72.39 0)
+    (effects (font (size 1.27 1.27)) (justify left bottom))
+  )
+  (hierarchical_label "IMU_INT1" (shape input) (at 134.62 97.79 0)
+    (effects (font (size 1.27 1.27)) (justify left))
+  )
+  (hierarchical_label "IMU_SPI_SCK" (shape input) (at 134.62 82.55 0)
+    (effects (font (size 1.27 1.27)) (justify left))
+  )
+  (hierarchical_label "IMU_INT2" (shape input) (at 91.44 62.23 180)
     (effects (font (size 1.27 1.27)) (justify right))
   )
@@
     (effects (font (size 1.27 1.27)) (justify left))
   )
-  (hierarchical_label "ON_MONITOR" (shape input) (at 91.44 82.55 180)
-    (effects (font (size 1.27 1.27)) (justify right))
-  )
-  (hierarchical_label "SWDO" (shape input) (at 134.62 95.25 0)
+  (hierarchical_label "ON_MONITOR" (shape input) (at 134.62 69.85 0)
+    (effects (font (size 1.27 1.27)) (justify left))
+  )
+  (hierarchical_label "SWDO" (shape input) (at 134.62 107.95 0)
     (effects (font (size 1.27 1.27)) (justify left))
   )
@@
     (effects (font (size 1.27 1.27)) (justify left))
   )
-  (hierarchical_label "IMU_SPI_MOSI" (shape input) (at 134.62 74.93 0)
-    (effects (font (size 1.27 1.27)) (justify left))
-  )
-  (hierarchical_label "IMU_SPI_CS" (shape input) (at 134.62 97.79 0)
-    (effects (font (size 1.27 1.27)) (justify left))
-  )
-  (hierarchical_label "IMU_SPI_MISO" (shape input) (at 91.44 110.49 180)
-    (effects (font (size 1.27 1.27)) (justify right))
+  (hierarchical_label "IMU_SPI_MOSI" (shape input) (at 134.62 90.17 0)
+    (effects (font (size 1.27 1.27)) (justify left))
+  )
+  (hierarchical_label "IMU_SPI_CS" (shape input) (at 134.62 92.71 0)
+    (effects (font (size 1.27 1.27)) (justify left))
+  )
+  (hierarchical_label "IMU_SPI_MISO" (shape input) (at 134.62 85.09 0)
+    (effects (font (size 1.27 1.27)) (justify left))
   )
   (symbol (lib_id "Device:C") (at 270.51 125.73 0) (mirror y) (unit 1)

Commit message: 2022-09-05
Connections:
- net FLASH_D2: now also U5.36 (P0.14); no longer U5.38 (P0.16)
- net IMU_NRST: now reaches U5.41 (P0.17)
- net IMU_WAKE: now reaches U5.54 (P0.10/NFC2)
- new net IMU_BOOTN: U5.38 (P0.16)
Changed lines of the file:
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@@
   (paper "A4")
   (title_block
-    (date "2022-08-29")
+    (date "2022-09-05")
   )
   (junction (at 88.9 57.15) (diameter 0) (color 0 0 0 0)
@@
     (effects (font (size 1.27 1.27)) (justify left bottom))
   )
-  (label "FLASH_D2" (at 134.62 72.39 0)
+  (label "FLASH_D2" (at 134.62 67.31 0)
     (effects (font (size 1.27 1.27)) (justify left bottom))
   )
   (hierarchical_label "IMU_INT1" (shape input) (at 134.62 97.79 0)
+    (effects (font (size 1.27 1.27)) (justify left))
+  )
+  (hierarchical_label "IMU_BOOTN" (shape input) (at 134.62 72.39 0)
     (effects (font (size 1.27 1.27)) (justify left))
   )
@@
     (effects (font (size 1.27 1.27)) (justify left))
   )
+  (hierarchical_label "IMU_NRST" (shape input) (at 134.62 80.01 0)
+    (effects (font (size 1.27 1.27)) (justify left))
+  )
+  (hierarchical_label "IMU_WAKE" (shape input) (at 134.62 113.03 0)
+    (effects (font (size 1.27 1.27)) (justify left))
+  )
