File: 03_Curturit_Tx_MDBT.kicad_sch (KiCad schematic)
At the start: 14 parts, among them U5 MDBT50Q-1M, U6 W25Q32JWZPIQ, Y1 32.768kHz

Commit message: 2022-09-07 2
Parts:
- renumbered R23 to R22, R24 to R23, R25 to R24, R26 to R25, R27 to R26, R28 to R27
Changed lines of the file:
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@@
   (symbol (lib_id "power:Earth") (at 137.16 115.57 90) (unit 1)
     (in_bom yes) (on_board yes) (fields_autoplaced)
-    (property "Reference" "#PWR040" (id 0) (at 143.51 115.57 0)
+    (property "Reference" "#PWR039" (id 0) (at 143.51 115.57 0)
       (effects (font (size 1.27 1.27)) hide)
     )
@@
   (symbol (lib_id "Device:R") (at 252.73 83.82 90) (unit 1)
     (in_bom yes) (on_board yes)
-    (property "Reference" "R27" (id 0) (at 248.92 82.55 90)
+    (property "Reference" "R26" (id 0) (at 248.92 82.55 90)
       (effects (font (size 1.27 1.27)) (justify left))
     )
@@
   (symbol (lib_id "Device:R") (at 67.31 100.33 90) (unit 1)
     (in_bom yes) (on_board yes)
-    (property "Reference" "R24" (id 0) (at 63.5 99.06 90)
+    (property "Reference" "R23" (id 0) (at 63.5 99.06 90)
       (effects (font (size 1.27 1.27)) (justify left))
     )
@@
   (symbol (lib_id "power:Earth") (at 137.16 59.69 90) (unit 1)
     (in_bom yes) (on_board yes) (fields_autoplaced)
-    (property "Reference" "#PWR039" (id 0) (at 143.51 59.69 0)
+    (property "Reference" "#PWR038" (id 0) (at 143.51 59.69 0)
       (effects (font (size 1.27 1.27)) hide)
     )
@@
   (symbol (lib_id "power:+3V3") (at 165.1 82.55 270) (unit 1)
     (in_bom yes) (on_board yes) (fields_autoplaced)
-    (property "Reference" "#PWR042" (id 0) (at 161.29 82.55 0)
+    (property "Reference" "#PWR041" (id 0) (at 161.29 82.55 0)
       (effects (font (size 1.27 1.27)) hide)
     )
@@
   (symbol (lib_id "Device:R") (at 252.73 81.28 90) (unit 1)
     (in_bom yes) (on_board yes)
-    (property "Reference" "R26" (id 0) (at 248.92 80.01 90)
+    (property "Reference" "R25" (id 0) (at 248.92 80.01 90)
       (effects (font (size 1.27 1.27)) (justify left))
     )
@@
   (symbol (lib_id "Device:R") (at 252.73 88.9 90) (unit 1)
     (in_bom yes) (on_board yes)
-    (property "Reference" "R28" (id 0) (at 248.92 87.63 90)
+    (property "Reference" "R27" (id 0) (at 248.92 87.63 90)
       (effects (font (size 1.27 1.27)) (justify left))
     )
@@
   (symbol (lib_id "Device:R") (at 161.29 82.55 90) (unit 1)
     (in_bom yes) (on_board yes)
-    (property "Reference" "R25" (id 0) (at 158.75 80.01 90))
+    (property "Reference" "R24" (id 0) (at 158.75 80.01 90))
     (property "Value" "10k" (id 1) (at 161.29 82.55 90))
     (property "Footprint" "Resistor_SMD:R_0402_1005Metric" (id 2) (at 161.29 84.328 90)
@@
   (symbol (lib_id "power:Earth") (at 270.51 129.54 0) (unit 1)
     (in_bom yes) (on_board yes) (fields_autoplaced)
-    (property "Reference" "#PWR048" (id 0) (at 270.51 135.89 0)
+    (property "Reference" "#PWR046" (id 0) (at 270.51 135.89 0)
       (effects (font (size 1.27 1.27)) hide)
     )
@@
   (symbol (lib_id "power:Earth") (at 189.23 129.54 0) (unit 1)
     (in_bom yes) (on_board yes) (fields_autoplaced)
-    (property "Reference" "#PWR043" (id 0) (at 189.23 135.89 0)
+    (property "Reference" "#PWR042" (id 0) (at 189.23 135.89 0)
       (effects (font (size 1.27 1.27)) hide)
     )
@@
   (symbol (lib_id "power:VBUS") (at 137.16 57.15 270) (unit 1)
     (in_bom yes) (on_board yes) (fields_autoplaced)
-    (property "Reference" "#PWR038" (id 0) (at 133.35 57.15 0)
+    (property "Reference" "#PWR037" (id 0) (at 133.35 57.15 0)
       (effects (font (size 1.27 1.27)) hide)
     )
@@
   (symbol (lib_id "power:Earth") (at 219.71 139.7 0) (unit 1)
     (in_bom yes) (on_board yes) (fields_autoplaced)
-    (property "Reference" "#PWR045" (id 0) (at 219.71 146.05 0)
+    (property "Reference" "#PWR044" (id 0) (at 219.71 146.05 0)
       (effects (font (size 1.27 1.27)) hide)
     )
@@
   (symbol (lib_id "power:Earth") (at 88.9 92.71 270) (unit 1)
     (in_bom yes) (on_board yes) (fields_autoplaced)
-    (property "Reference" "#PWR035" (id 0) (at 82.55 92.71 0)
+    (property "Reference" "#PWR034" (id 0) (at 82.55 92.71 0)
       (effects (font (size 1.27 1.27)) hide)
     )
@@
   (symbol (lib_id "Device:R") (at 67.31 92.71 90) (unit 1)
     (in_bom yes) (on_board yes)
-    (property "Reference" "R23" (id 0) (at 63.5 91.44 90)
+    (property "Reference" "R22" (id 0) (at 63.5 91.44 90)
       (effects (font (size 1.27 1.27)) (justify left))
     )
@@
   (symbol (lib_id "power:+3V3") (at 205.74 78.74 0) (unit 1)
     (in_bom yes) (on_board yes) (fields_autoplaced)
-    (property "Reference" "#PWR044" (id 0) (at 205.74 82.55 0)
+    (property "Reference" "#PWR043" (id 0) (at 205.74 82.55 0)
       (effects (font (size 1.27 1.27)) hide)
     )
@@
   (symbol (lib_id "power:+1V8") (at 270.51 116.84 0) (unit 1)
     (in_bom yes) (on_board yes) (fields_autoplaced)
-    (property "Reference" "#PWR047" (id 0) (at 270.51 120.65 0)
+    (property "Reference" "#PWR045" (id 0) (at 270.51 120.65 0)
       (effects (font (size 1.27 1.27)) hide)
     )
@@
   (symbol (lib_id "power:Earth") (at 154.94 95.25 0) (unit 1)
     (in_bom yes) (on_board yes) (fields_autoplaced)
-    (property "Reference" "#PWR041" (id 0) (at 154.94 101.6 0)
+    (property "Reference" "#PWR040" (id 0) (at 154.94 101.6 0)
       (effects (font (size 1.27 1.27)) hide)
     )
@@
   (symbol (lib_id "power:Earth") (at 88.9 52.07 180) (unit 1)
     (in_bom yes) (on_board yes) (fields_autoplaced)
-    (property "Reference" "#PWR034" (id 0) (at 88.9 45.72 0)
+    (property "Reference" "#PWR033" (id 0) (at 88.9 45.72 0)
       (effects (font (size 1.27 1.27)) hide)
     )
@@
   (symbol (lib_id "power:+1V8") (at 88.9 130.81 90) (unit 1)
     (in_bom yes) (on_board yes) (fields_autoplaced)
-    (property "Reference" "#PWR037" (id 0) (at 92.71 130.81 0)
+    (property "Reference" "#PWR036" (id 0) (at 92.71 130.81 0)
       (effects (font (size 1.27 1.27)) hide)
     )
@@
   (symbol (lib_id "power:+1V8") (at 88.9 125.73 90) (unit 1)
     (in_bom yes) (on_board yes) (fields_autoplaced)
-    (property "Reference" "#PWR036" (id 0) (at 92.71 125.73 0)
-      (effects (font (size 1.27 1.27)) hide)
-    )
+    (property "Reference" "#PWR035" (id 0) (at 92.71 125.73 0)
+      (effects (font (size 1.27 1.27)) hide)
+    )

Commit message: 2022-09-07 3
Parts:
- removed C14, C15: 12pF, Capacitor_SMD:C_0402_1005Metric, symbol Device:C
- removed R22, R23: 0, Resistor_SMD:R_0402_1005Metric, symbol Device:R
- removed Y1: 32.768kHz, Crystal:Crystal_SMD_3215-2Pin_3.2x1.5mm, symbol Device:Crystal
Changed lines of the file:
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@@
   (junction (at 270.51 119.38) (diameter 0) (color 0 0 0 0)
   )
-  (junction (at 43.18 100.33) (diameter 0) (color 0 0 0 0)
-  )
   (junction (at 152.4 77.47) (diameter 0) (color 0 0 0 0)
   )
@@
   (junction (at 154.94 82.55) (diameter 0) (color 0 0 0 0)
   )
-  (junction (at 43.18 92.71) (diameter 0) (color 0 0 0 0)
-  )
   (wire (pts (xy 270.51 116.84) (xy 270.51 119.38))
     (stroke (width 0) (type default) (color 0 0 0 0))
@@
     (stroke (width 0) (type default) (color 0 0 0 0))
   )
-  (wire (pts (xy 91.44 97.79) (xy 71.12 97.79))
-    (stroke (width 0) (type default) (color 0 0 0 0))
-  )
   (wire (pts (xy 247.65 119.38) (xy 270.51 119.38))
     (stroke (width 0) (type default) (color 0 0 0 0))
@@
     (stroke (width 0) (type default) (color 0 0 0 0))
   )
-  (wire (pts (xy 27.94 92.71) (xy 30.48 92.71))
-    (stroke (width 0) (type default) (color 0 0 0 0))
-  )
   (wire (pts (xy 154.94 82.55) (xy 154.94 87.63))
     (stroke (width 0) (type default) (color 0 0 0 0))
@@
     (stroke (width 0) (type default) (color 0 0 0 0))
   )
-  (wire (pts (xy 27.94 100.33) (xy 30.48 100.33))
-    (stroke (width 0) (type default) (color 0 0 0 0))
-  )
   (wire (pts (xy 88.9 125.73) (xy 91.44 125.73))
     (stroke (width 0) (type default) (color 0 0 0 0))
@@
     (stroke (width 0) (type default) (color 0 0 0 0))
   )
-  (wire (pts (xy 71.12 92.71) (xy 71.12 97.79))
-    (stroke (width 0) (type default) (color 0 0 0 0))
-  )
   (wire (pts (xy 88.9 130.81) (xy 91.44 130.81))
     (stroke (width 0) (type default) (color 0 0 0 0))
@@
     (stroke (width 0) (type default) (color 0 0 0 0))
   )
-  (wire (pts (xy 43.18 100.33) (xy 63.5 100.33))
-    (stroke (width 0) (type default) (color 0 0 0 0))
-  )
   (wire (pts (xy 205.74 88.9) (xy 205.74 83.82))
     (stroke (width 0) (type default) (color 0 0 0 0))
   )
-  (wire (pts (xy 71.12 100.33) (xy 91.44 100.33))
-    (stroke (width 0) (type default) (color 0 0 0 0))
-  )
   (wire (pts (xy 88.9 52.07) (xy 88.9 57.15))
     (stroke (width 0) (type default) (color 0 0 0 0))
@@
     (stroke (width 0) (type default) (color 0 0 0 0))
   )
-  (wire (pts (xy 38.1 92.71) (xy 43.18 92.71))
-    (stroke (width 0) (type default) (color 0 0 0 0))
-  )
   (wire (pts (xy 154.94 87.63) (xy 157.48 87.63))
     (stroke (width 0) (type default) (color 0 0 0 0))
@@
   )
   (wire (pts (xy 80.01 64.77) (xy 91.44 64.77))
-    (stroke (width 0) (type default) (color 0 0 0 0))
-  )
-  (wire (pts (xy 43.18 92.71) (xy 63.5 92.71))
-    (stroke (width 0) (type default) (color 0 0 0 0))
-  )
-  (wire (pts (xy 38.1 100.33) (xy 43.18 100.33))
     (stroke (width 0) (type default) (color 0 0 0 0))
   )
@@
     (pin "1")
   )
-  (symbol (lib_id "Device:Crystal") (at 43.18 96.52 90) (unit 1)
-    (in_bom yes) (on_board yes)
-    (property "Reference" "Y1" (id 0) (at 46.99 95.2499 90)
-      (effects (font (size 1.27 1.27)) (justify right))
-    )
-    (property "Value" "32.768kHz" (id 1) (at 46.99 97.79 90)
-      (effects (font (size 1.27 1.27)) (justify right))
-    )
-    (property "Footprint" "Crystal:Crystal_SMD_3215-2Pin_3.2x1.5mm" (id 2) (at 43.18 96.52 0)
-      (effects (font (size 1.27 1.27)) hide)
-    )
-    (property "Datasheet" "https://www.mouser.kr/datasheet/2/3/ABS07-11028.pdf" (id 3) (at 43.18 96.52 0)
-      (effects (font (size 1.27 1.27)) hide)
-    )
-    (property "MPN" "ABS07-32.768KHZ-T" (id 4) (at 43.18 96.52 90)
-      (effects (font (size 1.27 1.27)) hide)
-    )
-    (pin "1")
-    (pin "2")
-  )
   (symbol (lib_id "Device:R") (at 252.73 83.82 90) (unit 1)
     (in_bom yes) (on_board yes)
@@
     (pin "3")
     (pin "4")
-  )
-  (symbol (lib_id "power:Earth") (at 27.94 100.33 270) (unit 1)
-    (in_bom yes) (on_board yes) (fields_autoplaced)
-    (property "Reference" "#PWR032" (id 0) (at 21.59 100.33 0)
-      (effects (font (size 1.27 1.27)) hide)
-    )
-    (property "Value" "Earth" (id 1) (at 24.13 100.33 0)
-      (effects (font (size 1.27 1.27)) hide)
-    )
-    (property "Footprint" "" (id 2) (at 27.94 100.33 0)
-      (effects (font (size 1.27 1.27)) hide)
-    )
-    (property "Datasheet" "~" (id 3) (at 27.94 100.33 0)
-      (effects (font (size 1.27 1.27)) hide)
-    )
-    (pin "1")
-  )
-  (symbol (lib_id "Device:R") (at 67.31 100.33 90) (unit 1)
-    (in_bom yes) (on_board yes)
-    (property "Reference" "R23" (id 0) (at 63.5 99.06 90)
-      (effects (font (size 1.27 1.27)) (justify left))
-    )
-    (property "Value" "0" (id 1) (at 67.31 100.33 90))
-    (property "Footprint" "Resistor_SMD:R_0402_1005Metric" (id 2) (at 67.31 102.108 90)
-      (effects (font (size 1.27 1.27)) hide)
-    )
-    (property "Datasheet" "~" (id 3) (at 67.31 100.33 0)
-      (effects (font (size 1.27 1.27)) hide)
-    )
-    (property "MPN" "0402WGF0000TCE" (id 4) (at 67.31 100.33 0)
-      (effects (font (size 1.27 1.27)) hide)
-    )
-    (pin "1")
-    (pin "2")
   )
   (symbol (lib_id "power:Earth") (at 137.16 59.69 90) (unit 1)
@@
     (pin "2")
   )
-  (symbol (lib_id "Device:C") (at 34.29 92.71 90) (unit 1)
-    (in_bom yes) (on_board yes)
-    (property "Reference" "C14" (id 0) (at 29.21 91.44 90))
-    (property "Value" "12pF" (id 1) (at 34.29 88.9 90))
-    (property "Footprint" "Capacitor_SMD:C_0402_1005Metric" (id 2) (at 38.1 91.7448 0)
-      (effects (font (size 1.27 1.27)) hide)
-    )
-    (property "Datasheet" "~" (id 3) (at 34.29 92.71 0)
-      (effects (font (size 1.27 1.27)) hide)
-    )
-    (property "MPN" "CC0402JRNPO9BN120" (id 4) (at 34.29 92.71 0)
-      (effects (font (size 1.27 1.27)) hide)
-    )
-    (pin "1")
-    (pin "2")
-  )
-  (symbol (lib_id "Device:C") (at 34.29 100.33 90) (unit 1)
-    (in_bom yes) (on_board yes)
-    (property "Reference" "C15" (id 0) (at 29.21 99.06 90))
-    (property "Value" "12pF" (id 1) (at 34.29 96.52 90))
-    (property "Footprint" "Capacitor_SMD:C_0402_1005Metric" (id 2) (at 38.1 99.3648 0)
-      (effects (font (size 1.27 1.27)) hide)
-    )
-    (property "Datasheet" "~" (id 3) (at 34.29 100.33 0)
-      (effects (font (size 1.27 1.27)) hide)
-    )
-    (property "MPN" "CC0402JRNPO9BN120" (id 4) (at 34.29 100.33 0)
-      (effects (font (size 1.27 1.27)) hide)
-    )
-    (pin "1")
-    (pin "2")
-  )
   (symbol (lib_id "Device:R") (at 161.29 82.55 90) (unit 1)
     (in_bom yes) (on_board yes)
@@
     (pin "1")
   )
-  (symbol (lib_id "Device:R") (at 67.31 92.71 90) (unit 1)
-    (in_bom yes) (on_board yes)
-    (property "Reference" "R22" (id 0) (at 63.5 91.44 90)
-      (effects (font (size 1.27 1.27)) (justify left))
-    )
-    (property "Value" "0" (id 1) (at 67.31 92.71 90))
-    (property "Footprint" "Resistor_SMD:R_0402_1005Metric" (id 2) (at 67.31 94.488 90)
-      (effects (font (size 1.27 1.27)) hide)
-    )
-    (property "Datasheet" "~" (id 3) (at 67.31 92.71 0)
-      (effects (font (size 1.27 1.27)) hide)
-    )
-    (property "MPN" "0402WGF0000TCE" (id 4) (at 67.31 92.71 0)
-      (effects (font (size 1.27 1.27)) hide)
-    )
-    (pin "1")
-    (pin "2")
-  )
   (symbol (lib_id "power:+3V3") (at 205.74 78.74 0) (unit 1)
     (in_bom yes) (on_board yes) (fields_autoplaced)
@@
       (effects (font (size 1.27 1.27)) hide)
     )
-    (pin "1")
-  )
-  (symbol (lib_id "power:Earth") (at 27.94 92.71 270) (unit 1)
-    (in_bom yes) (on_board yes) (fields_autoplaced)
-    (property "Reference" "#PWR031" (id 0) (at 21.59 92.71 0)
-      (effects (font (size 1.27 1.27)) hide)
-    )
-    (property "Value" "Earth" (id 1) (at 24.13 92.71 0)
-      (effects (font (size 1.27 1.27)) hide)
-    )
-    (property "Footprint" "" (id 2) (at 27.94 92.71 0)
-      (effects (font (size 1.27 1.27)) hide)
-    )
-    (property "Datasheet" "~" (id 3) (at 27.94 92.71 0)
-      (effects (font (size 1.27 1.27)) hide)
-    )

Commit message: 2022-10-13
Parts:
- removed U6: W25Q32JWZPIQ, Local_devices:SON127P600X500X80-9N-D, symbol W25Q32JWZPIQ:W25Q32JWZPIQ
- added C14, C15: 12pF, Capacitor_SMD:C_0402_1005Metric, symbol Device:C
- added U6: MX25R6435FM2IH0, Package_SO:SOP-8_5.28x5.23mm_P1.27mm, symbol Memory_Flash:MX25R3235FM2xx0
- added Y1: 32.768MHz, Crystal:Crystal_SMD_2012-2Pin_2.0x1.2mm, symbol Device:Crystal
- U5: SKU (none) -> 113990582
Connections:
- net +1V8: now also C16.2, U6.8 (VCC); no longer C16.1
- net Earth: now also C16.1, C14.1, C15.1, U6.4 (GND); no longer C16.2
- net FLASH_SPI0_CS: now also U6.1 (~{CS})
- net FLASH_SPI0_SCK: now also U6.6 (SCLK)
- net at U5.17 (P0.00/XL1): now also C14.2, Y1.2
- net at U5.18 (P0.01/XL2): now also C15.2, Y1.1
- net BNO_BOOTN renamed GPIO_MCSB4
- net BNO_NRST renamed HOST_NRST
- net BNO_WAKE: no longer names the net of U5.54 (P0.10/NFC2)
- net FLASH_D2 renamed FLASH_SPI0_D2
- net FLASH_SPI0_D2: now also U6.3 (~{WP}/SIO2)
- net FLASH_D3 renamed FLASH_SPI0_D3
- net FLASH_SPI0_D3: now also U6.7 (~{RESET}/SIO3)
- net FLASH_SPI0_MISO renamed FLASH_SPI0_D1
- net FLASH_SPI0_D1: now also U6.2 (SO/SIO1)
- net FLASH_SPI0_MOSI renamed FLASH_SPI0_D0
- net FLASH_SPI0_D0: now also U6.5 (SI/SIO0)
