File: 03_Curturit_Tx_MDBT.kicad_sch (KiCad schematic)
At the start: 16 parts, among them U5 MDBT50Q-1M, U6 W25Q32JWZPIQ, U7 DS28E05R+T, Y1 32.768kHz

Commit message: 2022-09-06 1
Parts:
- removed R22: 4.7k, Resistor_SMD:R_0402_1005Metric, symbol Device:R
- removed U7: DS28E05R+T, Local_devices:SOT95P237X112-3N, symbol DS28E05R+T:DS28E05R+T
Connections:
- net FLASH_D2: no longer U6.7 (~{HOLD_OR_}/RESET_(IO3))
- net FLASH_D3: now also U6.7 (~{HOLD_OR_}/RESET_(IO3))
- net LDO_ON: now also U5.24 (P0.08); no longer U5.9 (P0.03)
- net BATT_SCL: now reaches U5.16 (P0.27)
- net GPOUT: now reaches U5.22 (P0.06)
- net BATT_SDA: now reaches U5.23 (P0.07)
- net BIN: now reaches U5.29 (P0.12)
- net IMU_BOOTN renamed BNO_BOOTN
- net IMU_INT1 renamed HOST_INTN
- net IMU_INT2: no longer names the net of U5.3 (P1.10)
- net IMU_NRST renamed BNO_NRST
- net IMU_SPI_CS renamed HOST_CSN
- net IMU_SPI_MISO renamed HOST_MISO
- net IMU_SPI_MOSI renamed HOST_MOSI
- net IMU_SPI_SCK renamed HOST_SCLK
- net IMU_WAKE renamed BNO_WAKE
- net PROM_RW: no longer names the net of U5.21 (P0.05)
- net SWDO: no longer names the net of U5.52 (P0.09/NFC1)
Changed lines of the file:
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@@
   (paper "A4")
   (title_block
-    (date "2022-09-05")
+    (date "2022-09-06")
   )
   (junction (at 88.9 57.15) (diameter 0) (color 0 0 0 0)
@@
   (junction (at 270.51 119.38) (diameter 0) (color 0 0 0 0)
   )
-  (junction (at 50.8 107.95) (diameter 0) (color 0 0 0 0)
-  )
   (junction (at 43.18 100.33) (diameter 0) (color 0 0 0 0)
   )
@@
     (stroke (width 0) (type default) (color 0 0 0 0))
   )
-  (wire (pts (xy 50.8 107.95) (xy 50.8 110.49))
-    (stroke (width 0) (type default) (color 0 0 0 0))
-  )
   (wire (pts (xy 154.94 82.55) (xy 152.4 82.55))
     (stroke (width 0) (type default) (color 0 0 0 0))
@@
     (stroke (width 0) (type default) (color 0 0 0 0))
   )
-  (wire (pts (xy 50.8 107.95) (xy 91.44 107.95))
-    (stroke (width 0) (type default) (color 0 0 0 0))
-  )
-  (wire (pts (xy 210.82 55.88) (xy 213.36 55.88))
-    (stroke (width 0) (type default) (color 0 0 0 0))
-  )
   (wire (pts (xy 154.94 87.63) (xy 157.48 87.63))
     (stroke (width 0) (type default) (color 0 0 0 0))
@@
     (stroke (width 0) (type default) (color 0 0 0 0))
   )
-  (wire (pts (xy 48.26 107.95) (xy 50.8 107.95))
-    (stroke (width 0) (type default) (color 0 0 0 0))
-  )
   (wire (pts (xy 43.18 92.71) (xy 63.5 92.71))
     (stroke (width 0) (type default) (color 0 0 0 0))
@@
   (wire (pts (xy 38.1 100.33) (xy 43.18 100.33))
     (stroke (width 0) (type default) (color 0 0 0 0))
-  )
-  (label "PROM_RW" (at 48.26 107.95 180)
-    (effects (font (size 1.27 1.27)) (justify right bottom))
   )
   (label "FLASH_SPI0_MOSI" (at 265.43 127 180)
@@
     (effects (font (size 1.27 1.27)) (justify right bottom))
   )
-  (label "FLASH_D2" (at 265.43 121.92 180)
+  (label "FLASH_D3" (at 265.43 121.92 180)
     (effects (font (size 1.27 1.27)) (justify right bottom))
   )
@@
     (effects (font (size 1.27 1.27)) (justify right bottom))
   )
-  (label "PROM_RW" (at 210.82 55.88 180)
-    (effects (font (size 1.27 1.27)) (justify right bottom))
-  )
   (label "FLASH_SPI0_SCK" (at 73.66 67.31 0)
     (effects (font (size 1.27 1.27)) (justify left bottom))
@@
     (effects (font (size 1.27 1.27)) (justify left bottom))
   )
-  (hierarchical_label "IMU_INT1" (shape input) (at 134.62 97.79 0)
-    (effects (font (size 1.27 1.27)) (justify left))
-  )
-  (hierarchical_label "IMU_BOOTN" (shape input) (at 134.62 72.39 0)
-    (effects (font (size 1.27 1.27)) (justify left))
-  )
-  (hierarchical_label "IMU_SPI_SCK" (shape input) (at 134.62 82.55 0)
-    (effects (font (size 1.27 1.27)) (justify left))
-  )
-  (hierarchical_label "IMU_INT2" (shape input) (at 91.44 62.23 180)
+  (hierarchical_label "HOST_INTN" (shape input) (at 134.62 97.79 0)
+    (effects (font (size 1.27 1.27)) (justify left))
+  )
+  (hierarchical_label "BATT_SDA" (shape input) (at 91.44 113.03 180)
     (effects (font (size 1.27 1.27)) (justify right))
   )
+  (hierarchical_label "BNO_BOOTN" (shape input) (at 134.62 72.39 0)
+    (effects (font (size 1.27 1.27)) (justify left))
+  )
+  (hierarchical_label "HOST_SCLK" (shape input) (at 134.62 82.55 0)
+    (effects (font (size 1.27 1.27)) (justify left))
+  )
+  (hierarchical_label "BATT_SCL" (shape input) (at 91.44 95.25 180)
+    (effects (font (size 1.27 1.27)) (justify right))
+  )
   (hierarchical_label "SWDIO" (shape input) (at 134.62 105.41 0)
     (effects (font (size 1.27 1.27)) (justify left))
@@
     (effects (font (size 1.27 1.27)) (justify left))
   )
-  (hierarchical_label "SWDO" (shape input) (at 134.62 107.95 0)
-    (effects (font (size 1.27 1.27)) (justify left))
-  )
   (hierarchical_label "USBdata_P" (shape input) (at 137.16 64.77 0)
     (effects (font (size 1.27 1.27)) (justify left))
@@
     (effects (font (size 1.27 1.27)) (justify left))
   )
-  (hierarchical_label "LDO_ON" (shape input) (at 91.44 77.47 180)
+  (hierarchical_label "LDO_ON" (shape input) (at 91.44 115.57 180)
     (effects (font (size 1.27 1.27)) (justify right))
   )
@@
     (effects (font (size 1.27 1.27)) (justify left))
   )
-  (hierarchical_label "IMU_SPI_MOSI" (shape input) (at 134.62 90.17 0)
-    (effects (font (size 1.27 1.27)) (justify left))
-  )
-  (hierarchical_label "IMU_SPI_CS" (shape input) (at 134.62 92.71 0)
-    (effects (font (size 1.27 1.27)) (justify left))
-  )
-  (hierarchical_label "IMU_SPI_MISO" (shape input) (at 134.62 85.09 0)
-    (effects (font (size 1.27 1.27)) (justify left))
-  )
-  (hierarchical_label "IMU_NRST" (shape input) (at 134.62 80.01 0)
-    (effects (font (size 1.27 1.27)) (justify left))
-  )
-  (hierarchical_label "IMU_WAKE" (shape input) (at 134.62 113.03 0)
+  (hierarchical_label "HOST_MOSI" (shape input) (at 134.62 90.17 0)
+    (effects (font (size 1.27 1.27)) (justify left))
+  )
+  (hierarchical_label "BIN" (shape input) (at 91.44 128.27 180)
+    (effects (font (size 1.27 1.27)) (justify right))
+  )
+  (hierarchical_label "HOST_CSN" (shape input) (at 134.62 92.71 0)
+    (effects (font (size 1.27 1.27)) (justify left))
+  )
+  (hierarchical_label "HOST_MISO" (shape input) (at 134.62 85.09 0)
+    (effects (font (size 1.27 1.27)) (justify left))
+  )
+  (hierarchical_label "GPOUT" (shape input) (at 91.44 110.49 180)
+    (effects (font (size 1.27 1.27)) (justify right))
+  )
+  (hierarchical_label "BNO_NRST" (shape input) (at 134.62 80.01 0)
+    (effects (font (size 1.27 1.27)) (justify left))
+  )
+  (hierarchical_label "BNO_WAKE" (shape input) (at 134.62 113.03 0)
     (effects (font (size 1.27 1.27)) (justify left))
   )
@@
     (pin "1")
   )
-  (symbol (lib_id "Device:R") (at 50.8 114.3 0) (unit 1)
-    (in_bom yes) (on_board yes)
-    (property "Reference" "R22" (id 0) (at 52.07 110.49 0)
-      (effects (font (size 1.27 1.27)) (justify left))
-    )
-    (property "Value" "4.7k" (id 1) (at 50.8 114.3 90))
-    (property "Footprint" "Resistor_SMD:R_0402_1005Metric" (id 2) (at 49.022 114.3 90)
-      (effects (font (size 1.27 1.27)) hide)
-    )
-    (property "Datasheet" "~" (id 3) (at 50.8 114.3 0)
-      (effects (font (size 1.27 1.27)) hide)
-    )
-    (property "MPN" "0402WGJ0472TCE" (id 4) (at 50.8 114.3 0)
-      (effects (font (size 1.27 1.27)) hide)
-    )
-    (pin "1")
-    (pin "2")
-  )
   (symbol (lib_id "Device:Crystal") (at 43.18 96.52 90) (unit 1)
     (in_bom yes) (on_board yes)
@@
     )
     (property "Datasheet" "~" (id 3) (at 137.16 59.69 0)
-      (effects (font (size 1.27 1.27)) hide)
-    )
-    (pin "1")
-  )
-  (symbol (lib_id "power:Earth") (at 238.76 55.88 90) (unit 1)
-    (in_bom yes) (on_board yes) (fields_autoplaced)
-    (property "Reference" "#PWR046" (id 0) (at 245.11 55.88 0)
-      (effects (font (size 1.27 1.27)) hide)
-    )
-    (property "Value" "Earth" (id 1) (at 242.57 55.88 0)
-      (effects (font (size 1.27 1.27)) hide)
-    )
-    (property "Footprint" "" (id 2) (at 238.76 55.88 0)
-      (effects (font (size 1.27 1.27)) hide)
-    )
-    (property "Datasheet" "~" (id 3) (at 238.76 55.88 0)
       (effects (font (size 1.27 1.27)) hide)
     )
@@
     (pin "1")
   )
-  (symbol (lib_id "DS28E05R+T:DS28E05R+T") (at 213.36 55.88 0) (unit 1)
-    (in_bom yes) (on_board yes) (fields_autoplaced)
-    (property "Reference" "U7" (id 0) (at 226.06 48.26 0))
-    (property "Value" "DS28E05R+T" (id 1) (at 226.06 50.8 0))
-    (property "Footprint" "Local_devices:SOT95P237X112-3N" (id 2) (at 234.95 53.34 0)
-      (effects (font (size 1.27 1.27)) (justify left) hide)
-    )
-    (property "Datasheet" "https://datasheets.maximintegrated.com/en/ds/DS28E05.pdf" (id 3) (at 234.95 55.88 0)
-      (effects (font (size 1.27 1.27)) (justify left) hide)
-    )
-    (property "Description" "EEPROM 1-Wire 112-BYTE EEPROM" (id 4) (at 234.95 58.42 0)
-      (effects (font (size 1.27 1.27)) (justify left) hide)
-    )
-    (property "Height" "1.12" (id 5) (at 234.95 60.96 0)
-      (effects (font (size 1.27 1.27)) (justify left) hide)
-    )
-    (property "Mouser Part Number" "700-DS28E05R+T" (id 6) (at 234.95 63.5 0)
-      (effects (font (size 1.27 1.27)) (justify left) hide)
-    )
-    (property "Mouser Price/Stock" "https://www.mouser.co.uk/ProductDetail/Maxim-Integrated/DS28E05R%2bT?qs=FoGyQ%2FpCy0g%252BVkc25tOVnQ%3D%3D" (id 7) (at 234.95 66.04 0)
-      (effects (font (size 1.27 1.27)) (justify left) hide)
-    )
-    (property "Manufacturer_Name" "Maxim Integrated" (id 8) (at 234.95 68.58 0)
-      (effects (font (size 1.27 1.27)) (justify left) hide)
-    )
-    (property "Manufacturer_Part_Number" "DS28E05R+T" (id 9) (at 234.95 71.12 0)
-      (effects (font (size 1.27 1.27)) (justify left) hide)
-    )
-    (property "MPN" "DS28E05R+T" (id 10) (at 213.36 55.88 0)
-      (effects (font (size 1.27 1.27)) hide)
-    )
-    (pin "1")
-    (pin "2")
-    (pin "3")
-  )
   (symbol (lib_id "IN-P32TATRGB:IN-P32TATRGB") (at 243.84 81.28 0) (mirror y) (unit 1)
     (in_bom yes) (on_board yes) (fields_autoplaced)
@@
       (effects (font (size 1.27 1.27)) hide)
     )
-    (pin "1")
-  )
-  (symbol (lib_id "power:+1V8") (at 50.8 118.11 180) (unit 1)
-    (in_bom yes) (on_board yes)
-    (property "Reference" "#PWR033" (id 0) (at 50.8 114.3 0)
-      (effects (font (size 1.27 1.27)) hide)
-    )
-    (property "Value" "+1V8" (id 1) (at 48.26 121.92 0)
-      (effects (font (size 1.27 1.27)) (justify right))
-    )
-    (property "Footprint" "" (id 2) (at 50.8 118.11 0)
-      (effects (font (size 1.27 1.27)) hide)
-    )
-    (property "Datasheet" "" (id 3) (at 50.8 118.11 0)
-      (effects (font (size 1.27 1.27)) hide)
-    )

Commit message: 2022-09-07
Parts:
- removed C15: 12pF, Capacitor_SMD:C_0402_1005Metric, symbol Device:C
- removed R23, R24: 0, Resistor_SMD:R_0402_1005Metric, symbol Device:R
- removed Y1: 32.768kHz, Crystal:Crystal_SMD_3215-2Pin_3.2x1.5mm, symbol Device:Crystal
- C14: value 12pF -> 10uF; footprint Capacitor_SMD:C_0402_1005Metric -> Capacitor_SMD:C_0603_1608Metric; MPN CC0402JRNPO9BN120 -> CC0603KRX5R6BB106
- renumbered R25 to R24, R26 to R25, R27 to R26, R28 to R27
Connections:
- net +1V8: now also C14.1, R24.2
- net +3V3: no longer R24.2
- net Earth: now also C14.2, S2.1, S2.2; no longer C14.1, S2.3, S2.4
- net MCU_RESET: now also S2.3, S2.4; no longer S2.1, S2.2
Other:
- moved on the sheet: S2

Commit message: 2022-10-24 added crystal
Parts:
- added C15, C17: 12pF, Capacitor_SMD:C_0402_1005Metric, symbol Device:C
- added Y1: 32.768kHz, Crystal:Crystal_SMD_2012-2Pin_2.0x1.2mm, symbol Device:Crystal
Connections:
- net Earth: now also C15.1, C17.2
- net at U5.17 (P0.00/XL1): now also C15.2, Y1.2
- net at U5.18 (P0.01/XL2): now also C17.1, Y1.1
Changed lines of the file:
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@@
   (junction (at 71.12 125.73) (diameter 0) (color 0 0 0 0)
   )
+  (junction (at 52.07 99.06) (diameter 0) (color 0 0 0 0)
+  )
+  (junction (at 64.77 95.25) (diameter 0) (color 0 0 0 0)
+  )
   (junction (at 71.12 130.81) (diameter 0) (color 0 0 0 0)
   )
@@
   (junction (at 154.94 95.25) (diameter 0) (color 0 0 0 0)
   )
+  (junction (at 64.77 102.87) (diameter 0) (color 0 0 0 0)
+  )
   (junction (at 154.94 87.63) (diameter 0) (color 0 0 0 0)
   )
@@
     (stroke (width 0) (type default) (color 0 0 0 0))
   )
+  (wire (pts (xy 59.69 102.87) (xy 64.77 102.87))
+    (stroke (width 0) (type default) (color 0 0 0 0))
+  )
   (wire (pts (xy 146.05 95.25) (xy 134.62 95.25))
     (stroke (width 0) (type default) (color 0 0 0 0))
@@
     (stroke (width 0) (type default) (color 0 0 0 0))
   )
+  (wire (pts (xy 64.77 95.25) (xy 78.74 95.25))
+    (stroke (width 0) (type default) (color 0 0 0 0))
+  )
   (wire (pts (xy 154.94 82.55) (xy 152.4 82.55))
     (stroke (width 0) (type default) (color 0 0 0 0))
@@
     (stroke (width 0) (type default) (color 0 0 0 0))
   )
+  (wire (pts (xy 59.69 95.25) (xy 64.77 95.25))
+    (stroke (width 0) (type default) (color 0 0 0 0))
+  )
   (wire (pts (xy 248.92 88.9) (xy 205.74 88.9))
     (stroke (width 0) (type default) (color 0 0 0 0))
@@
     (stroke (width 0) (type default) (color 0 0 0 0))
   )
+  (wire (pts (xy 78.74 95.25) (xy 78.74 97.79))
+    (stroke (width 0) (type default) (color 0 0 0 0))
+  )
+  (wire (pts (xy 91.44 100.33) (xy 78.74 100.33))
+    (stroke (width 0) (type default) (color 0 0 0 0))
+  )
   (wire (pts (xy 205.74 88.9) (xy 205.74 83.82))
     (stroke (width 0) (type default) (color 0 0 0 0))
@@
     (stroke (width 0) (type default) (color 0 0 0 0))
   )
+  (wire (pts (xy 78.74 100.33) (xy 78.74 102.87))
+    (stroke (width 0) (type default) (color 0 0 0 0))
+  )
+  (wire (pts (xy 78.74 97.79) (xy 91.44 97.79))
+    (stroke (width 0) (type default) (color 0 0 0 0))
+  )
   (wire (pts (xy 154.94 87.63) (xy 157.48 87.63))
     (stroke (width 0) (type default) (color 0 0 0 0))
@@
     (stroke (width 0) (type default) (color 0 0 0 0))
   )
+  (wire (pts (xy 52.07 95.25) (xy 52.07 99.06))
+    (stroke (width 0) (type default) (color 0 0 0 0))
+  )
   (wire (pts (xy 80.01 64.77) (xy 91.44 64.77))
+    (stroke (width 0) (type default) (color 0 0 0 0))
+  )
+  (wire (pts (xy 52.07 99.06) (xy 52.07 102.87))
+    (stroke (width 0) (type default) (color 0 0 0 0))
+  )
+  (wire (pts (xy 78.74 102.87) (xy 64.77 102.87))
     (stroke (width 0) (type default) (color 0 0 0 0))
   )
@@
     (pin "1")
   )
+  (symbol (lib_id "Device:C") (at 55.88 95.25 90) (unit 1)
+    (in_bom yes) (on_board yes) (fields_autoplaced)
+    (property "Reference" "C15" (id 0) (at 55.88 87.63 90))
+    (property "Value" "12pF" (id 1) (at 55.88 90.17 90))
+    (property "Footprint" "Capacitor_SMD:C_0402_1005Metric" (id 2) (at 59.69 94.2848 0)
+      (effects (font (size 1.27 1.27)) hide)
+    )
+    (property "Datasheet" "~" (id 3) (at 55.88 95.25 0)
+      (effects (font (size 1.27 1.27)) hide)
+    )
+    (pin "1")
+    (pin "2")
+  )
   (symbol (lib_id "Device:R") (at 252.73 83.82 90) (unit 1)
     (in_bom yes) (on_board yes)
@@
     (pin "3")
     (pin "4")
+  )
+  (symbol (lib_id "power:Earth") (at 52.07 99.06 270) (unit 1)
+    (in_bom yes) (on_board yes) (fields_autoplaced)
+    (property "Reference" "#PWR032" (id 0) (at 45.72 99.06 0)
+      (effects (font (size 1.27 1.27)) hide)
+    )
+    (property "Value" "Earth" (id 1) (at 48.26 99.06 0)
+      (effects (font (size 1.27 1.27)) hide)
+    )
+    (property "Footprint" "" (id 2) (at 52.07 99.06 0)
+      (effects (font (size 1.27 1.27)) hide)
+    )
+    (property "Datasheet" "~" (id 3) (at 52.07 99.06 0)
+      (effects (font (size 1.27 1.27)) hide)
+    )
+    (pin "1")
   )
   (symbol (lib_id "power:Earth") (at 137.16 59.69 90) (unit 1)
@@
     (pin "1")
   )
+  (symbol (lib_id "Device:Crystal") (at 64.77 99.06 90) (unit 1)
+    (in_bom yes) (on_board yes) (fields_autoplaced)
+    (property "Reference" "Y1" (id 0) (at 68.58 97.7899 90)
+      (effects (font (size 1.27 1.27)) (justify right))
+    )
+    (property "Value" "32.768kHz" (id 1) (at 68.58 100.3299 90)
+      (effects (font (size 1.27 1.27)) (justify right))
+    )
+    (property "Footprint" "Crystal:Crystal_SMD_2012-2Pin_2.0x1.2mm" (id 2) (at 64.77 99.06 0)
+      (effects (font (size 1.27 1.27)) hide)
+    )
+    (property "Datasheet" "~" (id 3) (at 64.77 99.06 0)
+      (effects (font (size 1.27 1.27)) hide)
+    )
+    (property "MPN" "FC-12M" (id 4) (at 64.77 99.06 90)
+      (effects (font (size 1.27 1.27)) hide)
+    )
+    (pin "1")
+    (pin "2")
+  )
   (symbol (lib_id "Device:R") (at 161.29 82.55 90) (unit 1)
     (in_bom yes) (on_board yes)
@@
     (pin "1")
   )
+  (symbol (lib_id "Device:C") (at 55.88 102.87 270) (unit 1)
+    (in_bom yes) (on_board yes)
+    (property "Reference" "C17" (id 0) (at 55.88 109.22 90))
+    (property "Value" "12pF" (id 1) (at 55.88 106.68 90))
+    (property "Footprint" "Capacitor_SMD:C_0402_1005Metric" (id 2) (at 52.07 103.8352 0)
+      (effects (font (size 1.27 1.27)) hide)
+    )
+    (property "Datasheet" "~" (id 3) (at 55.88 102.87 0)
+      (effects (font (size 1.27 1.27)) hide)
+    )
+    (pin "1")
+    (pin "2")
+  )
   (symbol (lib_id "power:+1V8") (at 165.1 82.55 270) (unit 1)
