File: 03_Curturit_Tx_MDBT.kicad_sch (KiCad schematic)
At the start: 13 parts, among them U5 MDBT50Q-1M, U6 W25Q32JWZPIQ, Y1 32.768kHz

Commit message: 2022-10-27
Parts:
- removed LED2: IN-P32TATRGB, Local_devices:INP32TATRGB, symbol IN-P32TATRGB:IN-P32TATRGB
- added LED2: CLV1L-FKB-CJ1N1E1BB7B3B3, LED_SMD:LED_Cree-PLCC4_3.2x2.8mm_CCW, symbol Device:LED_ARGB
- R26, R27: value 33 -> 100; MPN 0402WGJ0330TCE -> 0402WGF1000TCE
Connections:
- net +3V3: now also LED2.1 (A)
- net at R26.1: now also LED2.3 (GK)
- net at R25.1: now also LED2.2 (RK)
- net at R27.1: now also LED2.4 (BK)
Other:
- moved on the sheet: R25
Changed lines of the file:
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@@
-    (stroke (width 0) (type default) (color 0 0 0 0))
-  )
-  (wire (pts (xy 205.74 81.28) (xy 208.28 81.28))
-    (stroke (width 0) (type default) (color 0 0 0 0))
-  )
-  (wire (pts (xy 243.84 83.82) (xy 248.92 83.82))
     (stroke (width 0) (type default) (color 0 0 0 0))
   )
@@
     (stroke (width 0) (type default) (color 0 0 0 0))
   )
-  (wire (pts (xy 243.84 81.28) (xy 248.92 81.28))
-    (stroke (width 0) (type default) (color 0 0 0 0))
-  )
   (wire (pts (xy 59.69 95.25) (xy 64.77 95.25))
     (stroke (width 0) (type default) (color 0 0 0 0))
   )
-  (wire (pts (xy 248.92 88.9) (xy 205.74 88.9))
-    (stroke (width 0) (type default) (color 0 0 0 0))
-  )
   (wire (pts (xy 189.23 129.54) (xy 189.23 127))
     (stroke (width 0) (type default) (color 0 0 0 0))
@@
     (stroke (width 0) (type default) (color 0 0 0 0))
   )
-  (wire (pts (xy 205.74 88.9) (xy 205.74 83.82))
-    (stroke (width 0) (type default) (color 0 0 0 0))
-  )
   (wire (pts (xy 88.9 52.07) (xy 88.9 57.15))
     (stroke (width 0) (type default) (color 0 0 0 0))
   )
-  (wire (pts (xy 205.74 78.74) (xy 205.74 81.28))
-    (stroke (width 0) (type default) (color 0 0 0 0))
-  )
   (wire (pts (xy 78.74 100.33) (xy 78.74 102.87))
     (stroke (width 0) (type default) (color 0 0 0 0))
@@
   )
   (wire (pts (xy 247.65 121.92) (xy 265.43 121.92))
-    (stroke (width 0) (type default) (color 0 0 0 0))
-  )
-  (wire (pts (xy 205.74 83.82) (xy 208.28 83.82))
     (stroke (width 0) (type default) (color 0 0 0 0))
   )
@@
     (effects (font (size 1.27 1.27)) (justify left bottom))
   )
-  (label "MCU_LED_R" (at 256.54 81.28 0)
+  (label "MCU_LED_R" (at 228.6 77.47 0)
     (effects (font (size 1.27 1.27)) (justify left bottom))
   )
@@
     (effects (font (size 1.27 1.27)) (justify left bottom))
   )
-  (label "MCU_LED_B" (at 256.54 88.9 0)
+  (label "MCU_LED_B" (at 228.6 87.63 0)
     (effects (font (size 1.27 1.27)) (justify left bottom))
   )
@@
     (effects (font (size 1.27 1.27)) (justify left bottom))
   )
-  (label "MCU_LED_G" (at 256.54 83.82 0)
+  (label "MCU_LED_G" (at 228.6 82.55 0)
     (effects (font (size 1.27 1.27)) (justify left bottom))
   )
@@
     )
     (property "Datasheet" "~" (id 3) (at 55.88 95.25 0)
-      (effects (font (size 1.27 1.27)) hide)
-    )
-    (pin "1")
-    (pin "2")
-  )
-  (symbol (lib_id "Device:R") (at 252.73 83.82 90) (unit 1)
-    (in_bom yes) (on_board yes)
-    (property "Reference" "R26" (id 0) (at 248.92 82.55 90)
-      (effects (font (size 1.27 1.27)) (justify left))
-    )
-    (property "Value" "33" (id 1) (at 252.73 83.82 90))
-    (property "Footprint" "Resistor_SMD:R_0402_1005Metric" (id 2) (at 252.73 85.598 90)
-      (effects (font (size 1.27 1.27)) hide)
-    )
-    (property "Datasheet" "~" (id 3) (at 252.73 83.82 0)
-      (effects (font (size 1.27 1.27)) hide)
-    )
-    (property "MPN" "0402WGJ0330TCE" (id 4) (at 252.73 83.82 0)
       (effects (font (size 1.27 1.27)) hide)
     )
@@
     (pin "9")
   )
-  (symbol (lib_id "Device:R") (at 252.73 81.28 90) (unit 1)
+  (symbol (lib_id "Device:R") (at 224.79 87.63 90) (unit 1)
     (in_bom yes) (on_board yes)
-    (property "Reference" "R25" (id 0) (at 248.92 80.01 90)
+    (property "Reference" "R27" (id 0) (at 226.06 85.09 90)
       (effects (font (size 1.27 1.27)) (justify left))
     )
-    (property "Value" "100" (id 1) (at 252.73 81.28 90))
-    (property "Footprint" "Resistor_SMD:R_0402_1005Metric" (id 2) (at 252.73 83.058 90)
-      (effects (font (size 1.27 1.27)) hide)
-    )
-    (property "Datasheet" "~" (id 3) (at 252.73 81.28 0)
-      (effects (font (size 1.27 1.27)) hide)
-    )
-    (property "MPN" "0402WGF1000TCE" (id 4) (at 252.73 81.28 0)
-      (effects (font (size 1.27 1.27)) hide)
-    )
-    (pin "1")
-    (pin "2")
-  )
-  (symbol (lib_id "Device:R") (at 252.73 88.9 90) (unit 1)
+    (property "Value" "100" (id 1) (at 224.79 87.63 90))
+    (property "Footprint" "Resistor_SMD:R_0402_1005Metric" (id 2) (at 224.79 89.408 90)
+      (effects (font (size 1.27 1.27)) hide)
+    )
+    (property "Datasheet" "~" (id 3) (at 224.79 87.63 0)
+      (effects (font (size 1.27 1.27)) hide)
+    )
+    (property "MPN" "0402WGF1000TCE" (id 4) (at 224.79 87.63 0)
+      (effects (font (size 1.27 1.27)) hide)
+    )
+    (pin "1")
+    (pin "2")
+  )
+  (symbol (lib_id "Device:R") (at 224.79 77.47 90) (unit 1)
     (in_bom yes) (on_board yes)
-    (property "Reference" "R27" (id 0) (at 248.92 87.63 90)
+    (property "Reference" "R25" (id 0) (at 226.06 74.93 90)
       (effects (font (size 1.27 1.27)) (justify left))
     )
-    (property "Value" "33" (id 1) (at 252.73 88.9 90))
-    (property "Footprint" "Resistor_SMD:R_0402_1005Metric" (id 2) (at 252.73 90.678 90)
-      (effects (font (size 1.27 1.27)) hide)
-    )
-    (property "Datasheet" "~" (id 3) (at 252.73 88.9 0)
-      (effects (font (size 1.27 1.27)) hide)
-    )
-    (property "MPN" "0402WGJ0330TCE" (id 4) (at 252.73 88.9 0)
+    (property "Value" "100" (id 1) (at 224.79 77.47 90))
+    (property "Footprint" "Resistor_SMD:R_0402_1005Metric" (id 2) (at 224.79 79.248 90)
+      (effects (font (size 1.27 1.27)) hide)
+    )
+    (property "Datasheet" "~" (id 3) (at 224.79 77.47 0)
+      (effects (font (size 1.27 1.27)) hide)
+    )
+    (property "MPN" "0402WGF1000TCE" (id 4) (at 224.79 77.47 0)
+      (effects (font (size 1.27 1.27)) hide)
+    )
+    (pin "1")
+    (pin "2")
+  )
+  (symbol (lib_id "Device:R") (at 224.79 82.55 90) (unit 1)
+    (in_bom yes) (on_board yes)
+    (property "Reference" "R26" (id 0) (at 226.06 80.01 90)
+      (effects (font (size 1.27 1.27)) (justify left))
+    )
+    (property "Value" "100" (id 1) (at 224.79 82.55 90))
+    (property "Footprint" "Resistor_SMD:R_0402_1005Metric" (id 2) (at 224.79 84.328 90)
+      (effects (font (size 1.27 1.27)) hide)
+    )
+    (property "Datasheet" "~" (id 3) (at 224.79 82.55 0)
+      (effects (font (size 1.27 1.27)) hide)
+    )
+    (property "MPN" "0402WGF1000TCE" (id 4) (at 224.79 82.55 0)
       (effects (font (size 1.27 1.27)) hide)
     )
@@
     (pin "1")
     (pin "2")
+  )
+  (symbol (lib_id "Device:LED_ARGB") (at 215.9 82.55 0) (mirror y) (unit 1)
+    (in_bom yes) (on_board yes) (fields_autoplaced)
+    (property "Reference" "LED2" (id 0) (at 215.9 68.58 0))
+    (property "Value" "CLV1L-FKB-CJ1N1E1BB7B3B3" (id 1) (at 215.9 71.12 0))
+    (property "Footprint" "LED_SMD:LED_Cree-PLCC4_3.2x2.8mm_CCW" (id 2) (at 215.9 83.82 0)
+      (effects (font (size 1.27 1.27)) hide)
+    )
+    (property "Datasheet" "~" (id 3) (at 215.9 83.82 0)
+      (effects (font (size 1.27 1.27)) hide)
+    )
+    (property "MPN" "CLV1L-FKB-CJ1N1E1BB7B3B3" (id 4) (at 215.9 82.55 0)
+      (effects (font (size 1.27 1.27)) hide)
+    )
+    (pin "1")
+    (pin "2")
+    (pin "3")
+    (pin "4")
   )
   (symbol (lib_id "Device:R") (at 161.29 82.55 90) (unit 1)
@@
     (pin "1")
   )
-  (symbol (lib_id "power:+3V3") (at 205.74 78.74 0) (unit 1)
-    (in_bom yes) (on_board yes) (fields_autoplaced)
-    (property "Reference" "#PWR043" (id 0) (at 205.74 82.55 0)
-      (effects (font (size 1.27 1.27)) hide)
-    )
-    (property "Value" "+3V3" (id 1) (at 205.74 73.66 0))
-    (property "Footprint" "" (id 2) (at 205.74 78.74 0)
-      (effects (font (size 1.27 1.27)) hide)
-    )
-    (property "Datasheet" "" (id 3) (at 205.74 78.74 0)
-      (effects (font (size 1.27 1.27)) hide)
-    )
-    (pin "1")
-  )
-  (symbol (lib_id "IN-P32TATRGB:IN-P32TATRGB") (at 243.84 81.28 0) (mirror y) (unit 1)
-    (in_bom yes) (on_board yes) (fields_autoplaced)
-    (property "Reference" "LED2" (id 0) (at 226.06 73.66 0))
-    (property "Value" "IN-P32TATRGB" (id 1) (at 226.06 76.2 0))
-    (property "Footprint" "Local_devices:INP32TATRGB" (id 2) (at 212.09 78.74 0)
-      (effects (font (size 1.27 1.27)) (justify left) hide)
-    )
-    (property "Datasheet" "http://www.inolux-corp.com/datasheet/SMDLED/RGB%20Top%20View/IN-P32TATRGB_V1.0.pdf" (id 3) (at 212.09 81.28 0)
-      (effects (font (size 1.27 1.27)) (justify left) hide)
-    )
-    (property "Description" "Standard LEDs - SMD RGB LED" (id 4) (at 212.09 83.82 0)
-      (effects (font (size 1.27 1.27)) (justify left) hide)
-    )
-    (property "Height" "1.9" (id 5) (at 212.09 86.36 0)
-      (effects (font (size 1.27 1.27)) (justify left) hide)
-    )
-    (property "Mouser Part Number" "743-IN-P32TATRGB" (id 6) (at 212.09 88.9 0)
-      (effects (font (size 1.27 1.27)) (justify left) hide)
-    )
-    (property "Mouser Price/Stock" "https://www.mouser.co.uk/ProductDetail/Inolux/IN-P32TATRGB?qs=fAHHVMwC%252BbjKmGK7RdhY0g%3D%3D" (id 7) (at 212.09 91.44 0)
-      (effects (font (size 1.27 1.27)) (justify left) hide)
-    )
-    (property "Manufacturer_Name" "Inolux" (id 8) (at 212.09 93.98 0)
-      (effects (font (size 1.27 1.27)) (justify left) hide)
-    )
-    (property "Manufacturer_Part_Number" "IN-P32TATRGB" (id 9) (at 212.09 96.52 0)
-      (effects (font (size 1.27 1.27)) (justify left) hide)
-    )
-    (property "MPN" "IN-P32TATRGB" (id 10) (at 243.84 81.28 0)
-      (effects (font (size 1.27 1.27)) hide)
-    )
-    (pin "1")
-    (pin "2")
-    (pin "3")
-    (pin "4")
+  (symbol (lib_id "power:+3V3") (at 210.82 82.55 90) (unit 1)
+    (in_bom yes) (on_board yes) (fields_autoplaced)
+    (property "Reference" "#PWR043" (id 0) (at 214.63 82.55 0)
+      (effects (font (size 1.27 1.27)) hide)
+    )
+    (property "Value" "+3V3" (id 1) (at 207.01 82.5499 90)
+      (effects (font (size 1.27 1.27)) (justify left))
+    )
+    (property "Footprint" "" (id 2) (at 210.82 82.55 0)
+      (effects (font (size 1.27 1.27)) hide)
+    )
+    (property "Datasheet" "" (id 3) (at 210.82 82.55 0)
+      (effects (font (size 1.27 1.27)) hide)
+    )
+    (pin "1")
   )
   (symbol (lib_id "power:+1V8") (at 270.51 116.84 0) (unit 1)

Commit message: 2022-11-01
Parts:
- removed S2: SKSCLDE010, Local_devices:SKSCLDE010, symbol SKSCLDE010:SKSCLDE010
- added S2: Reset, Button_Switch_SMD:SW_SPST_B3U-1000P, symbol Switch:SW_Push
- C14: value 10uF -> 10uF/1608
- C15, C17: value 12pF -> 12pF/1005
- R25, R26, R27: value 100 -> 470; MPN 0402WGF1000TCE -> 0402WGF4700TCE
Connections:
- net Earth: now also S2.2
- net MCU_RESET: now also S2.1
Changed lines of the file:
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@@
   (junction (at 152.4 77.47) (diameter 0) (color 0 0 0 0)
   )
-  (junction (at 154.94 95.25) (diameter 0) (color 0 0 0 0)
-  )
   (junction (at 64.77 102.87) (diameter 0) (color 0 0 0 0)
   )
-  (junction (at 154.94 87.63) (diameter 0) (color 0 0 0 0)
-  )
   (junction (at 154.94 82.55) (diameter 0) (color 0 0 0 0)
   )
@@
     (stroke (width 0) (type default) (color 0 0 0 0))
   )
-  (wire (pts (xy 154.94 95.25) (xy 157.48 95.25))
-    (stroke (width 0) (type default) (color 0 0 0 0))
-  )
   (wire (pts (xy 173.99 119.38) (xy 191.77 119.38))
     (stroke (width 0) (type default) (color 0 0 0 0))
@@
   )
   (wire (pts (xy 78.74 97.79) (xy 91.44 97.79))
-    (stroke (width 0) (type default) (color 0 0 0 0))
-  )
-  (wire (pts (xy 154.94 87.63) (xy 157.48 87.63))
     (stroke (width 0) (type default) (color 0 0 0 0))
   )
@@
     (in_bom yes) (on_board yes) (fields_autoplaced)
     (property "Reference" "C15" (id 0) (at 55.88 87.63 90))
-    (property "Value" "12pF" (id 1) (at 55.88 90.17 90))
+    (property "Value" "12pF/1005" (id 1) (at 55.88 90.17 90))
     (property "Footprint" "Capacitor_SMD:C_0402_1005Metric" (id 2) (at 59.69 94.2848 0)
       (effects (font (size 1.27 1.27)) hide)
@@
     (pin "1")
     (pin "2")
-  )
-  (symbol (lib_id "SKSCLDE010:SKSCLDE010") (at 154.94 90.17 90) (unit 1)
-    (in_bom yes) (on_board yes) (fields_autoplaced)
-    (property "Reference" "S2" (id 0) (at 158.75 90.1699 90)
-      (effects (font (size 1.27 1.27)) (justify right))
-    )
-    (property "Value" "SKSCLDE010" (id 1) (at 158.75 92.7099 90)
-      (effects (font (size 1.27 1.27)) (justify right))
-    )
-    (property "Footprint" "Local_devices:SKSCLDE010" (id 2) (at 154.94 90.17 0)
-      (effects (font (size 1.27 1.27)) (justify left bottom) hide)
-    )
-    (property "Datasheet" "https://file.elecfans.com/web1/M00/B8/ED/o4YBAF6BmEGAH9mVAAh24-M3Ykk719.pdf?filename=SKSCLDE010-ALPS.pdf" (id 3) (at 154.94 90.17 0)
-      (effects (font (size 1.27 1.27)) (justify left bottom) hide)
-    )
-    (property "MPN" "SKSCLDE010" (id 4) (at 154.94 90.17 0)
-      (effects (font (size 1.27 1.27)) hide)
-    )
-    (pin "1")
-    (pin "2")
-    (pin "3")
-    (pin "4")
   )
   (symbol (lib_id "power:Earth") (at 52.07 99.06 270) (unit 1)
@@
       (effects (font (size 1.27 1.27)) (justify right))
     )
-    (property "Value" "10uF" (id 1) (at 72.39 137.16 0)
+    (property "Value" "10uF/1608" (id 1) (at 72.39 137.16 0)
       (effects (font (size 1.27 1.27)) (justify right))
     )
@@
       (effects (font (size 1.27 1.27)) (justify left))
     )
-    (property "Value" "100" (id 1) (at 224.79 87.63 90))
+    (property "Value" "470" (id 1) (at 224.79 87.63 90))
     (property "Footprint" "Resistor_SMD:R_0402_1005Metric" (id 2) (at 224.79 89.408 90)
       (effects (font (size 1.27 1.27)) hide)
@@
       (effects (font (size 1.27 1.27)) hide)
     )
-    (property "MPN" "0402WGF1000TCE" (id 4) (at 224.79 87.63 0)
+    (property "MPN" "0402WGF4700TCE" (id 4) (at 224.79 87.63 0)
       (effects (font (size 1.27 1.27)) hide)
     )
@@
       (effects (font (size 1.27 1.27)) (justify left))
     )
-    (property "Value" "100" (id 1) (at 224.79 77.47 90))
+    (property "Value" "470" (id 1) (at 224.79 77.47 90))
     (property "Footprint" "Resistor_SMD:R_0402_1005Metric" (id 2) (at 224.79 79.248 90)
       (effects (font (size 1.27 1.27)) hide)
@@
       (effects (font (size 1.27 1.27)) hide)
     )
-    (property "MPN" "0402WGF1000TCE" (id 4) (at 224.79 77.47 0)
+    (property "MPN" "0402WGF4700TCE" (id 4) (at 224.79 77.47 0)
       (effects (font (size 1.27 1.27)) hide)
     )
@@
       (effects (font (size 1.27 1.27)) (justify left))
     )
-    (property "Value" "100" (id 1) (at 224.79 82.55 90))
+    (property "Value" "470" (id 1) (at 224.79 82.55 90))
     (property "Footprint" "Resistor_SMD:R_0402_1005Metric" (id 2) (at 224.79 84.328 90)
       (effects (font (size 1.27 1.27)) hide)
@@
       (effects (font (size 1.27 1.27)) hide)
     )
-    (property "MPN" "0402WGF1000TCE" (id 4) (at 224.79 82.55 0)
+    (property "MPN" "0402WGF4700TCE" (id 4) (at 224.79 82.55 0)
       (effects (font (size 1.27 1.27)) hide)
     )
@@
     (pin "1")
   )
+  (symbol (lib_id "Switch:SW_Push") (at 154.94 92.71 270) (unit 1)
+    (in_bom yes) (on_board yes) (fields_autoplaced)
+    (property "Reference" "S2" (id 0) (at 158.75 91.4399 90)
+      (effects (font (size 1.27 1.27)) (justify left))
+    )
+    (property "Value" "Reset" (id 1) (at 158.75 93.9799 90)
+      (effects (font (size 1.27 1.27)) (justify left))
+    )
+    (property "Footprint" "Button_Switch_SMD:SW_SPST_B3U-1000P" (id 2) (at 160.02 92.71 0)
+      (effects (font (size 1.27 1.27)) hide)
+    )
+    (property "Datasheet" "~" (id 3) (at 160.02 92.71 0)
+      (effects (font (size 1.27 1.27)) hide)
+    )
+    (pin "1")
+    (pin "2")
+  )
   (symbol (lib_id "power:Earth") (at 88.9 92.71 270) (unit 1)
     (in_bom yes) (on_board yes) (fields_autoplaced)
@@
     (pin "1")
   )
-  (symbol (lib_id "power:Earth") (at 154.94 95.25 0) (unit 1)
-    (in_bom yes) (on_board yes) (fields_autoplaced)
-    (property "Reference" "#PWR040" (id 0) (at 154.94 101.6 0)
-      (effects (font (size 1.27 1.27)) hide)
-    )
-    (property "Value" "Earth" (id 1) (at 154.94 99.06 0)
-      (effects (font (size 1.27 1.27)) hide)
-    )
-    (property "Footprint" "" (id 2) (at 154.94 95.25 0)
-      (effects (font (size 1.27 1.27)) hide)
-    )
-    (property "Datasheet" "~" (id 3) (at 154.94 95.25 0)
+  (symbol (lib_id "power:Earth") (at 154.94 97.79 0) (unit 1)
+    (in_bom yes) (on_board yes) (fields_autoplaced)
+    (property "Reference" "#PWR040" (id 0) (at 154.94 104.14 0)
+      (effects (font (size 1.27 1.27)) hide)
+    )
+    (property "Value" "Earth" (id 1) (at 154.94 101.6 0)
+      (effects (font (size 1.27 1.27)) hide)
+    )
+    (property "Footprint" "" (id 2) (at 154.94 97.79 0)
+      (effects (font (size 1.27 1.27)) hide)
+    )
+    (property "Datasheet" "~" (id 3) (at 154.94 97.79 0)
       (effects (font (size 1.27 1.27)) hide)
     )
@@
     (in_bom yes) (on_board yes)
     (property "Reference" "C17" (id 0) (at 55.88 109.22 90))
-    (property "Value" "12pF" (id 1) (at 55.88 106.68 90))
+    (property "Value" "12pF/1005" (id 1) (at 55.88 106.68 90))
     (property "Footprint" "Capacitor_SMD:C_0402_1005Metric" (id 2) (at 52.07 103.8352 0)
       (effects (font (size 1.27 1.27)) hide)
