File: 04_Culturit_Tx_BHI260.kicad_sch (KiCad schematic)
At the start: 1 part, among them U15 BHI260AP

Commit message: 2022-08-09
Other:
- moved on the sheet: U15
Changed lines of the file:
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@@
 (kicad_sch (version 20211123) (generator eeschema)
   (paper "A4")
-  (symbol (lib_id "BHI260AP:BHI260AP") (at 139.7 72.39 0) (unit 1)
+  (symbol (lib_id "BHI260AP:BHI260AP") (at 95.25 68.58 0) (unit 1)
     (in_bom yes) (on_board yes) (fields_autoplaced)
-    (property "Reference" "U15" (id 0) (at 158.75 64.77 0))
-    (property "Value" "BHI260AP" (id 1) (at 158.75 67.31 0))
-    (property "Footprint" "Local_devices:BHI260AP" (id 2) (at 173.99 69.85 0)
+    (property "Reference" "U15" (id 0) (at 114.3 60.96 0))
+    (property "Value" "BHI260AP" (id 1) (at 114.3 63.5 0))
+    (property "Footprint" "Local_devices:BHI260AP" (id 2) (at 129.54 66.04 0)
       (effects (font (size 1.27 1.27)) (justify left) hide)
     )
-    (property "Datasheet" "https://www.bosch-sensortec.com/media/boschsensortec/downloads/datasheets/bst-bhi260ap-ds000.pdf" (id 3) (at 173.99 72.39 0)
+    (property "Datasheet" "https://www.bosch-sensortec.com/media/boschsensortec/downloads/datasheets/bst-bhi260ap-ds000.pdf" (id 3) (at 129.54 68.58 0)
       (effects (font (size 1.27 1.27)) (justify left) hide)
     )
-    (property "Description" "Multiple Function Sensor Modules Self-Learning AI sensor with integrated microcontroller and an IMU" (id 4) (at 173.99 74.93 0)
+    (property "Description" "Multiple Function Sensor Modules Self-Learning AI sensor with integrated microcontroller and an IMU" (id 4) (at 129.54 71.12 0)
       (effects (font (size 1.27 1.27)) (justify left) hide)
     )
-    (property "Height" "0.87" (id 5) (at 173.99 77.47 0)
+    (property "Height" "0.87" (id 5) (at 129.54 73.66 0)
       (effects (font (size 1.27 1.27)) (justify left) hide)
     )
-    (property "Mouser Part Number" "262-BHI260AP" (id 6) (at 173.99 80.01 0)
+    (property "Mouser Part Number" "262-BHI260AP" (id 6) (at 129.54 76.2 0)
       (effects (font (size 1.27 1.27)) (justify left) hide)
     )
-    (property "Mouser Price/Stock" "https://www.mouser.co.uk/ProductDetail/Bosch-Sensortec/BHI260AP?qs=T94vaHKWudTEPTnGI%252BTy9w%3D%3D" (id 7) (at 173.99 82.55 0)
+    (property "Mouser Price/Stock" "https://www.mouser.co.uk/ProductDetail/Bosch-Sensortec/BHI260AP?qs=T94vaHKWudTEPTnGI%252BTy9w%3D%3D" (id 7) (at 129.54 78.74 0)
       (effects (font (size 1.27 1.27)) (justify left) hide)
     )
-    (property "Manufacturer_Name" "Bosch Sensortec" (id 8) (at 173.99 85.09 0)
+    (property "Manufacturer_Name" "Bosch Sensortec" (id 8) (at 129.54 81.28 0)
       (effects (font (size 1.27 1.27)) (justify left) hide)
     )
-    (property "Manufacturer_Part_Number" "BHI260AP" (id 9) (at 173.99 87.63 0)
+    (property "Manufacturer_Part_Number" "BHI260AP" (id 9) (at 129.54 83.82 0)
       (effects (font (size 1.27 1.27)) (justify left) hide)
     )

Commit message: 2022-08-10
Parts:
- added C27, C29, C31, C32, C33: 100nF, Capacitor_SMD:C_0402_1005Metric, symbol Device:C
- added C28: 200nF, Capacitor_SMD:C_0402_1005Metric, symbol Device:C
- added C30: 1uF(1608), Capacitor_SMD:C_0603_1608Metric, symbol Device:C
- added LED4: ORANGE, LED_SMD:LED_0805_2012Metric, symbol Device:LED
- added R39, R40, R43, R44, R45, R46, R47, R52, R53, R54: 0, Resistor_SMD:R_0402_1005Metric, symbol Device:R
- added R41, R42, R48, R49, R50, R51: 4.7k, Resistor_SMD:R_0402_1005Metric, symbol Device:R
- added R55: 470, Resistor_SMD:R_0402_1005Metric, symbol Device:R
- added U14: BMM150, Package_CSP:WLCSP-12_1.56x1.56mm_P0.4mm, symbol Sensor_Magnetic:BMM150
- added U16: DS28E05R+T, Local_devices:SOT95P237X112-3N, symbol DS28E05R+T:DS28E05R+T
- added U17: W25Q32JWZPIQ, Local_devices:SON127P600X500X80-9N-D, symbol W25Q32JWZPIQ:W25Q32JWZPIQ
Connections:
- net at U15.1 (M3SDA): now also R50.2, R53.1
- net GPIO2/INT: now reaches U15.10 (HIRQ)
- net SDI/SDA: now reaches U15.11 (HSDX)
- net VDDIO: now reaches U15.12 (VDDIO_2)
- net VDDIO: now also U15.42 (VDDIO_3), U15.7 (VDDIO_1), C29.2, C30.2, C31.1, C32.1, C33.1, LED4.2 (A), R41.1, R42.1, R48.1, R49.1, R50.1, R51.1, U14.A1 (PS), U14.B2 (VDDIO), U14.E5 (VDD), U17.8 (VCC)
- net B260_TP12: now reaches U15.13 (M2SCX)
- net QSPI_CSN: now reaches U15.14 (QSPI_CSN)
- net QSPI_CSN: now also U17.1 (~{CS})
- net QSPI_D1: now reaches U15.15 (QSPI_D1)
- net QSPI_D1: now also U17.2 (DO_(IO1))
- net BMP390_INT: now reaches U15.16 (MCSB3)
- net Earth: now reaches U15.17 (GNDIO_1)
- net Earth: now also U15.25 (GND_1), U15.26 (GND_2), U15.27 (GND_3), U15.36 (GNDIO_2), C27.2, C28.1, C29.1, C30.1, C31.2, C32.2, C33.2, R46.2, R47.2, R54.1, U14.C5 (GND), U14.E1 (GND), U14.E3 (GND), U16.3 (GND), U17.4 (GND), U17.9 (EP)
- net BMM150_INT: now reaches U15.18 (MCSB2)
- net BMM150_INT: now also R40.2, R43.2
- net GPIO3/INT2: now reaches U15.19 (MCSB4)
- net at U15.2 (M3SCL): now also R51.2, R52.1
- net QSPI_D2: now reaches U15.20 (QSPI_D2)
- net QSPI_D2: now also U17.3 (~{WP_(IO2}))
- net B260_TP5: now reaches U15.21 (OCSB)
- net at U15.22 (ASCX): now also R42.2, R45.2
- net B260_TP7: now reaches U15.23 (JTAG_CLK)
- net B260_TP6: now reaches U15.24 (JTAG_DIO)
- net VDD: now reaches U15.28 (VDD)
- net VDD: now also C27.1
- net B260_TP9: now reaches U15.29 (M1SCX)
- net B260_TP9: now also R49.2
- net HOST_BOOT: now reaches U15.3 (HOSTBOOT)
- net HOST_BOOT: now also R54.2
- net at U15.30 (ASDX): now also R41.2, R44.2
- net B260_TP1: now reaches U15.31 (RESV3)
- net SDO: now reaches U15.32 (HSDO)
- net SCK/SCL: now reaches U15.33 (HSCX)
- net CS: now reaches U15.34 (HCSB)
- net B260_TP14: now reaches U15.35 (M2SDX)
- net B260_TP15: now reaches U15.37 (M2SDI)
- net at U15.38 (MCSB1): now also R55.2
- net B260_TP4: now reaches U15.39 (OSDO)
- net QSPI_D0: now reaches U15.4 (QSPI_D0)
- net QSPI_D0: now also U17.5 (DI_(IO0))
- net B260_TP2: now reaches U15.40 (RESV2)
- net B260_TP3: now reaches U15.41 (RESV1)
- net B260_TP11: now reaches U15.43 (M1SDI)
- net B260_TP10: now reaches U15.44 (M1SDX)
- net B260_TP10: now also R48.2
- net QSPI_CLK: now reaches U15.5 (QSPI_CLK)
- net QSPI_CLK: now also U17.6 (CLK)
- net at U15.6 (VREG): now also C28.2
- net QSPI_D3: now reaches U15.8 (QSPI_D3)
- net QSPI_D3: now also U17.7 (~{HOLD_OR_}/RESET_(IO3))
- net RESET: now reaches U15.9 (RESETN)
- net RESET: now also R39.1
- new net: R44.1, U14.B4 (SDI)
- new net: R45.1, U14.A3 (SCK)
- new net: LED4.1 (K), R55.1
- new net: R47.1, U14.C1 (SDO)
- new net: R46.1, U14.A5 (CSB)
- new net: R40.1, U14.D2 (INT)
- new net: R43.1, U14.D4 (DRDY)
- new net GPIO0: R52.2
- new net GPIO1: R53.2
- new net GPIO5: R39.2
- new net PROM_RW: U16.1 (IO)
Other:
- moved on the sheet: U15

Commit message: 2022-08-11 2
Parts:
- C27, C29, C31, C32, C33: MPN (none) -> CC0402KRX7R7BB104
- C28: MPN (none) -> CC0402KRX7R7BB224
- C30: MPN (none) -> CC0603KRX7R8BB105
- LED4: MPN (none) -> 17-215UYC/S530-A3/TR8
- R39, R40, R43, R44, R45, R46, R47, R52, R53, R54: MPN (none) -> 0402WGF0000TCE
- R41, R42, R48, R49, R50, R51: MPN (none) -> 0402WGJ0472TCE
- R55: MPN (none) -> RC0402FR-07470RL
- U14: MPN (none) -> BMM150
- U15: MPN (none) -> BHI260AP
- U16: MPN (none) -> DS28E05R+T
- U17: MPN (none) -> W25Q32JWZPIQ
Changed lines of the file:
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@@
+      (effects (font (size 1.27 1.27)) hide)
+    )
+    (property "MPN" "0402WGJ0472TCE" (id 4) (at 160.02 54.61 0)
       (effects (font (size 1.27 1.27)) hide)
     )
@@
       (effects (font (size 1.27 1.27)) hide)
     )
+    (property "MPN" "0402WGF0000TCE" (id 4) (at 57.15 50.8 0)
+      (effects (font (size 1.27 1.27)) hide)
+    )
     (pin "1")
     (pin "2")
@@
       (effects (font (size 1.27 1.27)) hide)
     )
+    (property "MPN" "CC0603KRX7R8BB105" (id 4) (at 26.67 60.96 0)
+      (effects (font (size 1.27 1.27)) hide)
+    )
     (pin "1")
     (pin "2")
@@
       (effects (font (size 1.27 1.27)) hide)
     )
+    (property "MPN" "CC0402KRX7R7BB104" (id 4) (at 227.33 50.8 0)
+      (effects (font (size 1.27 1.27)) hide)
+    )
     (pin "1")
     (pin "2")
@@
     )
     (property "Datasheet" "~" (id 3) (at 26.67 66.04 0)
+      (effects (font (size 1.27 1.27)) hide)
+    )
+    (property "MPN" "CC0402KRX7R7BB104" (id 4) (at 26.67 66.04 0)
       (effects (font (size 1.27 1.27)) hide)
     )
@@
       (effects (font (size 1.27 1.27)) hide)
     )
+    (property "MPN" "0402WGF0000TCE" (id 4) (at 182.88 60.96 0)
+      (effects (font (size 1.27 1.27)) hide)
+    )
     (pin "1")
     (pin "2")
@@
     )
     (property "Datasheet" "~" (id 3) (at 266.7 128.27 0)
+      (effects (font (size 1.27 1.27)) hide)
+    )
+    (property "MPN" "CC0402KRX7R7BB104" (id 4) (at 266.7 128.27 0)
       (effects (font (size 1.27 1.27)) hide)
     )
@@
       (effects (font (size 1.27 1.27)) hide)
     )
+    (property "MPN" "0402WGF0000TCE" (id 4) (at 57.15 53.34 0)
+      (effects (font (size 1.27 1.27)) hide)
+    )
     (pin "1")
     (pin "2")
@@
       (effects (font (size 1.27 1.27)) hide)
     )
+    (property "MPN" "0402WGJ0472TCE" (id 4) (at 127 118.11 0)
+      (effects (font (size 1.27 1.27)) hide)
+    )
     (pin "1")
     (pin "2")
@@
       (effects (font (size 1.27 1.27)) hide)
     )
+    (property "MPN" "0402WGJ0472TCE" (id 4) (at 162.56 54.61 0)
+      (effects (font (size 1.27 1.27)) hide)
+    )
     (pin "1")
     (pin "2")
@@
       (effects (font (size 1.27 1.27)) hide)
     )
+    (property "MPN" "0402WGJ0472TCE" (id 4) (at 68.58 44.45 0)
+      (effects (font (size 1.27 1.27)) hide)
+    )
     (pin "1")
     (pin "2")
@@
       (effects (font (size 1.27 1.27)) hide)
     )
+    (property "MPN" "0402WGJ0472TCE" (id 4) (at 66.04 44.45 0)
+      (effects (font (size 1.27 1.27)) hide)
+    )
     (pin "1")
     (pin "2")
@@
       (effects (font (size 1.27 1.27)) hide)
     )
+    (property "MPN" "0402WGF0000TCE" (id 4) (at 182.88 66.04 0)
+      (effects (font (size 1.27 1.27)) hide)
+    )
     (pin "1")
     (pin "2")
@@
       (effects (font (size 1.27 1.27)) hide)
     )
+    (property "MPN" "RC0402FR-07470RL" (id 4) (at 140.97 88.9 0)
+      (effects (font (size 1.27 1.27)) hide)
+    )
     (pin "1")
     (pin "2")
@@
       (effects (font (size 1.27 1.27)) hide)
     )
+    (property "MPN" "0402WGF0000TCE" (id 4) (at 78.74 44.45 0)
+      (effects (font (size 1.27 1.27)) hide)
+    )
     (pin "1")
     (pin "2")
@@
     (property "Manufacturer_Part_Number" "W25Q32JWZPIQ" (id 9) (at 245.11 137.16 0)
       (effects (font (size 1.27 1.27)) (justify left) hide)
+    )
+    (property "MPN" "W25Q32JWZPIQ" (id 10) (at 193.04 121.92 0)
+      (effects (font (size 1.27 1.27)) hide)
     )
     (pin "1")
@@
       (effects (font (size 1.27 1.27)) hide)
     )
+    (property "MPN" "CC0402KRX7R7BB224" (id 4) (at 57.15 63.5 0)
+      (effects (font (size 1.27 1.27)) hide)
+    )
     (pin "1")
     (pin "2")
@@
       (effects (font (size 1.27 1.27)) hide)
     )
+    (property "MPN" "0402WGF0000TCE" (id 4) (at 200.66 74.93 0)
+      (effects (font (size 1.27 1.27)) hide)
+    )
     (pin "1")
     (pin "2")
@@
       (effects (font (size 1.27 1.27)) (justify left) hide)
     )
+    (property "MPN" "DS28E05R+T" (id 10) (at 210.82 96.52 0)
+      (effects (font (size 1.27 1.27)) hide)
+    )
     (pin "1")
     (pin "2")
@@
     )
     (property "Datasheet" "https://www.mouser.com/datasheet/2/783/BST-BMM150-DS001-01-786480.pdf" (id 3) (at 212.09 57.15 0)
+      (effects (font (size 1.27 1.27)) hide)
+    )
+    (property "MPN" "BMM150" (id 4) (at 220.98 63.5 0)
       (effects (font (size 1.27 1.27)) hide)
     )
@@
       (effects (font (size 1.27 1.27)) hide)
     )
+    (property "MPN" "0402WGF0000TCE" (id 4) (at 240.03 63.5 0)
+      (effects (font (size 1.27 1.27)) hide)
+    )
     (pin "1")
     (pin "2")
@@
       (effects (font (size 1.27 1.27)) hide)
     )
+    (property "MPN" "0402WGF0000TCE" (id 4) (at 203.2 74.93 0)
+      (effects (font (size 1.27 1.27)) hide)
+    )
     (pin "1")
     (pin "2")
@@
       (effects (font (size 1.27 1.27)) hide)
     )
+    (property "MPN" "17-215UYC/S530-A3/TR8" (id 4) (at 148.59 88.9 0)
+      (effects (font (size 1.27 1.27)) hide)
+    )
     (pin "1")
     (pin "2")
@@
     )
     (property "Datasheet" "~" (id 3) (at 138.43 63.5 0)
+      (effects (font (size 1.27 1.27)) hide)
+    )
+    (property "MPN" "CC0402KRX7R7BB104" (id 4) (at 138.43 63.5 0)
       (effects (font (size 1.27 1.27)) hide)
     )
@@
       (effects (font (size 1.27 1.27)) hide)
     )
+    (property "MPN" "0402WGJ0472TCE" (id 4) (at 127 39.37 0)
+      (effects (font (size 1.27 1.27)) hide)
+    )
     (pin "1")
     (pin "2")
@@
       (effects (font (size 1.27 1.27)) hide)
     )
+    (property "MPN" "0402WGF0000TCE" (id 4) (at 59.69 71.12 0)
+      (effects (font (size 1.27 1.27)) hide)
+    )
     (pin "1")
     (pin "2")
@@
     )
     (property "Datasheet" "~" (id 3) (at 227.33 45.72 0)
+      (effects (font (size 1.27 1.27)) hide)
+    )
+    (property "MPN" "CC0402KRX7R7BB104" (id 4) (at 227.33 45.72 0)
       (effects (font (size 1.27 1.27)) hide)
     )
@@
       (effects (font (size 1.27 1.27)) hide)
     )
+    (property "MPN" "0402WGF0000TCE" (id 4) (at 240.03 60.96 0)
+      (effects (font (size 1.27 1.27)) hide)
+    )
     (pin "1")
     (pin "2")
@@
       (effects (font (size 1.27 1.27)) (justify left) hide)
     )
-    (pin "1")
+    (property "MPN" "BHI260AP" (id 10) (at 81.28 50.8 0)
+      (effects (font (size 1.27 1.27)) hide)
+    )
+    (pin "1")

Commit message: 2022-08-26
Parts:
- renumbered C30 to C14, C29 to C15, C28 to C16, C27 to C17, C31 to C18, C32 to C19, C33 to C20, LED4 to LED3, R53 to R28, R52 to R29, R39 to R30, R51 to R31, R50 to R32, R54 to R33, R49 to R34, R48 to R35, R55 to R36, R41 to R37, R42 to R38, R44 to R39, R45 to R40, R47 to R41, R46 to R42, R40 to R44, U15 to U5, U17 to U6, U16 to U7, U14 to U8

Commit message: 2022-08-29
Parts:
- removed R28, R29, R30: 0, Resistor_SMD:R_0402_1005Metric, symbol Device:R
- removed R31, R32, R34, R35: 4.7k, Resistor_SMD:R_0402_1005Metric, symbol Device:R
- removed U7: DS28E05R+T, Local_devices:SOT95P237X112-3N, symbol DS28E05R+T:DS28E05R+T
- renumbered C14 to C17, C15 to C18, C16 to C19, C17 to C20, C18 to C21, C19 to C22, C20 to C23, R33 to R29, R36 to R30, R37 to R31, R38 to R32, R39 to R33, R40 to R34, R41 to R35, R42 to R36, R43 to R37, R44 to R38, U8 to U10, U5 to U8, U6 to U9
Connections:
- net VDDIO is gone; now on net +1V8: C17.2, C18.2, C21.1, C22.1, C23.1, LED3.2 (A), R31.1, R32.1, U10.A1 (PS), U10.B2 (VDDIO), U10.E5 (VDD), U8.12 (VDDIO_2), U8.42 (VDDIO_3), U8.7 (VDDIO_1), U9.8 (VCC)
- net QSPI_D1: no longer U9.2 (DO_(IO1))
- net QSPI_D2: no longer U9.3 (~{WP_(IO2}))
- net B260_TP1: no longer names the net of U8.31 (RESV3)
- net B260_TP10: no longer names the net of U8.44 (M1SDX)
- net B260_TP11: no longer names the net of U8.43 (M1SDI)
- net B260_TP12: no longer names the net of U8.13 (M2SCX)
- net B260_TP14: no longer names the net of U8.35 (M2SDX)
- net B260_TP15: no longer names the net of U8.37 (M2SDI)
- net B260_TP2: no longer names the net of U8.40 (RESV2)
- net B260_TP3: no longer names the net of U8.41 (RESV1)
- net B260_TP4: no longer names the net of U8.39 (OSDO)
- net B260_TP5: no longer names the net of U8.21 (OCSB)
- net B260_TP6 renamed BHI2x_JTAG_DIO
- net B260_TP7 renamed BHI2x_JTAG_CLK
- net B260_TP9: no longer names the net of U8.29 (M1SCX)
- net BMP390_INT: no longer names the net of U8.16 (MCSB3)
- net CS renamed APP_SPI_CS
- net GPIO2/INT renamed GPIO2/INT1
- net HOST_BOOT: no longer names the net of R29.2, U8.3 (HOSTBOOT)
- net RESET: no longer names the net of U8.9 (RESETN)
- net SCK/SCL renamed APP_SPI_SCK
- net SDI/SDA renamed APP_SPI_MOSI
- net SDO renamed APP_SPI_MISO
- net VDD renamed +1V8

Commit message: 2022-09-06 1
Connections:
- net RESETN: now reaches U8.9 (RESETN)
Changed lines of the file:
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@@
     (effects (font (size 1.27 1.27)) (justify left))
+  )
+  (hierarchical_label "RESETN" (shape input) (at 81.28 71.12 180)
+    (effects (font (size 1.27 1.27)) (justify right))
   )
   (hierarchical_label "APP_SPI_MOSI" (shape input) (at 71.12 76.2 180)
