File: 04_Culturit_Tx_BHI260.kicad_sch (KiCad schematic)
At the start: 21 parts, among them U10 BMM150, U8 BHI260AP, U9 W25Q32JWZPIQ

Commit message: 2022-09-07
Connections:
- net APP_SPI_CS renamed HOST_CS
- net APP_SPI_MISO renamed HOST_MISO
- net APP_SPI_MOSI renamed HOST_MOSI
- net APP_SPI_SCK renamed HOST_SCK
- net BHI2x_JTAG_CLK: no longer names the net of U8.23 (JTAG_CLK)
- net BHI2x_JTAG_DIO: no longer names the net of U8.24 (JTAG_DIO)
- net GPIO2/INT1 renamed HIRQ
- net GPIO3/INT2 renamed MCSB4
- net RESETN renamed BNO_NRST
Changed lines of the file:
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@@
   (paper "A4")
   (title_block
-    (date "2022-08-29")
+    (date "2022-09-06")
   )
   (junction (at 38.1 66.04) (diameter 0) (color 0 0 0 0)
@@
     (stroke (width 0) (type default) (color 0 0 0 0))
   )
-  (wire (pts (xy 121.92 50.8) (xy 121.92 48.26))
-    (stroke (width 0) (type default) (color 0 0 0 0))
-  )
   (wire (pts (xy 144.78 109.22) (xy 144.78 99.06))
     (stroke (width 0) (type default) (color 0 0 0 0))
@@
     (stroke (width 0) (type default) (color 0 0 0 0))
   )
-  (wire (pts (xy 121.92 48.26) (xy 129.54 48.26))
-    (stroke (width 0) (type default) (color 0 0 0 0))
-  )
   (wire (pts (xy 119.38 88.9) (xy 137.16 88.9))
     (stroke (width 0) (type default) (color 0 0 0 0))
@@
     (stroke (width 0) (type default) (color 0 0 0 0))
   )
-  (wire (pts (xy 119.38 53.34) (xy 129.54 53.34))
-    (stroke (width 0) (type default) (color 0 0 0 0))
-  )
   (wire (pts (xy 81.28 111.76) (xy 162.56 111.76))
     (stroke (width 0) (type default) (color 0 0 0 0))
@@
   )
   (wire (pts (xy 119.38 63.5) (xy 132.08 63.5))
-    (stroke (width 0) (type default) (color 0 0 0 0))
-  )
-  (wire (pts (xy 119.38 50.8) (xy 121.92 50.8))
     (stroke (width 0) (type default) (color 0 0 0 0))
   )
@@
     (effects (font (size 1.27 1.27)) (justify left bottom))
   )
-  (hierarchical_label "GPIO3{slash}INT2" (shape input) (at 68.58 96.52 180)
+  (hierarchical_label "MCSB4" (shape input) (at 68.58 96.52 180)
     (effects (font (size 1.27 1.27)) (justify right))
   )
-  (hierarchical_label "APP_SPI_CS" (shape input) (at 119.38 78.74 0)
+  (hierarchical_label "HOST_CS" (shape input) (at 119.38 78.74 0)
     (effects (font (size 1.27 1.27)) (justify left))
   )
-  (hierarchical_label "BHI2x_JTAG_DIO" (shape input) (at 129.54 53.34 0)
+  (hierarchical_label "BNO_NRST" (shape input) (at 81.28 71.12 180)
+    (effects (font (size 1.27 1.27)) (justify right))
+  )
+  (hierarchical_label "HOST_MOSI" (shape input) (at 71.12 76.2 180)
+    (effects (font (size 1.27 1.27)) (justify right))
+  )
+  (hierarchical_label "HOST_MISO" (shape input) (at 119.38 73.66 0)
     (effects (font (size 1.27 1.27)) (justify left))
   )
-  (hierarchical_label "RESETN" (shape input) (at 81.28 71.12 180)
+  (hierarchical_label "HIRQ" (shape input) (at 71.12 73.66 180)
     (effects (font (size 1.27 1.27)) (justify right))
   )
-  (hierarchical_label "APP_SPI_MOSI" (shape input) (at 71.12 76.2 180)
-    (effects (font (size 1.27 1.27)) (justify right))
-  )
-  (hierarchical_label "BHI2x_JTAG_CLK" (shape input) (at 129.54 48.26 0)
+  (hierarchical_label "HOST_SCK" (shape input) (at 119.38 76.2 0)
     (effects (font (size 1.27 1.27)) (justify left))
   )
-  (hierarchical_label "APP_SPI_MISO" (shape input) (at 119.38 73.66 0)
-    (effects (font (size 1.27 1.27)) (justify left))
-  )
-  (hierarchical_label "GPIO2{slash}INT1" (shape input) (at 71.12 73.66 180)
-    (effects (font (size 1.27 1.27)) (justify right))
-  )
-  (hierarchical_label "APP_SPI_SCK" (shape input) (at 119.38 76.2 0)
-    (effects (font (size 1.27 1.27)) (justify left))
-  )

Commit message: 2022-09-07 2
Parts:
- renumbered R29 to R28, R30 to R29, R31 to R30, R32 to R31, R33 to R32, R34 to R33, R35 to R34, R36 to R35, R37 to R36, R38 to R37, U8 to U7, U9 to U8, U10 to U9

Commit message: 2022-09-07 3
Connections:
- net QSPI_D1: now also U8.2 (DO_(IO1))
- net QSPI_D2: now also U8.3 (~{WP_(IO2}))
Changed lines of the file:
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@@
+    (stroke (width 0) (type default) (color 0 0 0 0))
+  )
+  (wire (pts (xy 182.88 124.46) (xy 193.04 124.46))
     (stroke (width 0) (type default) (color 0 0 0 0))
   )
@@
     (stroke (width 0) (type default) (color 0 0 0 0))
   )
+  (wire (pts (xy 182.88 127) (xy 193.04 127))
+    (stroke (width 0) (type default) (color 0 0 0 0))
+  )

Commit message: 2022-10-13
Parts:
- removed C23: 100nF, Capacitor_SMD:C_0402_1005Metric, symbol Device:C
- removed U8: W25Q32JWZPIQ, Local_devices:SON127P600X500X80-9N-D, symbol W25Q32JWZPIQ:W25Q32JWZPIQ
- LED3: SKU (none) -> 304090039
Connections:
- net BNO_NRST renamed HOST_NRST
- net HIRQ renamed HOST_INT
- net MCSB4 renamed GPIO_MCSB4
