File: 01_Culturit_Tx_UsbCon.kicad_sch (KiCad schematic)
At the start: 15 parts, among them J1 USB4105-GF-A, J2 Battery

Commit message: 2022-08-08
Parts:
- added C6: 4.7uF(2012), Capacitor_SMD:C_0805_2012Metric, symbol Device:C
- added D3: LXES1UTAA1-157, Local_devices:LXES1UTAA1157, symbol LXES1UTAA1-157:LXES1UTAA1-157
- added LED2: ORANGE, LED_SMD:LED_0805_2012Metric, symbol Device:LED
- added R11: 2M, Resistor_SMD:R_0402_1005Metric, symbol Device:R
- added R12: 10k, Resistor_SMD:R_0402_1005Metric, symbol Device:R
- added R13, R8: 1M, Resistor_SMD:R_0402_1005Metric, symbol Device:R
- added R14: 300k, Resistor_SMD:R_0402_1005Metric, symbol Device:R
- added R15: 180k, Resistor_SMD:R_0402_1005Metric, symbol Device:R
- added R5: 470, Resistor_SMD:R_0402_1005Metric, symbol Device:R
- added SW1: PCM12SMTR, Local_devices:PCM12SMTR, symbol PCM12SMTR:PCM12SMTR
- added U1: MCP73832T-2ACI_MC, Local_devices:SON50P300X200X100-9N-D, symbol MCP73832T-2ACI_MC:MCP73832T-2ACI_MC
- added U2, U4: CSD25304W1015, Local_devices:BGA6C50P2X3_95X145X62, symbol CSD25304W1015:CSD25304W1015
- added U3: DMN65D8L-7, Package_TO_SOT_SMD:SOT-23, symbol Device:Q_NMOS_GSD
- C4: value 1uF -> 4.7uF(2012); footprint Capacitor_SMD:C_0603_1608Metric -> Capacitor_SMD:C_0805_2012Metric
Connections:
- net Earth: now also C4.2, C6.2, D3.2 (GND/LINE-1), R12.2, R15.2, SW1.2 (COM), U1.6 (VSS), U1.9 (EP), U3.2 (S)
- net VUSB: now also LED2.2 (A), U1.1 (VDD_1), U1.2 (VDD_2)
- net +BATT: now reaches F2.2
- net +BATT: now also C6.1, R11.2, R13.2, R8.2, U1.3 (VBAT_1), U1.4 (VBAT_2), U2.A2 (S_1), U2.B1 (S_2), U2.B2 (S_3), U4.A2 (S_1), U4.B1 (S_2), U4.B2 (S_3)
- new net: LED2.1 (K), R5.1
- new net: R5.2, U1.5 (STAT)
- new net: R14.1, U4.C1 (D_1), U4.C2 (D_2)
- new net: R12.1, U1.8 (PROG)
- new net: D3.1 (LINE-1/GND), R11.1, SW1.1 (NC), U3.1 (G)
- new net: R8.1, U2.A1 (G), U3.3 (D)
- new net VBAT_MON: R14.2, R15.1
- new net VBAT_MON_EN: R13.1, U4.A1 (G)
- new net VDRAIN: U2.C1 (D_1), U2.C2 (D_2)
Other:
- moved on the sheet: C4

Commit message: 2022-08-11 2
Parts:
- C1: MPN (none) -> CC0402KRX7R7BB104
- C2: MPN (none) -> CC0402KRX7R7BB224
- C4, C6: MPN (none) -> CC0805KKX5R8BB475
- D2: MPN (none) -> VBUS052CD-FAH-GS08
- D3: MPN (none) -> LXES1UTAA1-157
- F1: MPN (none) -> 0ZCJ0050AF2E
- F2: MPN (none) -> 0ZCJ0075FF2E
- FB1: MPN (none) -> BLM15AG700SN1D
- J1: MPN (none) -> USB4105-GF-A
- L1: MPN (none) -> DLM0QSN500HY2D
- LED2: MPN (none) -> 17-215UYC/S530-A3/TR8
- R1, R2: MPN (none) -> RC0402JR-0722RL
- R11: MPN (none) -> 0402WGF2004TCE
- R12: MPN (none) -> RC0402JR-0710KL
- R13, R8: MPN (none) -> RC0402FR-071ML
- R14: MPN (none) -> CR0402FF3003G
- R15: MPN (none) -> 0402WGJ0184TCE
- R3: MPN (none) -> RC0603FR-071ML
- R5: MPN (none) -> RC0402FR-07470RL
- SW1: MPN (none) -> PCM12SMTR
- U1: MPN (none) -> MCP73832T-2ACI/MC
- U2, U4: MPN (none) -> CSD25304W1015
- U3: MPN (none) -> DMN65D8L-7
Changed lines of the file:
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@@
+      (effects (font (size 1.27 1.27)) hide)
+    )
+    (property "MPN" "CC0805KKX5R8BB475" (id 4) (at 58.42 101.6 0)
       (effects (font (size 1.27 1.27)) hide)
     )
@@
     )
     (property "Datasheet" "https://www.vishay.com/docs/81881/vbus052c.pdf" (id 3) (at 142.24 69.85 0)
+      (effects (font (size 1.27 1.27)) hide)
+    )
+    (property "MPN" "VBUS052CD-FAH-GS08" (id 4) (at 142.24 69.85 0)
       (effects (font (size 1.27 1.27)) hide)
     )
@@
       (effects (font (size 1.27 1.27)) hide)
     )
+    (property "MPN" "RC0402FR-07470RL" (id 4) (at 100.33 97.79 0)
+      (effects (font (size 1.27 1.27)) hide)
+    )
     (pin "1")
     (pin "2")
@@
     )
     (property "Datasheet" "~" (id 3) (at 63.5 119.38 0)
+      (effects (font (size 1.27 1.27)) hide)
+    )
+    (property "MPN" "CC0805KKX5R8BB475" (id 4) (at 63.5 119.38 0)
       (effects (font (size 1.27 1.27)) hide)
     )
@@
     (property "Manufacturer_Part_Number" "DLM0QSN500HY2D" (id 9) (at 123.19 36.83 0)
       (effects (font (size 1.27 1.27)) (justify left) hide)
+    )
+    (property "MPN" "DLM0QSN500HY2D" (id 10) (at 106.68 52.07 0)
+      (effects (font (size 1.27 1.27)) hide)
     )
     (pin "1")
@@
     (property "STANDARD" "Manufacturer Recommendations" (id 7) (at 50.8 52.07 0)
       (effects (font (size 1.27 1.27)) (justify left bottom) hide)
+    )
+    (property "MPN" "USB4105-GF-A" (id 8) (at 50.8 52.07 0)
+      (effects (font (size 1.27 1.27)) hide)
     )
     (pin "A1_B12")
@@
       (effects (font (size 1.27 1.27)) (justify left) hide)
     )
+    (property "MPN" "CSD25304W1015" (id 10) (at 40.64 151.13 0)
+      (effects (font (size 1.27 1.27)) hide)
+    )
     (pin "A1")
     (pin "A2")
@@
       (effects (font (size 1.27 1.27)) hide)
     )
+    (property "MPN" "RC0402JR-0722RL" (id 4) (at 142.24 52.07 0)
+      (effects (font (size 1.27 1.27)) hide)
+    )
     (pin "1")
     (pin "2")
@@
       (effects (font (size 1.27 1.27)) hide)
     )
+    (property "MPN" "RC0402JR-0710KL" (id 4) (at 115.57 107.95 0)
+      (effects (font (size 1.27 1.27)) hide)
+    )
     (pin "1")
     (pin "2")
@@
       (effects (font (size 1.27 1.27)) hide)
     )
+    (property "MPN" "RC0402JR-0722RL" (id 4) (at 142.24 49.53 0)
+      (effects (font (size 1.27 1.27)) hide)
+    )
     (pin "1")
     (pin "2")
@@
       (effects (font (size 1.27 1.27)) (justify left) hide)
     )
+    (property "MPN" "0ZCJ0075FF2E" (id 10) (at 38.1 113.03 0)
+      (effects (font (size 1.27 1.27)) hide)
+    )
     (pin "1")
     (pin "2")
@@
     )
     (property "Datasheet" "~" (id 3) (at 140.97 144.78 0)
+      (effects (font (size 1.27 1.27)) hide)
+    )
+    (property "MPN" "DMN65D8L-7" (id 4) (at 140.97 144.78 0)
       (effects (font (size 1.27 1.27)) hide)
     )
@@
       (effects (font (size 1.27 1.27)) hide)
     )
+    (property "MPN" "17-215UYC/S530-A3/TR8" (id 4) (at 85.09 97.79 0)
+      (effects (font (size 1.27 1.27)) hide)
+    )
     (pin "1")
     (pin "2")
@@
       (effects (font (size 1.27 1.27)) hide)
     )
+    (property "MPN" "0402WGF2004TCE" (id 4) (at 129.54 125.73 0)
+      (effects (font (size 1.27 1.27)) hide)
+    )
     (pin "1")
     (pin "2")
@@
     (property "Manufacturer_Part_Number" "PCM12SMTR" (id 9) (at 96.52 173.99 0)
       (effects (font (size 1.27 1.27)) (justify left) hide)
+    )
+    (property "MPN" "PCM12SMTR" (id 10) (at 111.76 152.4 0)
+      (effects (font (size 1.27 1.27)) hide)
     )
     (pin "1")
@@
       (effects (font (size 1.27 1.27)) hide)
     )
+    (property "MPN" "RC0603FR-071ML" (id 4) (at 85.09 62.23 0)
+      (effects (font (size 1.27 1.27)) hide)
+    )
     (pin "1")
     (pin "2")
@@
       (effects (font (size 1.27 1.27)) (justify left) hide)
     )
+    (property "MPN" "BLM15AG700SN1D" (id 10) (at 129.54 27.94 0)
+      (effects (font (size 1.27 1.27)) hide)
+    )
     (pin "1")
     (pin "2")
@@
     )
     (property "Datasheet" "~" (id 3) (at 154.94 31.75 0)
+      (effects (font (size 1.27 1.27)) hide)
+    )
+    (property "MPN" "CC0402KRX7R7BB224" (id 4) (at 154.94 31.75 0)
       (effects (font (size 1.27 1.27)) hide)
     )
@@
       (effects (font (size 1.27 1.27)) hide)
     )
+    (property "MPN" "RC0402FR-071ML" (id 4) (at 50.8 134.62 0)
+      (effects (font (size 1.27 1.27)) hide)
+    )
     (pin "1")
     (pin "2")
@@
       (effects (font (size 1.27 1.27)) hide)
     )
+    (property "MPN" "CC0402KRX7R7BB104" (id 4) (at 119.38 31.75 0)
+      (effects (font (size 1.27 1.27)) hide)
+    )
     (pin "1")
     (pin "2")
@@
     (property "Manufacturer_Part_Number" "LXES1UTAA1-157" (id 9) (at 156.21 179.07 0)
       (effects (font (size 1.27 1.27)) (justify left) hide)
+    )
+    (property "MPN" "LXES1UTAA1-157" (id 10) (at 129.54 163.83 0)
+      (effects (font (size 1.27 1.27)) hide)
     )
     (pin "1")
@@
       (effects (font (size 1.27 1.27)) hide)
     )
+    (property "MPN" "0402WGJ0184TCE" (id 4) (at 71.12 170.18 0)
+      (effects (font (size 1.27 1.27)) hide)
+    )
     (pin "1")
     (pin "2")
@@
       (effects (font (size 1.27 1.27)) hide)
     )
+    (property "MPN" "RC0402FR-071ML" (id 4) (at 143.51 125.73 0)
+      (effects (font (size 1.27 1.27)) hide)
+    )
     (pin "1")
     (pin "2")
@@
       (effects (font (size 1.27 1.27)) (justify left) hide)
     )
+    (property "MPN" "0ZCJ0050AF2E" (id 10) (at 80.01 27.94 0)
+      (effects (font (size 1.27 1.27)) hide)
+    )
     (pin "1")
     (pin "2")
@@
     (property "Manufacturer_Part_Number" "CSD25304W1015" (id 9) (at 175.26 113.03 0)
       (effects (font (size 1.27 1.27)) (justify left) hide)
+    )
+    (property "MPN" "CSD25304W1015" (id 10) (at 153.67 128.27 0)
+      (effects (font (size 1.27 1.27)) hide)
     )
     (pin "A1")
@@
       (effects (font (size 1.27 1.27)) hide)
     )
+    (property "MPN" "CR0402FF3003G" (id 4) (at 71.12 157.48 0)
+      (effects (font (size 1.27 1.27)) hide)
+    )
     (pin "1")
     (pin "2")
@@
       (effects (font (size 1.27 1.27)) (justify left) hide)
     )
-    (pin "1")
+    (property "MPN" "MCP73832T-2ACI/MC" (id 10) (at 76.2 107.95 0)
+      (effects (font (size 1.27 1.27)) hide)
+    )
+    (pin "1")

Commit message: 2022-08-25
Parts:
- removed C4, C6: 4.7uF(2012), Capacitor_SMD:C_0805_2012Metric, symbol Device:C
- removed D1: SMAJ7.0A, Diode_SMD:D_SMA, symbol Device:D_Schottky
- removed D2: VBUS052CD-FAH-GS08, Local_devices:LLP1713-7L, symbol Local_devices:VBUS052CD-FAH-GS08
- removed D3: LXES1UTAA1-157, Local_devices:LXES1UTAA1157, symbol LXES1UTAA1-157:LXES1UTAA1-157
- removed F1: 0ZCJ0050AF2E, Local_devices:FUSC3216X120N, symbol 0ZCJ0050AF2E:0ZCJ0050AF2E
- removed F2: 0ZCJ0075FF2E, Local_devices:FUSC3216X120N, symbol 0ZCJ0050AF2E:0ZCJ0050AF2E
- removed FB1: BLM15AG700SN1D, Local_devices:BLM15AG700SN1D, symbol BLM15AG700SN1D:BLM15AG700SN1D
- removed J2: Battery, Connector_PinHeader_2.54mm:PinHeader_1x02_P2.54mm_Vertical, symbol Connector_Generic:Conn_01x02
- removed L1: DLM0QSN500HY2D, Local_devices:DLM0QSB120HY2D, symbol DLM0QSN500HY2D:DLM0QSN500HY2D
- removed LED2: ORANGE, LED_SMD:LED_0805_2012Metric, symbol Device:LED
- removed R11: 2M, Resistor_SMD:R_0402_1005Metric, symbol Device:R
- removed R12: 10k, Resistor_SMD:R_0402_1005Metric, symbol Device:R
- removed R13, R8: 1M, Resistor_SMD:R_0402_1005Metric, symbol Device:R
- removed R15: 180k, Resistor_SMD:R_0402_1005Metric, symbol Device:R
- removed SW1: PCM12SMTR, Local_devices:PCM12SMTR, symbol PCM12SMTR:PCM12SMTR
- removed U1: MCP73832T-2ACI_MC, Local_devices:SON50P300X200X100-9N-D, symbol MCP73832T-2ACI_MC:MCP73832T-2ACI_MC
- removed U2, U4: CSD25304W1015, Local_devices:BGA6C50P2X3_95X145X62, symbol CSD25304W1015:CSD25304W1015
- removed U3: DMN65D8L-7, Package_TO_SOT_SMD:SOT-23, symbol Device:Q_NMOS_GSD
- added C1: 10uF/1608, Capacitor_SMD:C_0603_1608Metric, symbol Device:C
- added C3: 100nF, Capacitor_SMD:C_0402_1005Metric, symbol Device:C
- added CN2: 2.54 X 2P, Connector_PinHeader_2.54mm:PinHeader_1x02_P2.54mm_Vertical, symbol Connector_Generic:Conn_01x02
- added FB1: MMZ1005Y121CT000, symbol Device:FerriteBead
- added LED1: APHHS1005SURCK, Local_devices:LEDC1005X50N, symbol APHHS1005SURCK:APHHS1005SURCK
- added R1: WFCP0402R0100FE66, Resistor_SMD:R_0402_1005Metric, symbol Device:R
- added R3, R4, R7: 10k, Resistor_SMD:R_0402_1005Metric, symbol Device:R
- added U1: MAX1555EZK+T, Local_devices:SOT95P275X110-5N, symbol MAX1555EZK+T:MAX1555EZK+T
- added U2: BQ27441DRZR-G1A, Local_devices:IC_BQ27441DRZR-G1A, symbol BQ27441DRZR-G1A:BQ27441DRZR-G1A
- C2: value 220nF, 16V -> 100nF; MPN CC0402KRX7R7BB224 -> CC0402KRX7R7BB104; SKU (none) -> 302010004
- C31: renamed from C1; value 100nF, 16V -> 10nF; MPN CC0402KRX7R7BB104 -> CC0402KRX7R9BB103; SKU (none) -> 302010006
- R13: renamed from R1; MPN RC0402JR-0722RL -> RC0402FR-0722RL; SKU (none) -> 301010052
- R14: value 300k -> 22; MPN CR0402FF3003G -> RC0402FR-0722RL; SKU (none) -> 301010052
- R2: value 22 -> 330; MPN RC0402JR-0722RL -> RC0402FR-07330RL; SKU (none) -> 301010466
- R5: value 470 -> 10k; MPN RC0402FR-07470RL -> RC0402JR-0710KL
- renumbered C3 to C4, R3 to R6
Connections:
- net D+ is gone; now on net DP: R13.1
- net VBAT_MON is gone; now on net USB_DN: R14.2
- net DN: now also R14.1
- net Earth: now also R2.2, C1.2, C3.1, CN2.2 (Pin_2), R7.1, U1.2 (GND), U2.13 (EXP), U2.14 (EXP), U2.15 (EXP), U2.16 (EXP), U2.17 (EXP), U2.18 (EXP), U2.19 (EXP), U2.3 (VSS)
- net USB_DN: no longer R2.2
- net GPOUT: now reaches R5.1
- net GPOUT: now also U2.12 (GPOUT)
- net VDD_nRF: now reaches R5.2
- net VDD_nRF: now also R3.2, R4.2
- net at J1.A4_B9 (VBUS), J1.B4_A9 (VBUS): now also C31.1, FB1.2
- net D-: no longer names the net of R2.1
- net D-: now also LED1.1
- net VUSB renamed VBUS
- net VBUS: now also FB1.1, U1.1 (USB)
- new net: C1.1, CN2.1 (Pin_1), R1.2, U2.6 (BAT), U2.8 (SRP)
- new net: C3.2, U2.5 (VDD)
- new net: LED1.2, U1.3 (~{POK(}CHG))
- new net BATT_SCL: R4.1, U2.2 (SCL)
- new net BATT_SDA: R3.1, U2.1 (SDA)
- new net BIN: R7.2, U2.10 (BIN)
- new net VSYS: R1.1, U1.5 (BAT), U2.7 (SRN)
- no-connect marks 0 -> 1
Other:
- moved on the sheet: C2, C31, R13

Commit message: 2022-08-26
Parts:
- renumbered C4 to C1, C31 to C2, C2 to C3, C3 to C4, C1 to C5, CN2 to CN1, R6 to R1, R13 to R2, R14 to R3, R2 to R4, R1 to R6, R3 to R8, R4 to R9
Other:
- moved on the sheet: C1, C2, C3, C4, C5, CN1, FB1, J1, LED1, R1, R2, R3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

Commit message: 2022-08-29
Parts:
- renumbered J1 to J2
Changed lines of the file:
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@@
   (paper "A4")
   (title_block
-    (date "2022-08-16")
+    (date "2022-08-26")
   )
   (junction (at 245.11 100.33) (diameter 0) (color 0 0 0 0)
@@
   (symbol (lib_id "power:Earth") (at 135.89 120.65 0) (unit 1)
     (in_bom yes) (on_board yes) (fields_autoplaced)
-    (property "Reference" "#PWR07" (id 0) (at 135.89 127 0)
+    (property "Reference" "#PWR09" (id 0) (at 135.89 127 0)
       (effects (font (size 1.27 1.27)) hide)
     )
@@
   (symbol (lib_id "power:Earth") (at 135.89 92.71 270) (unit 1)
     (in_bom yes) (on_board yes) (fields_autoplaced)
-    (property "Reference" "#PWR06" (id 0) (at 129.54 92.71 0)
+    (property "Reference" "#PWR08" (id 0) (at 129.54 92.71 0)
       (effects (font (size 1.27 1.27)) hide)
     )
@@
   (symbol (lib_id "power:GNDPWR") (at 72.39 115.57 0) (unit 1)
     (in_bom yes) (on_board yes) (fields_autoplaced)
-    (property "Reference" "#PWR01" (id 0) (at 72.39 120.65 0)
+    (property "Reference" "#PWR03" (id 0) (at 72.39 120.65 0)
       (effects (font (size 1.27 1.27)) hide)
     )
@@
   (symbol (lib_id "power:Earth") (at 261.62 72.39 0) (unit 1)
     (in_bom yes) (on_board yes) (fields_autoplaced)
-    (property "Reference" "#PWR011" (id 0) (at 261.62 78.74 0)
+    (property "Reference" "#PWR013" (id 0) (at 261.62 78.74 0)
       (effects (font (size 1.27 1.27)) hide)
     )
@@
   (symbol (lib_id "power:Earth") (at 240.03 82.55 0) (unit 1)
     (in_bom yes) (on_board yes) (fields_autoplaced)
-    (property "Reference" "#PWR09" (id 0) (at 240.03 88.9 0)
+    (property "Reference" "#PWR011" (id 0) (at 240.03 88.9 0)
       (effects (font (size 1.27 1.27)) hide)
     )
@@
   (symbol (lib_id "USB4105-GF-A:USB4105-GF-A") (at 49.53 93.98 0) (unit 1)
     (in_bom yes) (on_board yes) (fields_autoplaced)
-    (property "Reference" "J1" (id 0) (at 49.53 76.2 0))
+    (property "Reference" "J2" (id 0) (at 49.53 76.2 0))
     (property "Value" "USB4105-GF-A" (id 1) (at 49.53 78.74 0))
     (property "Footprint" "Local_devices:GCT_USB4105-GF-A" (id 2) (at 49.53 93.98 0)
@@
   (symbol (lib_id "power:Earth") (at 186.69 123.19 0) (unit 1)
     (in_bom yes) (on_board yes) (fields_autoplaced)
-    (property "Reference" "#PWR08" (id 0) (at 186.69 129.54 0)
+    (property "Reference" "#PWR010" (id 0) (at 186.69 129.54 0)
       (effects (font (size 1.27 1.27)) hide)
     )
@@
   (symbol (lib_id "power:VBUS") (at 135.89 67.31 0) (unit 1)
     (in_bom yes) (on_board yes) (fields_autoplaced)
-    (property "Reference" "#PWR05" (id 0) (at 135.89 71.12 0)
+    (property "Reference" "#PWR07" (id 0) (at 135.89 71.12 0)
       (effects (font (size 1.27 1.27)) hide)
     )
@@
   (symbol (lib_id "power:Earth") (at 95.25 115.57 0) (unit 1)
     (in_bom yes) (on_board yes) (fields_autoplaced)
-    (property "Reference" "#PWR02" (id 0) (at 95.25 121.92 0)
+    (property "Reference" "#PWR04" (id 0) (at 95.25 121.92 0)
       (effects (font (size 1.27 1.27)) hide)
     )
@@
   (symbol (lib_id "power:Earth") (at 245.11 115.57 0) (unit 1)
     (in_bom yes) (on_board yes) (fields_autoplaced)
-    (property "Reference" "#PWR010" (id 0) (at 245.11 121.92 0)
+    (property "Reference" "#PWR012" (id 0) (at 245.11 121.92 0)
       (effects (font (size 1.27 1.27)) hide)
     )
@@
   (symbol (lib_id "power:Earth") (at 123.19 77.47 0) (unit 1)
     (in_bom yes) (on_board yes) (fields_autoplaced)
-    (property "Reference" "#PWR04" (id 0) (at 123.19 83.82 0)
+    (property "Reference" "#PWR06" (id 0) (at 123.19 83.82 0)
       (effects (font (size 1.27 1.27)) hide)
     )
@@
   (symbol (lib_id "power:Earth") (at 100.33 77.47 0) (unit 1)
     (in_bom yes) (on_board yes) (fields_autoplaced)
-    (property "Reference" "#PWR03" (id 0) (at 100.33 83.82 0)
-      (effects (font (size 1.27 1.27)) hide)
-    )
+    (property "Reference" "#PWR05" (id 0) (at 100.33 83.82 0)
+      (effects (font (size 1.27 1.27)) hide)
+    )
