File: 01_Culturit_Tx_UsbCon.kicad_sch (KiCad schematic)
At the start: 20 parts, among them CN1 2.54 X 2P, J2 USB4105-GF-A, U1 MAX1555EZK+T, U2 BQ27441DRZR-G1A

Commit message: 2022-09-07 3
Parts:
- LED1: footprint Local_devices:LEDC1005X50N -> LED_SMD:LED_0402_1005Metric
Connections:
- net VDD_nRF renamed +1V8
Changed lines of the file:
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@@
     (effects (font (size 1.27 1.27)) (justify left bottom))
-  )
-  (global_label "VDD_nRF" (shape input) (at 252.73 90.17 0) (fields_autoplaced)
-    (effects (font (size 1.27 1.27)) (justify left))
-    (property "Intersheet References" "${INTERSHEET_REFS}" (id 0) (at 263.2469 90.0906 0)
-      (effects (font (size 1.27 1.27)) (justify left) hide)
-    )
   )
   (global_label "VSYS" (shape input) (at 176.53 69.85 180) (fields_autoplaced)
@@
     )
   )
-  (global_label "VDD_nRF" (shape input) (at 184.15 85.09 0) (fields_autoplaced)
-    (effects (font (size 1.27 1.27)) (justify left))
-    (property "Intersheet References" "${INTERSHEET_REFS}" (id 0) (at 194.6669 85.0106 0)
-      (effects (font (size 1.27 1.27)) (justify left) hide)
-    )
-  )
   (hierarchical_label "BIN" (shape input) (at 252.73 100.33 0)
     (effects (font (size 1.27 1.27)) (justify left))
@@
   (hierarchical_label "GPOUT" (shape input) (at 184.15 97.79 180)
     (effects (font (size 1.27 1.27)) (justify right))
+  )
+  (symbol (lib_id "power:+1V8") (at 252.73 90.17 270) (unit 1)
+    (in_bom yes) (on_board yes) (fields_autoplaced)
+    (property "Reference" "#PWR?" (id 0) (at 248.92 90.17 0)
+      (effects (font (size 1.27 1.27)) hide)
+    )
+    (property "Value" "+1V8" (id 1) (at 256.54 90.1699 90)
+      (effects (font (size 1.27 1.27)) (justify left))
+    )
+    (property "Footprint" "" (id 2) (at 252.73 90.17 0)
+      (effects (font (size 1.27 1.27)) hide)
+    )
+    (property "Datasheet" "" (id 3) (at 252.73 90.17 0)
+      (effects (font (size 1.27 1.27)) hide)
+    )
+    (pin "1")
   )
   (symbol (lib_id "power:Earth") (at 135.89 120.65 0) (unit 1)
@@
     (pin "2")
   )
+  (symbol (lib_id "power:+1V8") (at 184.15 85.09 0) (unit 1)
+    (in_bom yes) (on_board yes) (fields_autoplaced)
+    (property "Reference" "#PWR?" (id 0) (at 184.15 88.9 0)
+      (effects (font (size 1.27 1.27)) hide)
+    )
+    (property "Value" "+1V8" (id 1) (at 184.15 80.01 0))
+    (property "Footprint" "" (id 2) (at 184.15 85.09 0)
+      (effects (font (size 1.27 1.27)) hide)
+    )
+    (property "Datasheet" "" (id 3) (at 184.15 85.09 0)
+      (effects (font (size 1.27 1.27)) hide)
+    )
+    (pin "1")
+  )
   (symbol (lib_id "power:VBUS") (at 135.89 67.31 0) (unit 1)
     (in_bom yes) (on_board yes) (fields_autoplaced)
@@
       (effects (font (size 1.27 1.27)) (justify right))
     )
-    (property "Footprint" "Local_devices:LEDC1005X50N" (id 2) (at 132.08 100.33 0)
-      (effects (font (size 1.27 1.27)) (justify left bottom) hide)
-    )
+    (property "Footprint" "LED_SMD:LED_0402_1005Metric" (id 2) (at 132.08 100.33 0)
+      (effects (font (size 1.27 1.27)) (justify left bottom) hide)
+    )

Commit message: 2022-09-14
Parts:
- FB1: footprint (none) -> Inductor_SMD:L_0402_1005Metric
Changed lines of the file:
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@@
   (symbol (lib_id "power:+1V8") (at 252.73 90.17 270) (unit 1)
     (in_bom yes) (on_board yes) (fields_autoplaced)
-    (property "Reference" "#PWR?" (id 0) (at 248.92 90.17 0)
+    (property "Reference" "#PWR0101" (id 0) (at 248.92 90.17 0)
       (effects (font (size 1.27 1.27)) hide)
     )
@@
     (property "Reference" "FB1" (id 0) (at 114.3508 62.23 90))
     (property "Value" "MMZ1005Y121CT000" (id 1) (at 114.3508 64.77 90))
-    (property "Footprint" "" (id 2) (at 114.3 68.072 90)
+    (property "Footprint" "Inductor_SMD:L_0402_1005Metric" (id 2) (at 114.3 68.072 90)
       (effects (font (size 1.27 1.27)) hide)
     )
@@
   (symbol (lib_id "power:+1V8") (at 184.15 85.09 0) (unit 1)
     (in_bom yes) (on_board yes) (fields_autoplaced)
-    (property "Reference" "#PWR?" (id 0) (at 184.15 88.9 0)
-      (effects (font (size 1.27 1.27)) hide)
-    )
+    (property "Reference" "#PWR0102" (id 0) (at 184.15 88.9 0)
+      (effects (font (size 1.27 1.27)) hide)
+    )
