File: 01_Culturit_Tx_UsbCon.kicad_sch (KiCad schematic)
At the start: 20 parts, among them CN1 2.54 X 2P, J2 USB4105-GF-A, U1 MAX1555EZK+T, U2 BQ27441DRZR-G1A

Commit message: 2022-09-07
Parts:
- C1: value 1nF(1812),X7R,2kV -> 4.7nF/1608; footprint Capacitor_SMD:C_1812_4532Metric -> Capacitor_SMD:C_0603_1608Metric; MPN C1812C102KGRACAUTO -> CC0603KRX7R9BB472
- FB1: footprint (none) -> Inductor_SMD:L_0402_1005Metric
- LED1: footprint Local_devices:LEDC1005X50N -> LED_SMD:LED_0402_1005Metric
Connections:
- net Earth: no longer R4.2
- net VBUS: now also R4.2
- net VDD_nRF renamed +1V8
Changed lines of the file:
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@@
     (effects (font (size 1.27 1.27)) (justify left bottom))
-  )
-  (global_label "VDD_nRF" (shape input) (at 252.73 90.17 0) (fields_autoplaced)
-    (effects (font (size 1.27 1.27)) (justify left))
-    (property "Intersheet References" "${INTERSHEET_REFS}" (id 0) (at 263.2469 90.0906 0)
-      (effects (font (size 1.27 1.27)) (justify left) hide)
-    )
   )
   (global_label "VSYS" (shape input) (at 176.53 69.85 180) (fields_autoplaced)
@@
     )
   )
-  (global_label "VDD_nRF" (shape input) (at 184.15 85.09 0) (fields_autoplaced)
-    (effects (font (size 1.27 1.27)) (justify left))
-    (property "Intersheet References" "${INTERSHEET_REFS}" (id 0) (at 194.6669 85.0106 0)
-      (effects (font (size 1.27 1.27)) (justify left) hide)
-    )
-  )
   (hierarchical_label "BIN" (shape input) (at 252.73 100.33 0)
     (effects (font (size 1.27 1.27)) (justify left))
@@
   (hierarchical_label "GPOUT" (shape input) (at 184.15 97.79 180)
     (effects (font (size 1.27 1.27)) (justify right))
-  )
-  (symbol (lib_id "power:Earth") (at 135.89 120.65 0) (unit 1)
-    (in_bom yes) (on_board yes) (fields_autoplaced)
-    (property "Reference" "#PWR09" (id 0) (at 135.89 127 0)
-      (effects (font (size 1.27 1.27)) hide)
-    )
-    (property "Value" "Earth" (id 1) (at 135.89 124.46 0)
-      (effects (font (size 1.27 1.27)) hide)
-    )
-    (property "Footprint" "" (id 2) (at 135.89 120.65 0)
-      (effects (font (size 1.27 1.27)) hide)
-    )
-    (property "Datasheet" "~" (id 3) (at 135.89 120.65 0)
-      (effects (font (size 1.27 1.27)) hide)
-    )
-    (pin "1")
   )
   (symbol (lib_id "Device:R") (at 231.14 69.85 90) (unit 1)
@@
     (property "Reference" "FB1" (id 0) (at 114.3508 62.23 90))
     (property "Value" "MMZ1005Y121CT000" (id 1) (at 114.3508 64.77 90))
-    (property "Footprint" "" (id 2) (at 114.3 68.072 90)
+    (property "Footprint" "Inductor_SMD:L_0402_1005Metric" (id 2) (at 114.3 68.072 90)
       (effects (font (size 1.27 1.27)) hide)
     )
@@
     )
     (property "Datasheet" "~" (id 3) (at 240.03 82.55 0)
+      (effects (font (size 1.27 1.27)) hide)
+    )
+    (pin "1")
+  )
+  (symbol (lib_id "power:VBUS") (at 135.89 120.65 180) (unit 1)
+    (in_bom yes) (on_board yes) (fields_autoplaced)
+    (property "Reference" "#PWR0101" (id 0) (at 135.89 116.84 0)
+      (effects (font (size 1.27 1.27)) hide)
+    )
+    (property "Value" "VBUS" (id 1) (at 138.43 121.9199 0)
+      (effects (font (size 1.27 1.27)) (justify right))
+    )
+    (property "Footprint" "" (id 2) (at 135.89 120.65 0)
+      (effects (font (size 1.27 1.27)) hide)
+    )
+    (property "Datasheet" "" (id 3) (at 135.89 120.65 0)
       (effects (font (size 1.27 1.27)) hide)
     )
@@
     (in_bom yes) (on_board yes)
     (property "Reference" "C1" (id 0) (at 77.47 109.22 90))
-    (property "Value" "1nF(1812),X7R,2kV" (id 1) (at 83.82 114.3 90))
-    (property "Footprint" "Capacitor_SMD:C_1812_4532Metric" (id 2) (at 87.63 109.5248 0)
-      (effects (font (size 1.27 1.27)) hide)
-    )
-    (property "Datasheet" "https://www.mouser.kr/datasheet/2/212/1/KEM_C1076_X7R_HV_AUTO_SMD-1093301.pdf" (id 3) (at 83.82 110.49 0)
-      (effects (font (size 1.27 1.27)) hide)
-    )
-    (property "MPN" "C1812C102KGRACAUTO" (id 4) (at 83.82 110.49 90)
+    (property "Value" "4.7nF/1608" (id 1) (at 83.82 114.3 90))
+    (property "Footprint" "Capacitor_SMD:C_0603_1608Metric" (id 2) (at 87.63 109.5248 0)
+      (effects (font (size 1.27 1.27)) hide)
+    )
+    (property "Datasheet" "" (id 3) (at 83.82 110.49 0)
+      (effects (font (size 1.27 1.27)) hide)
+    )
+    (property "MPN" "CC0603KRX7R9BB472" (id 4) (at 83.82 110.49 90)
       (effects (font (size 1.27 1.27)) hide)
     )
@@
     (pin "2")
   )
+  (symbol (lib_id "power:+1V8") (at 184.15 85.09 0) (unit 1)
+    (in_bom yes) (on_board yes) (fields_autoplaced)
+    (property "Reference" "#PWR0103" (id 0) (at 184.15 88.9 0)
+      (effects (font (size 1.27 1.27)) hide)
+    )
+    (property "Value" "+1V8" (id 1) (at 184.15 80.01 0))
+    (property "Footprint" "" (id 2) (at 184.15 85.09 0)
+      (effects (font (size 1.27 1.27)) hide)
+    )
+    (property "Datasheet" "" (id 3) (at 184.15 85.09 0)
+      (effects (font (size 1.27 1.27)) hide)
+    )
+    (pin "1")
+  )
   (symbol (lib_id "Connector_Generic:Conn_01x02") (at 266.7 69.85 0) (unit 1)
     (in_bom yes) (on_board yes) (fields_autoplaced)
@@
       (effects (font (size 1.27 1.27)) (justify right))
     )
-    (property "Footprint" "Local_devices:LEDC1005X50N" (id 2) (at 132.08 100.33 0)
+    (property "Footprint" "LED_SMD:LED_0402_1005Metric" (id 2) (at 132.08 100.33 0)
       (effects (font (size 1.27 1.27)) (justify left bottom) hide)
     )
@@
     (pin "2")
   )
+  (symbol (lib_id "power:+1V8") (at 252.73 90.17 270) (unit 1)
+    (in_bom yes) (on_board yes) (fields_autoplaced)
+    (property "Reference" "#PWR0102" (id 0) (at 248.92 90.17 0)
+      (effects (font (size 1.27 1.27)) hide)
+    )
+    (property "Value" "+1V8" (id 1) (at 256.54 90.1699 90)
+      (effects (font (size 1.27 1.27)) (justify left))
+    )
+    (property "Footprint" "" (id 2) (at 252.73 90.17 0)
+      (effects (font (size 1.27 1.27)) hide)
+    )
+    (property "Datasheet" "" (id 3) (at 252.73 90.17 0)
+      (effects (font (size 1.27 1.27)) hide)
+    )
+    (pin "1")
+  )
   (symbol (lib_id "Device:R") (at 250.19 93.98 180) (unit 1)

Commit message: 2022-11-01
Parts:
- removed J2: USB4105-GF-A, Local_devices:GCT_USB4105-GF-A, symbol USB4105-GF-A:USB4105-GF-A
- added J2: USB4110-GF-A, Local_devices:USB4110GFA, symbol USB4110-GF-A:USB4110-GF-A
Connections:
- net DN: now also J2.A7, J2.B7
- net DP: now also J2.A6, J2.B6
- net Earth: now also J2.A1, J2.A12, J2.B1, J2.B12
- net GNDPWR: now also J2.MP1, J2.MP2, J2.MP3, J2.MP4
- net VUSB: now reaches C2.1, FB1.2
- net VUSB: now also J2.A4, J2.A9, J2.B4, J2.B9
