File: bno085.kicad_sch (KiCad schematic)
At the start: 9 parts, among them U8 BNO055

Commit message: 2022-09-07
Parts:
- removed C17, C19: 10nF, Capacitor_SMD:C_0402_1005Metric, symbol Device:C
- removed C18: 100nF, Capacitor_SMD:C_0402_1005Metric, symbol Device:C
- removed L2: BLM15AG121SN1D, Inductor_SMD:L_0402_1005Metric, symbol Device:L_Ferrite
- renumbered R29 to R28, R30 to R29, R31 to R30, U8 to U7
Changed lines of the file:
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@@
   (junction (at 110.49 93.98) (diameter 0) (color 0 0 0 0)
   )
-  (junction (at 50.8 63.5) (diameter 0) (color 0 0 0 0)
-  )
   (junction (at 106.68 88.9) (diameter 0) (color 0 0 0 0)
   )
@@
   )
   (junction (at 138.43 76.2) (diameter 0) (color 0 0 0 0)
-  )
-  (junction (at 86.36 63.5) (diameter 0) (color 0 0 0 0)
-  )
-  (junction (at 76.2 63.5) (diameter 0) (color 0 0 0 0)
   )
   (no_connect (at 156.21 83.82))
@@
     (stroke (width 0) (type default) (color 0 0 0 0))
   )
-  (wire (pts (xy 50.8 63.5) (xy 59.69 63.5))
-    (stroke (width 0) (type default) (color 0 0 0 0))
-  )
-  (wire (pts (xy 76.2 63.5) (xy 86.36 63.5))
-    (stroke (width 0) (type default) (color 0 0 0 0))
-  )
   (wire (pts (xy 110.49 93.98) (xy 125.73 93.98))
     (stroke (width 0) (type default) (color 0 0 0 0))
@@
     (stroke (width 0) (type default) (color 0 0 0 0))
   )
-  (wire (pts (xy 86.36 60.96) (xy 86.36 63.5))
-    (stroke (width 0) (type default) (color 0 0 0 0))
-  )
   (wire (pts (xy 110.49 86.36) (xy 110.49 93.98))
     (stroke (width 0) (type default) (color 0 0 0 0))
@@
     (stroke (width 0) (type default) (color 0 0 0 0))
   )
-  (wire (pts (xy 67.31 63.5) (xy 76.2 63.5))
-    (stroke (width 0) (type default) (color 0 0 0 0))
-  )
   (wire (pts (xy 138.43 73.66) (xy 138.43 76.2))
     (stroke (width 0) (type default) (color 0 0 0 0))
@@
   (wire (pts (xy 110.49 76.2) (xy 110.49 78.74))
     (stroke (width 0) (type default) (color 0 0 0 0))
-  )
-  (global_label "VDD_BNO" (shape input) (at 86.36 60.96 0) (fields_autoplaced)
-    (effects (font (size 1.27 1.27)) (justify left))
-    (property "Intersheet References" "${INTERSHEET_REFS}" (id 0) (at 97.3002 60.8806 0)
-      (effects (font (size 1.27 1.27)) (justify left) hide)
-    )
   )
   (global_label "VDD_BNO" (shape input) (at 138.43 73.66 90) (fields_autoplaced)
@@
     (effects (font (size 1.27 1.27)) (justify right))
   )
-  (symbol (lib_id "power:+3V3") (at 50.8 63.5 0) (unit 1)
-    (in_bom yes) (on_board yes) (fields_autoplaced)
-    (property "Reference" "#PWR049" (id 0) (at 50.8 67.31 0)
-      (effects (font (size 1.27 1.27)) hide)
-    )
-    (property "Value" "+3V3" (id 1) (at 50.8 58.42 0))
-    (property "Footprint" "" (id 2) (at 50.8 63.5 0)
-      (effects (font (size 1.27 1.27)) hide)
-    )
-    (property "Datasheet" "" (id 3) (at 50.8 63.5 0)
-      (effects (font (size 1.27 1.27)) hide)
-    )
-    (pin "1")
-  )
   (symbol (lib_id "Sensor_Motion:BNO055") (at 140.97 96.52 0) (unit 1)
     (in_bom yes) (on_board yes) (fields_autoplaced)
-    (property "Reference" "U8" (id 0) (at 145.5294 76.2 0)
+    (property "Reference" "U7" (id 0) (at 145.5294 76.2 0)
       (effects (font (size 1.27 1.27)) (justify left))
     )
@@
   (symbol (lib_id "Device:R") (at 163.83 97.79 0) (unit 1)
     (in_bom yes) (on_board yes)
-    (property "Reference" "R31" (id 0) (at 162.56 95.25 90)
+    (property "Reference" "R30" (id 0) (at 162.56 95.25 90)
       (effects (font (size 1.27 1.27)) (justify left))
     )
@@
   (symbol (lib_id "power:Earth") (at 143.51 114.3 0) (unit 1)
     (in_bom yes) (on_board yes) (fields_autoplaced)
-    (property "Reference" "#PWR055" (id 0) (at 143.51 120.65 0)
+    (property "Reference" "#PWR053" (id 0) (at 143.51 120.65 0)
       (effects (font (size 1.27 1.27)) hide)
     )
@@
   (symbol (lib_id "power:Earth") (at 158.75 119.38 0) (unit 1)
     (in_bom yes) (on_board yes) (fields_autoplaced)
-    (property "Reference" "#PWR056" (id 0) (at 158.75 125.73 0)
+    (property "Reference" "#PWR054" (id 0) (at 158.75 125.73 0)
       (effects (font (size 1.27 1.27)) hide)
     )
@@
     (pin "1")
   )
-  (symbol (lib_id "power:Earth") (at 50.8 71.12 0) (unit 1)
-    (in_bom yes) (on_board yes) (fields_autoplaced)
-    (property "Reference" "#PWR050" (id 0) (at 50.8 77.47 0)
-      (effects (font (size 1.27 1.27)) hide)
-    )
-    (property "Value" "Earth" (id 1) (at 50.8 74.93 0)
-      (effects (font (size 1.27 1.27)) hide)
-    )
-    (property "Footprint" "" (id 2) (at 50.8 71.12 0)
-      (effects (font (size 1.27 1.27)) hide)
-    )
-    (property "Datasheet" "~" (id 3) (at 50.8 71.12 0)
-      (effects (font (size 1.27 1.27)) hide)
-    )
-    (pin "1")
-  )
-  (symbol (lib_id "power:Earth") (at 76.2 71.12 0) (unit 1)
-    (in_bom yes) (on_board yes) (fields_autoplaced)
-    (property "Reference" "#PWR051" (id 0) (at 76.2 77.47 0)
-      (effects (font (size 1.27 1.27)) hide)
-    )
-    (property "Value" "Earth" (id 1) (at 76.2 74.93 0)
-      (effects (font (size 1.27 1.27)) hide)
-    )
-    (property "Footprint" "" (id 2) (at 76.2 71.12 0)
-      (effects (font (size 1.27 1.27)) hide)
-    )
-    (property "Datasheet" "~" (id 3) (at 76.2 71.12 0)
-      (effects (font (size 1.27 1.27)) hide)
-    )
-    (pin "1")
-  )
   (symbol (lib_id "power:+3V3") (at 163.83 91.44 0) (unit 1)
     (in_bom yes) (on_board yes) (fields_autoplaced)
-    (property "Reference" "#PWR057" (id 0) (at 163.83 95.25 0)
+    (property "Reference" "#PWR055" (id 0) (at 163.83 95.25 0)
       (effects (font (size 1.27 1.27)) hide)
     )
@@
   (symbol (lib_id "power:+3V3") (at 106.68 76.2 0) (unit 1)
     (in_bom yes) (on_board yes) (fields_autoplaced)
-    (property "Reference" "#PWR053" (id 0) (at 106.68 80.01 0)
+    (property "Reference" "#PWR051" (id 0) (at 106.68 80.01 0)
       (effects (font (size 1.27 1.27)) hide)
     )
@@
   (symbol (lib_id "Device:R") (at 110.49 82.55 0) (unit 1)
     (in_bom yes) (on_board yes)
-    (property "Reference" "R30" (id 0) (at 109.22 80.01 90)
+    (property "Reference" "R29" (id 0) (at 109.22 80.01 90)
       (effects (font (size 1.27 1.27)) (justify left))
     )
@@
     (pin "2")
   )
-  (symbol (lib_id "Device:C") (at 50.8 67.31 0) (unit 1)
-    (in_bom yes) (on_board yes) (fields_autoplaced)
-    (property "Reference" "C17" (id 0) (at 54.61 66.0399 0)
-      (effects (font (size 1.27 1.27)) (justify left))
-    )
-    (property "Value" "10nF" (id 1) (at 54.61 68.5799 0)
-      (effects (font (size 1.27 1.27)) (justify left))
-    )
-    (property "Footprint" "Capacitor_SMD:C_0402_1005Metric" (id 2) (at 51.7652 71.12 0)
-      (effects (font (size 1.27 1.27)) hide)
-    )
-    (property "Datasheet" "~" (id 3) (at 50.8 67.31 0)
-      (effects (font (size 1.27 1.27)) hide)
-    )
-    (property "MPN" "CC0402KRX7R9BB103" (id 4) (at 50.8 67.31 0)
-      (effects (font (size 1.27 1.27)) hide)
-    )
-    (pin "1")
-    (pin "2")
-  )
-  (symbol (lib_id "power:Earth") (at 86.36 71.12 0) (unit 1)
-    (in_bom yes) (on_board yes) (fields_autoplaced)
-    (property "Reference" "#PWR052" (id 0) (at 86.36 77.47 0)
-      (effects (font (size 1.27 1.27)) hide)
-    )
-    (property "Value" "Earth" (id 1) (at 86.36 74.93 0)
-      (effects (font (size 1.27 1.27)) hide)
-    )
-    (property "Footprint" "" (id 2) (at 86.36 71.12 0)
-      (effects (font (size 1.27 1.27)) hide)
-    )
-    (property "Datasheet" "~" (id 3) (at 86.36 71.12 0)
-      (effects (font (size 1.27 1.27)) hide)
-    )
-    (pin "1")
-  )
   (symbol (lib_id "power:Earth") (at 138.43 114.3 0) (unit 1)
     (in_bom yes) (on_board yes) (fields_autoplaced)
-    (property "Reference" "#PWR054" (id 0) (at 138.43 120.65 0)
+    (property "Reference" "#PWR052" (id 0) (at 138.43 120.65 0)
       (effects (font (size 1.27 1.27)) hide)
     )
@@
     (pin "1")
   )
-  (symbol (lib_id "Device:L_Ferrite") (at 63.5 63.5 90) (unit 1)
-    (in_bom yes) (on_board yes) (fields_autoplaced)
-    (property "Reference" "L2" (id 0) (at 63.5 57.15 90))
-    (property "Value" "BLM15AG121SN1D" (id 1) (at 63.5 59.69 90))
-    (property "Footprint" "Inductor_SMD:L_0402_1005Metric" (id 2) (at 63.5 63.5 0)
-      (effects (font (size 1.27 1.27)) hide)
-    )
-    (property "Datasheet" "~" (id 3) (at 63.5 63.5 0)
-      (effects (font (size 1.27 1.27)) hide)
-    )
-    (property "MPN" "BLM15AG121SN1D" (id 4) (at 63.5 63.5 90)
-      (effects (font (size 1.27 1.27)) hide)
-    )
-    (pin "1")
-    (pin "2")
-  )
-  (symbol (lib_id "Device:C") (at 76.2 67.31 0) (unit 1)
-    (in_bom yes) (on_board yes)
-    (property "Reference" "C18" (id 0) (at 77.47 64.77 0)
-      (effects (font (size 1.27 1.27)) (justify left))
-    )
-    (property "Value" "100nF" (id 1) (at 69.85 69.85 0)
-      (effects (font (size 1.27 1.27)) (justify left))
-    )
-    (property "Footprint" "Capacitor_SMD:C_0402_1005Metric" (id 2) (at 77.1652 71.12 0)
-      (effects (font (size 1.27 1.27)) hide)
-    )
-    (property "Datasheet" "~" (id 3) (at 76.2 67.31 0)
-      (effects (font (size 1.27 1.27)) hide)
-    )
-    (property "MPN" "CC0402KRX7R7BB104" (id 4) (at 76.2 67.31 0)
-      (effects (font (size 1.27 1.27)) hide)
-    )
-    (pin "1")
-    (pin "2")
-  )
-  (symbol (lib_id "Device:C") (at 86.36 67.31 0) (unit 1)
-    (in_bom yes) (on_board yes) (fields_autoplaced)
-    (property "Reference" "C19" (id 0) (at 90.17 66.0399 0)
-      (effects (font (size 1.27 1.27)) (justify left))
-    )
-    (property "Value" "10nF" (id 1) (at 90.17 68.5799 0)
-      (effects (font (size 1.27 1.27)) (justify left))
-    )
-    (property "Footprint" "Capacitor_SMD:C_0402_1005Metric" (id 2) (at 87.3252 71.12 0)
-      (effects (font (size 1.27 1.27)) hide)
-    )
-    (property "Datasheet" "~" (id 3) (at 86.36 67.31 0)
-      (effects (font (size 1.27 1.27)) hide)
-    )
-    (property "MPN" "CC0402KRX7R9BB103" (id 4) (at 86.36 67.31 0)
-      (effects (font (size 1.27 1.27)) hide)
-    )
-    (pin "1")
-    (pin "2")
-  )
   (symbol (lib_id "Device:C") (at 158.75 115.57 0) (unit 1)
     (in_bom yes) (on_board yes)
@@
   (symbol (lib_id "Device:R") (at 106.68 82.55 0) (unit 1)
     (in_bom yes) (on_board yes)
-    (property "Reference" "R29" (id 0) (at 105.41 80.01 90)
-      (effects (font (size 1.27 1.27)) (justify left))
-    )
+    (property "Reference" "R28" (id 0) (at 105.41 80.01 90)
+      (effects (font (size 1.27 1.27)) (justify left))
+    )
