File: culturit_tx.kicad_pcb (KiCad board)
At the start: 4 copper layers, 50 x 50 mm, 14 parts, among them J1 USB4105-GF-A, U13 MDBT50Q-1M, U15 BHI260AP

Commit message: 2022-08-08
Parts:
- added C10: 2.2uF(2012), Capacitor_SMD:C_0805_2012Metric, F.Cu at (44.5, 42.0)
- added C12: 4.7uF(2012), Capacitor_SMD:C_0805_2012Metric, F.Cu at (52.0, 38.0)
- added C13: 120pF, Capacitor_SMD:C_0402_1005Metric, F.Cu at (59.0, 45.5)
- added C14: 10uF(2012), Capacitor_SMD:C_0805_2012Metric, F.Cu at (59.0, 43.5)
- added C15: 10uF(2012), Capacitor_SMD:C_0805_2012Metric, F.Cu at (59.0, 41.5)
- added C16: 100nF, Capacitor_SMD:C_0402_1005Metric, F.Cu at (57.5, 63.0)
- added C17: 100nF, Capacitor_SMD:C_0402_1005Metric, F.Cu at (60.0, 47.5)
- added C18: 100nF, Capacitor_SMD:C_0402_1005Metric, F.Cu at (56.0, 56.5)
- added C19: 1uF(1608), Capacitor_SMD:C_0603_1608Metric, F.Cu at (54.5, 59.0)
- added C20: 100nF, Capacitor_SMD:C_0402_1005Metric, F.Cu at (57.0, 47.5)
- added C21: 100nF, Capacitor_SMD:C_0402_1005Metric, F.Cu at (55.5, 63.0)
- added C22: 100nF, Capacitor_SMD:C_0402_1005Metric, F.Cu at (58.0, 56.5)
- added C23: 1uF(1608), Capacitor_SMD:C_0603_1608Metric, F.Cu at (58.0, 59.0)
- added C4: 4.7uF(2012), Capacitor_SMD:C_0805_2012Metric, F.Cu at (50.0, 22.0)
- added C6: 4.7uF(2012), Capacitor_SMD:C_0805_2012Metric, F.Cu at (53.5, 27.5)
- added C7: 2.2uF(2012), Capacitor_SMD:C_0805_2012Metric, F.Cu at (43.0, 34.5)
- added C9: 2.2uF(2012), Capacitor_SMD:C_0805_2012Metric, F.Cu at (48.0, 38.0)
- added D3: LXES1UTAA1-157, Local_devices:LXES1UTAA1157, F.Cu at (62.5, 35.0)
- added D4: SMAJ7.0A, Diode_SMD:D_SMA, F.Cu at (51.5, 53.5)
- added D5: SMAJ7.0A, Diode_SMD:D_SMA, F.Cu at (64.5, 53.5)
- added F2: 0ZCJ0075FF2E, Local_devices:FUSC3216X120N, F.Cu at (59.0, 26.5)
- added J2: Battery, Connector_PinHeader_2.54mm:PinHeader_1x02_P2.54mm_Vertical, F.Cu at (65.0, 26.5)
- added L2: 470nH, Inductor_SMD:L_0805_2012Metric, F.Cu at (58.0, 38.5)
- added LED2: ORANGE, LED_SMD:LED_0805_2012Metric, F.Cu at (54.5, 19.5)
- added R11: 2M, Resistor_SMD:R_0402_1005Metric, F.Cu at (48.0, 27.5)
- added R12: 10k, Resistor_SMD:R_0402_1005Metric, F.Cu at (57.5, 21.5)
- added R13: 1M, Resistor_SMD:R_0402_1005Metric, F.Cu at (53.0, 31.5)
- added R14: 300k, Resistor_SMD:R_0402_1005Metric, F.Cu at (53.5, 33.5)
- added R15: 180k, Resistor_SMD:R_0402_1005Metric, F.Cu at (52.0, 33.5)
- added R16: 0, Resistor_SMD:R_0402_1005Metric, F.Cu at (42.0, 28.0)
- added R17: 1k, Resistor_SMD:R_0402_1005Metric, F.Cu at (47.0, 34.5)
- added R18: 200k, Resistor_SMD:R_0402_1005Metric, F.Cu at (55.0, 39.5)
- added R19: 100k, Resistor_SMD:R_0402_1005Metric, F.Cu at (55.0, 40.5)
- added R20: 100, Resistor_SMD:R_0402_1005Metric, F.Cu at (56.5, 53.0)
- added R21: 1.91k, Resistor_SMD:R_0402_1005Metric, F.Cu at (56.5, 55.0)
- added R22: 100, Resistor_SMD:R_0402_1005Metric, F.Cu at (57.5, 53.0)
- added R23: 1.91k, Resistor_SMD:R_0402_1005Metric, F.Cu at (57.5, 55.0)
- added R5: 470, Resistor_SMD:R_0402_1005Metric, F.Cu at (57.5, 19.5)
- added R8: 1M, Resistor_SMD:R_0402_1005Metric, F.Cu at (47.0, 27.5)
- added SW1: PCM12SMTR, Local_devices:PCM12SMTR, F.Cu at (68.3, 34.0)
- added U1: MCP73832T-2ACI_MC, Local_devices:SON50P300X200X100-9N-D, F.Cu at (55.0, 23.5)
- added U10: TPS22916CNYFPT, Local_devices:BGA4C40P2X2_78X78X50, F.Cu at (55.5, 61.0)
- added U11: SN74AUP2G08RSER, Local_devices:RSE0008A, F.Cu at (57.0, 50.0)
- added U12: TPS22916CNYFPT, Local_devices:BGA4C40P2X2_78X78X50, F.Cu at (57.5, 61.0)
- added U2: CSD25304W1015, Local_devices:BGA6C50P2X3_95X145X62, F.Cu at (50.0, 27.0)
- added U3: DMN65D8L-7, Package_TO_SOT_SMD:SOT-23, F.Cu at (47.0, 31.0)
- added U4: CSD25304W1015, Local_devices:BGA6C50P2X3_95X145X62, F.Cu at (56.0, 32.5)
- added U5: TPS3839A09DBZR, Package_TO_SOT_SMD:SOT-23, F.Cu at (43.0, 31.0)
- added U7: LP5907QMFX-2.8Q1, Local_devices:SOT95P280X145-5N, F.Cu at (44.5, 38.5)
- added U8: TPS6282618DMQR, Local_devices:TPS6282618DMQR, F.Cu at (55.0, 37.5)
- added U9: SN74AUP2G08RSER, Local_devices:RSE0008A, F.Cu at (60.0, 50.0)
- moved U15 25.2 mm to (43.0, 59.0)
- moved U13 17.1 mm to (28.0, 55.0), turned to 90 degrees
Connections:
- U13 pad 1: unconnected-(U13-Pad1) -> Earth
- U13 pad 15: unconnected-(U13-Pad15) -> Earth
- U13 pad 2: unconnected-(U13-Pad2) -> Earth
- U13 pad 28: unconnected-(U13-Pad28) -> +1V8
- U13 pad 30: unconnected-(U13-Pad30) -> +1V8
- U13 pad 32: unconnected-(U13-Pad32) -> VUSB
- U13 pad 33: unconnected-(U13-Pad33) -> Earth
- U13 pad 55: unconnected-(U13-Pad55) -> Earth
Routing:
- net +1V8: track 0.00 -> 62.2 mm, vias 0 -> 3
- net VUSB: track 2.61 -> 50.7 mm, vias 0 -> 2
- net /Power/VDRAIN: track 0.00 -> 47.0 mm
- net +2V8: track 0.00 -> 34.0 mm, vias 0 -> 2
- net Earth: track 17.6 -> 50.0 mm, vias 44 -> 242
- net +BATT: track 0.00 -> 31.0 mm
- net Net-(D3-Pad1): track 0.00 -> 27.8 mm, vias 0 -> 2
- net Net-(C22-Pad1): track 0.00 -> 12.6 mm
- net Net-(C18-Pad1): track 0.00 -> 10.6 mm
- net /Power/UVL_RST: track 0.00 -> 10.1 mm
- net Net-(R8-Pad1): track 0.00 -> 9.94 mm
- net Net-(C7-Pad2): track 0.00 -> 9.64 mm
- net VDD: track 0.00 -> 9.30 mm, vias 0 -> 1
- net Net-(D5-Pad1): track 0.00 -> 8.81 mm
- net Net-(L2-Pad1): track 0.00 -> 7.55 mm
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- added copper zone on In2.Cu, net Earth
- added copper zone on In2.Cu, net VDD
Other:
- board text added: "+"
- board text added: "-"

Commit message: 2022-08-09
Parts:
- added C11: 1uF(1608), Capacitor_SMD:C_0603_1608Metric, F.Cu at (57.5, 45.5)
- added C24: 100pF, Capacitor_SMD:C_0402_1005Metric, F.Cu at (30.5, 37.0)
- added C25: 12pF, Capacitor_SMD:C_0402_1005Metric, F.Cu at (42.5, 58.8)
- added C26: 12pF, Capacitor_SMD:C_0402_1005Metric, F.Cu at (42.5, 56.8)
- added C8: 100nF, Capacitor_SMD:C_0402_1005Metric, F.Cu at (53.0, 45.5)
- added J3: FTR-105-02-L-D, Connector_PinHeader_1.27mm:PinHeader_2x05_P1.27mm_Vertical_SMD, F.Cu at (29.0, 41.5)
- added LED3: IN-P32TATRGB, Local_devices:INP32TATRGB, F.Cu at (30.5, 64.0)
- added R24: 4.7k, Resistor_SMD:R_0402_1005Metric, F.Cu at (17.5, 54.0)
- added R25: 0, Resistor_SMD:R_0402_1005Metric, F.Cu at (38.0, 58.2)
- added R26: 0, Resistor_SMD:R_0402_1005Metric, F.Cu at (38.0, 57.2)
- added R29: 4.7k, Resistor_SMD:R_0402_1005Metric, F.Cu at (17.5, 61.5)
- added R30: 4.7k, Resistor_SMD:R_0402_1005Metric, F.Cu at (17.5, 57.0)
- added R32: 100, Resistor_SMD:R_0402_1005Metric, F.Cu at (36.0, 62.5)
- added R33: NC, Resistor_SMD:R_0402_1005Metric, F.Cu at (54.0, 61.5)
- added R34: 33, Resistor_SMD:R_0402_1005Metric, F.Cu at (35.0, 62.5)
- added R35: NC, Resistor_SMD:R_0402_1005Metric, F.Cu at (43.0, 61.5)
- added R36: 33, Resistor_SMD:R_0402_1005Metric, F.Cu at (26.0, 62.5)
- added R37: 360, Resistor_SMD:R_0402_1005Metric, F.Cu at (40.0, 61.5)
- added R38: 360, Resistor_SMD:R_0402_1005Metric, F.Cu at (51.0, 61.5)
- added SW2: EVQ-P7J01P, Local_devices:EVQP7J01P, F.Cu at (41.5, 65.5)
- added SW3: EVQ-P7J01P, Local_devices:EVQP7J01P, F.Cu at (52.5, 65.5)
- added U6: TPS22916CNYFPT, Local_devices:BGA4C40P2X2_78X78X50, F.Cu at (55.0, 45.5)
- added Y1: 32.768kHz, Crystal:Crystal_SMD_3215-2Pin_3.2x1.5mm, F.Cu at (40.5, 57.8)
- moved U15 38.7 mm to (80.5, 49.5)
- moved R2 12.6 mm to (32.8, 35.2), turned to -90 degrees
- moved R1 12.4 mm to (31.8, 35.2), turned to -90 degrees
- moved U11 11.4 mm to (67.0, 44.5), turned to 90 degrees
- moved U9 11.0 mm to (67.0, 41.5), turned to 90 degrees
- moved C3 10.6 mm to (22.5, 34.0), turned to -90 degrees
- moved R3 10.3 mm to (25.5, 33.0), turned to -90 degrees
- moved C20 9.30 mm to (64.5, 42.0), turned to -90 degrees
- moved C17 5.70 mm to (64.5, 44.0), turned to 90 degrees
- moved D2 5.05 mm to (32.5, 27.5), turned to 90 degrees
- moved R20 4.92 mm to (61.0, 51.0)
- moved R22 4.92 mm to (62.0, 51.0)
- moved C16 4.92 mm to (62.0, 61.0)
- moved C18 4.92 mm to (60.5, 54.5)
- moved C19 4.92 mm to (59.0, 57.0)
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Connections:
- R1 pad 2: /USB Connector/USB_DP -> /MDBT50Q/USBdata_P
- R2 pad 2: /USB Connector/USB_DN -> /MDBT50Q/USBdata_N
- U11 pad 6: /Power/PS_EN1 -> /MDBT50Q/PS_EN1
- U13 pad 10: unconnected-(U13-Pad10) -> /MDBT50Q/SDA0
- U13 pad 11: unconnected-(U13-Pad11) -> /MDBT50Q/VBAT_MOT_EN
- U13 pad 12: unconnected-(U13-Pad12) -> /MDBT50Q/VBAT_MON
- U13 pad 13: unconnected-(U13-Pad13) -> /MDBT50Q/PS_EN2
- U13 pad 14: unconnected-(U13-Pad14) -> /MDBT50Q/SPI0_MISO
- U13 pad 16: unconnected-(U13-Pad16) -> /MDBT50Q/VDD_SEL
- U13 pad 17: unconnected-(U13-Pad17) -> Net-(R25-Pad2)
- U13 pad 18: unconnected-(U13-Pad18) -> Net-(R26-Pad2)
- U13 pad 19: unconnected-(U13-Pad19) -> /MDBT50Q/SCL0
- U13 pad 20: unconnected-(U13-Pad20) -> /MDBT50Q/AIN2_XDK
- U13 pad 21: unconnected-(U13-Pad21) -> /MDBT50Q/PROM_RW
- U13 pad 22: unconnected-(U13-Pad22) -> /MDBT50Q/SDI/SDA
- U13 pad 23: unconnected-(U13-Pad23) -> /MDBT50Q/MCU_LED_R
- U13 pad 25: unconnected-(U13-Pad25) -> /MDBT50Q/GPIO3/INT2
- U13 pad 26: unconnected-(U13-Pad26) -> /MDBT50Q/SWITCH1
- U13 pad 27: unconnected-(U13-Pad27) -> /MDBT50Q/MCU_LED_G
- U13 pad 29: unconnected-(U13-Pad29) -> /MDBT50Q/MCU_LED_B
- U13 pad 3: unconnected-(U13-Pad3) -> /MDBT50Q/PlugDet
- U13 pad 34: unconnected-(U13-Pad34) -> /MDBT50Q/USBdata_N
- U13 pad 35: unconnected-(U13-Pad35) -> /MDBT50Q/USBdata_P
- U13 pad 36: unconnected-(U13-Pad36) -> /MDBT50Q/GPIO0
- U13 pad 37: unconnected-(U13-Pad37) -> /MDBT50Q/GPIO1
- U13 pad 38: unconnected-(U13-Pad38) -> /MDBT50Q/SCK/SCL
- U13 pad 39: unconnected-(U13-Pad39) -> /MDBT50Q/SDO
- U13 pad 4: unconnected-(U13-Pad4) -> /MDBT50Q/IOXP_INT
- U13 pad 40: unconnected-(U13-Pad40) -> /MDBT50Q/MCU_RESET
- U13 pad 47: unconnected-(U13-Pad47) -> /MDBT50Q/SWDO
- U13 pad 48: unconnected-(U13-Pad48) -> /MDBT50Q/CS
- U13 pad 49: unconnected-(U13-Pad49) -> /MDBT50Q/SWITCH2
- U13 pad 5: unconnected-(U13-Pad5) -> /MDBT50Q/SPI0_SCK
- U13 pad 50: unconnected-(U13-Pad50) -> /MDBT50Q/GPIO5
- U13 pad 51: unconnected-(U13-Pad51) -> /MDBT50Q/SWDIO
- U13 pad 52: unconnected-(U13-Pad52) -> /MDBT50Q/GPIO_EXT2_XDK
- U13 pad 53: unconnected-(U13-Pad53) -> /MDBT50Q/SWDCLK
- U13 pad 54: unconnected-(U13-Pad54) -> /MDBT50Q/GPIO_EXT1_XDK
- U13 pad 6: unconnected-(U13-Pad6) -> /MDBT50Q/SPI0_CS
- U13 pad 60: unconnected-(U13-Pad60) -> /MDBT50Q/GPIO4
- U13 pad 61: unconnected-(U13-Pad61) -> /MDBT50Q/GPIO2/INT1
- U13 pad 7: unconnected-(U13-Pad7) -> /MDBT50Q/AIN3_XDK
- U13 pad 8: unconnected-(U13-Pad8) -> /MDBT50Q/SPI0_MOSI
- U13 pad 9: unconnected-(U13-Pad9) -> /MDBT50Q/PS_EN1
- U9 pad 6: /Power/VDD_SEL -> /MDBT50Q/VDD_SEL
- U9 pad 7: /Power/VDD_SEL -> /MDBT50Q/VDD_SEL
Routing:
- net +2V8: track 34.0 -> 81.1 mm, vias 2 -> 3
- net /MDBT50Q/USBdata_N: track 0.00 -> 15.4 mm
- net /MDBT50Q/USBdata_P: track 0.00 -> 15.4 mm
- net /MDBT50Q/MCU_RESET: track 0.00 -> 14.6 mm, vias 0 -> 2
- net GNDPWR: track 12.4 -> 0.00 mm
- net /MDBT50Q/SWDIO: track 0.00 -> 11.1 mm
- net Net-(R22-Pad2): track 2.06 -> 12.9 mm
- net /MDBT50Q/SWDCLK: track 0.00 -> 10.7 mm
- net /MDBT50Q/SWDO: track 0.00 -> 9.65 mm, vias 0 -> 2
- net +1V8: track 62.2 -> 68.2 mm
- net Net-(R35-Pad1): track 0.00 -> 5.58 mm
- net Net-(R33-Pad1): track 0.00 -> 5.58 mm
- net Net-(LED3-Pad1): track 0.00 -> 5.10 mm
- net Net-(F1-Pad1): track 10.6 -> 5.57 mm, vias 2 -> 1
- net /USB Connector/DP: track 10.3 -> 5.77 mm
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Other:
- board size 50 x 50 mm -> 50 x 52 mm

Commit message: 2022-08-10
Parts:
- added C27: 100nF, Capacitor_SMD:C_0402_1005Metric, F.Cu at (49.5, 52.5)
- added C28: 200nF, Capacitor_SMD:C_0402_1005Metric, F.Cu at (49.5, 49.5)
- added C29: 100nF, Capacitor_SMD:C_0402_1005Metric, F.Cu at (49.5, 46.5)
- added C30: 1uF(1608), Capacitor_SMD:C_0603_1608Metric, F.Cu at (48.5, 46.5)
- added C31: 100nF, Capacitor_SMD:C_0402_1005Metric, F.Cu at (36.0, 42.5)
- added C32: 100nF, Capacitor_SMD:C_0402_1005Metric, F.Cu at (38.5, 45.5)
- added C33: 100nF, Capacitor_SMD:C_0402_1005Metric, F.Cu at (51.0, 54.5)
- added LED4: ORANGE, LED_SMD:LED_0805_2012Metric, F.Cu at (36.0, 46.5)
- added R39: 0, Resistor_SMD:R_0402_1005Metric, F.Cu at (46.5, 47.0)
- added R40: 0, Resistor_SMD:R_0402_1005Metric, F.Cu at (38.5, 40.5)
- added R41: 4.7k, Resistor_SMD:R_0402_1005Metric, F.Cu at (40.0, 45.5)
- added R42: 4.7k, Resistor_SMD:R_0402_1005Metric, F.Cu at (43.0, 45.5)
- added R43: 0, Resistor_SMD:R_0402_1005Metric, F.Cu at (38.5, 38.5)
- added R44: 0, Resistor_SMD:R_0402_1005Metric, F.Cu at (41.0, 45.5)
- added R45: 0, Resistor_SMD:R_0402_1005Metric, F.Cu at (42.0, 45.5)
- added R46: 0, Resistor_SMD:R_0402_1005Metric, F.Cu at (38.0, 36.0)
- added R47: 0, Resistor_SMD:R_0402_1005Metric, F.Cu at (38.0, 34.5)
- added R48: 4.7k, Resistor_SMD:R_0402_1005Metric, F.Cu at (18.4, 76.6)
- added R49: 4.7k, Resistor_SMD:R_0402_1005Metric, F.Cu at (20.2, 78.6)
- added R50: 4.7k, Resistor_SMD:R_0402_1005Metric, F.Cu at (41.0, 49.7)
- added R51: 4.7k, Resistor_SMD:R_0402_1005Metric, F.Cu at (41.0, 52.7)
- added R52: 0, Resistor_SMD:R_0402_1005Metric, F.Cu at (41.0, 51.7)
- added R53: 0, Resistor_SMD:R_0402_1005Metric, F.Cu at (41.0, 50.7)
- added R54: 0, Resistor_SMD:R_0402_1005Metric, F.Cu at (49.5, 51.0)
- added R55: 470, Resistor_SMD:R_0402_1005Metric, F.Cu at (36.0, 48.0)
- added TP1: TestPoint, TestPoint:TestPoint_Pad_D2.5mm, B.Cu at (95.2, 62.1)
- added TP10: TestPoint, TestPoint:TestPoint_Pad_D2.5mm, B.Cu at (90.7, 59.1)
- added TP11: TestPoint, TestPoint:TestPoint_Pad_D2.5mm, B.Cu at (87.7, 54.5)
- added TP12: TestPoint, TestPoint:TestPoint_Pad_D2.5mm, B.Cu at (83.2, 50.0)
- added TP13: TestPoint, TestPoint:TestPoint_Pad_D4.0mm, B.Cu at (97.5, 50.8)
- added TP14: TestPoint, TestPoint:TestPoint_Pad_D2.5mm, B.Cu at (87.7, 50.0)
- added TP15: TestPoint, TestPoint:TestPoint_Pad_D2.5mm, B.Cu at (92.2, 54.5)
- added TP2: TestPoint, TestPoint:TestPoint_Pad_D2.5mm, B.Cu at (104.3, 62.1)
- added TP3: TestPoint, TestPoint:TestPoint_Pad_D2.5mm, B.Cu at (99.8, 62.1)
- added TP4: TestPoint, TestPoint:TestPoint_Pad_D2.5mm, B.Cu at (83.2, 54.5)
- added TP5: TestPoint, TestPoint:TestPoint_Pad_D2.5mm, B.Cu at (92.2, 50.0)
- added TP6: TestPoint, TestPoint:TestPoint_Pad_D4.0mm, B.Cu at (103.6, 50.8)
- added TP7: TestPoint, TestPoint:TestPoint_Pad_D4.0mm, B.Cu at (97.5, 56.8)
- added TP8: TestPoint, TestPoint:TestPoint_Pad_D4.0mm, B.Cu at (103.6, 56.8)
- added TP9: TestPoint, TestPoint:TestPoint_Pad_D2.5mm, B.Cu at (78.6, 50.0)
- added U14: BMM150, Package_CSP:WLCSP-12_1.56x1.56mm_P0.4mm, F.Cu at (38.5, 43.0)
- added U16: DS28E05R+T, Local_devices:SOT95P237X112-3N, F.Cu at (48.0, 64.5)
- added U17: W25Q32JWZPIQ, Local_devices:SON127P600X500X80-9N-D, F.Cu at (49.0, 58.0)
- moved U15 35.0 mm to (45.5, 50.5), turned to 180 degrees
- moved R33 2.06 mm to (56.0, 62.0)
- moved R38 2.06 mm to (53.0, 62.0)
- moved SW3 2.00 mm to (54.5, 65.5)
- moved R35 0.50 mm to (43.0, 62.0)
- moved R37 0.50 mm to (40.0, 62.0)
Connections:
- net /MDBT50Q/PROM_RW renamed /BHI260AP/PROM_RW
- R13 pad 1: /USB Connector/VBAT_MON_EN -> /MDBT50Q/VBAT_MOT_EN
- R14 pad 2: /USB Connector/VBAT_MON -> /MDBT50Q/VBAT_MON
- R15 pad 1: /USB Connector/VBAT_MON -> /MDBT50Q/VBAT_MON
- U13 pad 22: /MDBT50Q/SDI/SDA -> /BHI260AP/SDI/SDA
- U13 pad 25: /MDBT50Q/GPIO3/INT2 -> /BHI260AP/GPIO3/INT2
- U13 pad 36: /MDBT50Q/GPIO0 -> /BHI260AP/GPIO0
- U13 pad 37: /MDBT50Q/GPIO1 -> /BHI260AP/GPIO1
- U13 pad 38: /MDBT50Q/SCK/SCL -> /BHI260AP/SCK/SCL
- U13 pad 39: /MDBT50Q/SDO -> /BHI260AP/SDO
- U13 pad 48: /MDBT50Q/CS -> /BHI260AP/CS
- U13 pad 50: /MDBT50Q/GPIO5 -> /BHI260AP/GPIO5
- U13 pad 61: /MDBT50Q/GPIO2/INT1 -> /BHI260AP/GPIO2/INT
- U15 pad 1: unconnected-(U15-Pad1) -> Net-(R50-Pad2)
- U15 pad 10: unconnected-(U15-Pad10) -> /BHI260AP/GPIO2/INT
- U15 pad 11: unconnected-(U15-Pad11) -> /BHI260AP/SDI/SDA
- U15 pad 12: unconnected-(U15-Pad12) -> VDDIO
- U15 pad 13: unconnected-(U15-Pad13) -> /BHI260AP/B260_TP12
- U15 pad 14: unconnected-(U15-Pad14) -> /BHI260AP/QSPI_CSN
- U15 pad 15: unconnected-(U15-Pad15) -> /BHI260AP/QSPI_D1
- U15 pad 16: unconnected-(U15-Pad16) -> /BHI260AP/BMP390_INT
- U15 pad 17: unconnected-(U15-Pad17) -> Earth
- U15 pad 18: unconnected-(U15-Pad18) -> /BHI260AP/BMM150_INT
- U15 pad 19: unconnected-(U15-Pad19) -> /BHI260AP/GPIO3/INT2
- U15 pad 2: unconnected-(U15-Pad2) -> Net-(R51-Pad2)
- U15 pad 20: unconnected-(U15-Pad20) -> /BHI260AP/QSPI_D2
- U15 pad 21: unconnected-(U15-Pad21) -> /BHI260AP/B260_TP5
- U15 pad 22: unconnected-(U15-Pad22) -> Net-(R42-Pad2)
- U15 pad 23: unconnected-(U15-Pad23) -> /BHI260AP/B260_TP7
- U15 pad 24: unconnected-(U15-Pad24) -> /BHI260AP/B260_TP6
- U15 pad 25: unconnected-(U15-Pad25) -> Earth
- U15 pad 26: unconnected-(U15-Pad26) -> Earth
- U15 pad 27: unconnected-(U15-Pad27) -> Earth
- U15 pad 28: unconnected-(U15-Pad28) -> VDD
- U15 pad 29: unconnected-(U15-Pad29) -> /BHI260AP/B260_TP9
- U15 pad 3: unconnected-(U15-Pad3) -> /BHI260AP/HOST_BOOT
- U15 pad 30: unconnected-(U15-Pad30) -> Net-(R41-Pad2)
- U15 pad 31: unconnected-(U15-Pad31) -> /BHI260AP/B260_TP1
- U15 pad 32: unconnected-(U15-Pad32) -> /BHI260AP/SDO
- U15 pad 33: unconnected-(U15-Pad33) -> /BHI260AP/SCK/SCL
- U15 pad 34: unconnected-(U15-Pad34) -> /BHI260AP/CS
- U15 pad 35: unconnected-(U15-Pad35) -> /BHI260AP/B260_TP14
- U15 pad 36: unconnected-(U15-Pad36) -> Earth
- U15 pad 37: unconnected-(U15-Pad37) -> /BHI260AP/B260_TP15
- U15 pad 38: unconnected-(U15-Pad38) -> Net-(R55-Pad2)
- U15 pad 39: unconnected-(U15-Pad39) -> /BHI260AP/B260_TP4
- U15 pad 4: unconnected-(U15-Pad4) -> /BHI260AP/QSPI_D0
- U15 pad 40: unconnected-(U15-Pad40) -> /BHI260AP/B260_TP2
- U15 pad 41: unconnected-(U15-Pad41) -> /BHI260AP/B260_TP3
- U15 pad 42: unconnected-(U15-Pad42) -> VDDIO
- U15 pad 43: unconnected-(U15-Pad43) -> /BHI260AP/B260_TP11
- U15 pad 44: unconnected-(U15-Pad44) -> /BHI260AP/B260_TP10
- U15 pad 5: unconnected-(U15-Pad5) -> /BHI260AP/QSPI_CLK
- U15 pad 6: unconnected-(U15-Pad6) -> Net-(C28-Pad2)
- U15 pad 7: unconnected-(U15-Pad7) -> VDDIO
- U15 pad 8: unconnected-(U15-Pad8) -> /BHI260AP/QSPI_D3
- U15 pad 9: unconnected-(U15-Pad9) -> /BHI260AP/RESET
- U4 pad A1: /USB Connector/VBAT_MON_EN -> /MDBT50Q/VBAT_MOT_EN
Routing:
- net VDDIO: track 1.92 -> 35.5 mm, vias 0 -> 4
- net VUSB: track 52.8 -> 19.8 mm
- net +1V8: track 68.2 -> 42.2 mm
- net /BHI260AP/CS: track 0.00 -> 24.0 mm, vias 0 -> 2
- net /BHI260AP/SDO: track 0.00 -> 19.3 mm, vias 0 -> 4
- net /BHI260AP/QSPI_D0: track 0.00 -> 14.6 mm, vias 0 -> 2
- net /BHI260AP/QSPI_D3: track 0.00 -> 14.6 mm, vias 0 -> 2
- net /BHI260AP/QSPI_CLK: track 0.00 -> 13.9 mm, vias 0 -> 2
- net /BHI260AP/GPIO0: track 0.00 -> 12.3 mm, vias 0 -> 2
- net Net-(R50-Pad2): track 0.00 -> 12.1 mm
- net Net-(R41-Pad2): track 0.00 -> 11.4 mm, vias 0 -> 2
- net /BHI260AP/GPIO1: track 0.00 -> 11.4 mm, vias 0 -> 2
- net Net-(R55-Pad2): track 0.00 -> 10.8 mm, vias 0 -> 2
- net Net-(R51-Pad2): track 0.00 -> 10.7 mm, vias 0 -> 2
- net Net-(R42-Pad2): track 0.00 -> 9.74 mm
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
Commit message: 2022-08-11
Parts:
- moved TP8 68.0 mm to (36.0, 64.0)
- moved TP2 66.6 mm to (38.0, 56.0)
- moved TP3 59.9 mm to (40.5, 53.5)
- moved TP6 58.1 mm to (47.0, 64.0)
- moved TP5 57.8 mm to (35.0, 58.0)
- moved TP7 56.5 mm to (41.5, 64.0)
- moved TP15 54.4 mm to (38.0, 51.0)
- moved TP4 47.7 mm to (35.5, 53.5)
- moved TP11 47.4 mm to (40.5, 58.5)
- moved TP13 47.0 mm to (52.5, 64.0)
- moved TP1 46.0 mm to (51.5, 48.0)
- moved TP10 44.2 mm to (46.5, 58.5)
- moved R48 39.9 mm to (54.5, 59.5), turned to 180 degrees
- moved R49 39.7 mm to (54.5, 58.5), turned to 180 degrees
- moved TP14 39.0 mm to (49.0, 45.5)
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Routing:
- net +1V8: track 42.2 -> 110.5 mm, vias 3 -> 9
- net /MDBT50Q/PS_EN1: track 0.87 -> 58.6 mm, vias 1 -> 2
- net /MDBT50Q/VDD_SEL: track 1.21 -> 53.2 mm, vias 1 -> 2
- net /MDBT50Q/VBAT_MOT_EN: track 5.73 -> 51.2 mm, vias 0 -> 4
- net /MDBT50Q/VBAT_MON: track 1.50 -> 46.5 mm, vias 0 -> 4
- net VDDIO: track 35.5 -> 80.4 mm, vias 4 -> 9
- net /MDBT50Q/PS_EN2: track 1.13 -> 42.3 mm, vias 1 -> 6
- net /MDBT50Q/SWITCH2: track 3.60 -> 42.4 mm
- net VUSB: track 19.8 -> 51.3 mm
- net /BHI260AP/SDI/SDA: track 0.00 -> 29.9 mm, vias 0 -> 5
- net /BHI260AP/GPIO2/INT: track 0.95 -> 27.9 mm, vias 1 -> 2
- net /BHI260AP/GPIO5: track 0.00 -> 26.6 mm, vias 0 -> 2
- net /MDBT50Q/SDA0: track 0.00 -> 22.9 mm, vias 0 -> 2
- net /BHI260AP/PROM_RW: track 0.00 -> 21.2 mm, vias 0 -> 6
- net /BHI260AP/SCK/SCL: track 0.32 -> 21.0 mm, vias 1 -> 2
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- added copper zone on In2.Cu, net +1V8

Commit message: 2022-08-11 2
Routing:
- net /MDBT50Q/MCU_LED_B: track 16.6 -> 15.3 mm

Commit message: 2022-08-16
Parts:
- added R27: 10k, Resistor_SMD:R_0402_1005Metric, F.Cu at (25.0, 45.0)
- moved C13 5.15 mm to (55.0, 40.5)
- moved R19 1.02 mm to (55.0, 41.5)
- moved C31 1.00 mm to (38.0, 39.5)
- moved R46 1.00 mm to (39.0, 39.5)
- moved U14 1.00 mm to (38.5, 42.0), turned to 180 degrees
- turned U6 to 0 degrees
Connections:
- C13 pad 1: Earth -> Net-(R18-Pad2)
- U6 pad A1: +1V8 -> VDDIO
- U6 pad A2: VDDIO -> +1V8
- U8 pad 1: /Power/VDRAIN -> /Power/UVL_RST
Routing:
- net /Power/UVL_RST: track 10.1 -> 22.3 mm, vias 0 -> 2
- net Net-(R40-Pad1): track 2.03 -> 10.5 mm, vias 0 -> 2
- net Net-(R46-Pad1): track 1.45 -> 7.66 mm, vias 0 -> 2
- net /Power/VDRAIN: track 49.5 -> 43.7 mm
- net Net-(R47-Pad1): track 2.40 -> 7.71 mm, vias 0 -> 2
- net Earth: track 70.0 -> 73.9 mm, vias 283 -> 280
- net +1V8: track 110.5 -> 114.2 mm, vias 9 -> 10
- net /MDBT50Q/MCU_RESET: track 11.9 -> 14.1 mm
- net /MDBT50Q/PS_EN2: track 42.3 -> 40.5 mm
- net VDDIO: track 80.4 -> 81.8 mm
- net Net-(R18-Pad2): track 2.56 -> 3.63 mm
- net Net-(R43-Pad1): track 4.11 -> 3.15 mm
- net Net-(R44-Pad1): track 4.10 -> 5.03 mm, vias 0 -> 2
- net Net-(R45-Pad1): track 6.12 -> 5.44 mm

Commit message: 2022-08-24
Parts:
- moved C12 5.52 mm to (57.0, 37.5)
- moved L2 1.03 mm to (59.0, 38.5)
- moved C15 1.00 mm to (61.0, 38.5)
Routing:
- net Earth: track 73.9 -> 79.7 mm, vias 280 -> 281
- net Net-(L2-Pad1): track 7.55 -> 3.10 mm
- net /Power/VDRAIN: track 43.7 -> 41.6 mm
- net +1V8: track 114.2 -> 115.7 mm
- net Net-(D3-Pad1): track 28.7 -> 29.5 mm
