File: culturit_tx.kicad_pcb (KiCad board)
At the start: 4 copper layers, 27 x 27 mm, 65 parts, among them CN1 2.54 X 2P, J1 SWD, J2 USB4105-GF-A, Q1 MMBT2222LT1G, Q2 FDN340P, Q3 MMBT2222LT1G, U1 MAX1555EZK+T, U2 BQ27441DRZR-G1A, U3 TPS62A01ADRLR, U4 TCR3UG33A,LF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

Commit message: 2022-09-14 2
Routing:
- net Earth: vias 44 -> 43

Commit message: 2022-10-05
Routing:
- net Earth: track 57.9 -> 62.7 mm
Changed lines of the file:
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@@
       (rotate (xyz 0 0 0))
     )
+    (model "${KIPRJMOD}/lib/Local_devices.3dshapes/IN-P32TATRGB.stp"
+      (offset (xyz 0 0 0))
+      (scale (xyz 1 1 1))
+      (rotate (xyz 0 0 0))
+    )
   )
   (footprint "Local_devices:SKSCLDE010" (layer "F.Cu")
@@
     (fp_line (start -1.75 -1.4) (end -1.75 1.4) (layer "F.SilkS") (width 0.1))
     (fp_line (start -1.75 1.4) (end -0.8 1.4) (layer "F.SilkS") (width 0.1))
-    (pad "" np_thru_hole circle locked (at 0 -0.9 135) (size 0.55 0.55) (drill 0.55) (layers *.Cu *.Mask))
-    (pad "" np_thru_hole circle locked (at 0 0.9 135) (size 0.55 0.55) (drill 0.55) (layers *.Cu *.Mask))
+    (pad "" np_thru_hole circle locked (at 0 -0.9 135) (size 0.55 0.55) (drill 0.7) (layers F&B.Cu *.Mask))
+    (pad "" np_thru_hole circle locked (at 0 0.9 135) (size 0.55 0.55) (drill 0.7) (layers F&B.Cu *.Mask))
     (pad "1" smd rect locked (at -1.8 0.65 135) (size 1.4 0.9) (layers "F.Cu" "F.Paste" "F.Mask")
       (net 41 "Earth") (pintype "bidirectional"))
@@
   (segment (start 50.75 37.62) (end 50.85 37.52) (width 0.127) (layer "F.Cu") (net 41))
   (segment (start 53.2 55) (end 53 54.8) (width 0.4) (layer "F.Cu") (net 41))
+  (segment (start 58 43) (end 58 44) (width 0.127) (layer "F.Cu") (net 41))
   (segment (start 48 59.725) (end 47 60.725) (width 0.4) (layer "F.Cu") (net 41))
   (segment (start 50.75 38.1125) (end 50.75 37.62) (width 0.127) (layer "F.Cu") (net 41))
@@
   (segment (start 52.78 38.25) (end 51.6625 38.25) (width 0.127) (layer "F.Cu") (net 41))
   (segment (start 41.75 54.65) (end 42.85 54.65) (width 0.4) (layer "F.Cu") (net 41))
+  (segment (start 56.95 44) (end 56.95 42.55) (width 0.127) (layer "F.Cu") (net 41))
   (segment (start 51.6625 38.25) (end 51.6625 37.4825) (width 0.127) (layer "F.Cu") (net 41))
   (segment (start 53 43) (end 52.6 43.4) (width 0.4) (layer "F.Cu") (net 41))
@@
   (segment (start 60.26 50.225) (end 61.75 48.735) (width 0.4) (layer "F.Cu") (net 41))
   (segment (start 48.95 56.72) (end 48.95 55.7) (width 0.4) (layer "F.Cu") (net 41))
+  (segment (start 57.855739 43) (end 58 43) (width 0.127) (layer "F.Cu") (net 41))
+  (segment (start 57 42.5) (end 57.355739 42.5) (width 0.127) (layer "F.Cu") (net 41))
   (segment (start 53 54.8) (end 52.65 54.8) (width 0.4) (layer "F.Cu") (net 41))
+  (segment (start 58 44) (end 56.95 44) (width 0.127) (layer "F.Cu") (net 41))
   (segment (start 48 59.25) (end 48 60.175) (width 0.4) (layer "F.Cu") (net 41))
   (segment (start 53 42.48) (end 53 43) (width 0.4) (layer "F.Cu") (net 41))
@@
   (segment (start 59.75 50.225) (end 60.26 50.225) (width 0.4) (layer "F.Cu") (net 41))
   (segment (start 47.6 40.75) (end 47.57 40.72) (width 0.25) (layer "F.Cu") (net 41))
+  (segment (start 57.355739 42.5) (end 57.855739 43) (width 0.127) (layer "F.Cu") (net 41))
   (segment (start 48.97 40.75) (end 48.3375 40.75) (width 0.25) (layer "F.Cu") (net 41))
   (segment (start 44.52 59.75) (end 43.84 59.75) (width 0.4) (layer "F.Cu") (net 41))
   (segment (start 48.3375 40.75) (end 47.6 40.75) (width 0.25) (layer "F.Cu") (net 41))
   (segment (start 57.32 56.65) (end 57.6 56.65) (width 0.4) (layer "F.Cu") (net 41))
+  (segment (start 56.95 42.55) (end 57 42.5) (width 0.127) (layer "F.Cu") (net 41))
   (segment (start 53 38.47) (end 52.78 38.25) (width 0.127) (layer "F.Cu") (net 41))
   (segment (start 57.169239 39.25) (end 57.686827 39.767588) (width 0.4) (layer "F.Cu") (net 41))

Commit message: 2022-10-30
Parts:
- removed D1: MMBD4148, Local_devices:SOT23
- removed R12: 10k, Resistor_SMD:R_0402_1005Metric
- removed R13: 20k, Resistor_SMD:R_0402_1005Metric
- removed R15, R16: 1k, Resistor_SMD:R_0402_1005Metric
- added C15: 12pF, Capacitor_SMD:C_0402_1005Metric, F.Cu at (98.0, 38.8)
- added C17: 12pF, Capacitor_SMD:C_0402_1005Metric, F.Cu at (91.8, 43.6)
- added Y1: 32.768kHz, Crystal:Crystal_SMD_2012-2Pin_2.0x1.2mm, F.Cu at (94.7, 39.2)
- LED2: value IN-P32TATRGB -> CLV1L-FKB-CJ1N1E1BB7B3B3; footprint Local_devices:INP32TATRGB -> LED_SMD:LED_Cree-PLCC4_3.2x2.8mm_CCW
- Q1, Q3: value MMBT2222LT1G -> FDV303N; footprint Local_devices:SOT23 -> Package_TO_SOT_SMD:SOT-23; moved to F.Cu
- Q2: value FDN340P -> FDN352AP; footprint Local_devices:SOT23 -> Package_TO_SOT_SMD:SOT-23
- R11: value 20k -> 33k
- R18: value 1k -> 10k
- R26, R27: value 33 -> 100
- U4: value TCR3UG33A,LF -> MIC5317-3.3YM5-TR; footprint Local_devices:BGA4N35P2X2_64X64X33 -> Local_devices:SOT95P280X145-5N; moved to F.Cu
- moved R26 47.4 mm to (94.4, 41.6), turned to 0 degrees
- moved LED2 46.2 mm to (90.2, 40.0), turned to 0 degrees
- moved R27 42.9 mm to (88.9, 43.3), turned to 0 degrees
- moved Q3 22.2 mm to (74.0, 40.0)
- moved Q2 15.1 mm to (73.7, 44.6)
- moved U4 12.5 mm to (69.0, 40.1), turned to 0 degrees
- moved Q1 11.5 mm to (68.8, 44.6), turned to 0 degrees
Connections:
- C6 pad 1: Net-(C6-Pad1) -> Earth
- LED2 pad 1: Net-(LED2-Pad1) -> +3V3
- LED2 pad 2: +3V3 -> Net-(LED2-Pad2)
- Q1 pad 1: Net-(Q1-Pad1) -> Earth
- Q1 pad 3: Net-(Q1-Pad3) -> Net-(Q3-Pad3)
- Q2 pad 1: Net-(Q2-Pad1) -> Net-(Q3-Pad3)
- Q2 pad 2: Net-(C11-Pad1) -> VSYS
- Q2 pad 3: VSYS -> Net-(C11-Pad1)
- Q3 pad 1: Net-(Q3-Pad1) -> /MDBT50Q/LDO_ON
- R10 pad 1: Net-(C6-Pad1) -> Earth
- R14 pad 2: Net-(Q2-Pad1) -> Net-(Q3-Pad3)
- R17 pad 2: Net-(Q3-Pad1) -> /MDBT50Q/LDO_ON
- R18 pad 2: Net-(Q3-Pad1) -> Earth
- R25 pad 1: Net-(LED2-Pad1) -> Net-(LED2-Pad2)
- S1 pad 3: Net-(C6-Pad1) -> Earth
- S1 pad 4: Net-(C6-Pad1) -> Earth
- U5 pad 17: unconnected-(U5-Pad17) -> Net-(C15-Pad2)
- U5 pad 18: unconnected-(U5-Pad18) -> Net-(C17-Pad1)
Routing:
- net /MDBT50Q/MCU_LED_G: track 13.0 -> 0.00 mm, vias 4 -> 0
- net /MDBT50Q/MCU_LED_B: track 12.3 -> 0.00 mm
- net Earth: track 62.7 -> 50.6 mm, vias 43 -> 6
- net Net-(C6-Pad1): track 11.0 -> 0.00 mm, vias 1 -> 0
- net Net-(Q1-Pad1): track 5.42 -> 0.00 mm, vias 1 -> 0
- net Net-(LED2-Pad3): track 5.26 -> 0.00 mm
- net Net-(Q2-Pad1): track 5.16 -> 0.00 mm
- net Net-(LED2-Pad4): track 3.87 -> 0.00 mm
- net Net-(Q1-Pad3): track 3.38 -> 0.00 mm, vias 1 -> 0
- net +3V3: track 32.7 -> 29.4 mm, vias 5 -> 4
- net Net-(Q3-Pad3): track 2.57 -> 0.00 mm, vias 1 -> 0
- net Net-(Q3-Pad1): track 2.23 -> 0.00 mm
- net Net-(D1-Pad3): track 1.37 -> 0.00 mm
- net Net-(LED2-Pad1): track 1.33 -> 0.00 mm
- net Net-(C11-Pad1): track 13.5 -> 12.6 mm, vias 1 -> 0
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
Commit message: 2022-11-01
Parts:
- C11, C12, C16, C5, C6, L1, R17, R18, R19, R2, R20, R21, R28, R29, R3, R30, R5, R6, R7, R8, R9, U2, U3, U6: moved to F.Cu
- J1: footprint Local_devices:SWD_port -> Connector_PinHeader_2.54mm:PinHeader_1x04_P2.54mm_Vertical
- J2: value USB4105-GF-A -> USB4110-GF-A; footprint Local_devices:GCT_USB4105-GF-A -> Local_devices:USB4110GFA; moved to F.Cu
- R25, R26, R27: value 100 -> 470
- S2: value SKSCLDE010 -> Reset; footprint Local_devices:SKSCLDE010 -> Button_Switch_SMD:SW_SPST_B3U-1000P; moved to B.Cu
- moved R26 75.9 mm to (21.0, 22.0)
- moved C15 75.1 mm to (25.2, 20.0), turned to -90 degrees
- moved LED2 74.0 mm to (19.0, 19.7)
- moved Y1 72.3 mm to (24.5, 22.0)
- moved C17 72.0 mm to (23.8, 20.0), turned to 90 degrees
- moved R27 65.7 mm to (27.5, 20.0), turned to -90 degrees
- moved Q3 45.9 mm to (32.7, 20.1), turned to 180 degrees
- moved Q2 42.8 mm to (37.2, 22.1), turned to 180 degrees
- moved S1 42.3 mm to (46.0, 18.1), turned to 180 degrees
- moved Q1 40.6 mm to (37.2, 19.0), turned to 180 degrees
- moved C5 39.4 mm to (48.5, 21.0), turned to 90 degrees
- moved C6 39.0 mm to (42.4, 21.3)
- moved R10 38.0 mm to (44.6, 21.3), turned to -90 degrees
- moved R11 37.6 mm to (43.5, 21.3), turned to 90 degrees
- moved R6 36.0 mm to (46.8, 21.3), turned to 0 degrees
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Connections:
- C2 pad 1: Net-(C2-Pad1) -> /USB Connector/VUSB
- C6 pad 1: Earth -> Net-(C6-Pad1)
- FB1 pad 2: Net-(C2-Pad1) -> /USB Connector/VUSB
- Q1 pad 1: Earth -> Net-(C6-Pad1)
- R10 pad 1: Earth -> Net-(C6-Pad1)
- S1 pad 3: Earth -> Net-(C6-Pad1)
- S1 pad 4: Earth -> Net-(C6-Pad1)
- S2 pad 1: Earth -> /MDBT50Q/MCU_RESET
Routing:
- net /BNO085/BNO_BOOTN: track 4.52 -> 41.9 mm, vias 1 -> 3
- net Earth: track 50.6 -> 85.2 mm, vias 6 -> 101
- net /BNO085/BNO_NRST: track 7.49 -> 34.6 mm
- net +3V3: track 29.4 -> 56.4 mm, vias 4 -> 5
- net VBUS: track 24.0 -> 48.6 mm
- net /MDBT50Q/MCU_RESET: track 17.5 -> 41.2 mm, vias 2 -> 4
- net /BNO085/HOST_MISO: track 9.26 -> 31.5 mm
- net /MDBT50Q/USBdata_N: track 9.12 -> 31.3 mm, vias 1 -> 2
- net /MDBT50Q/BATT_SDA: track 11.2 -> 33.1 mm, vias 1 -> 2
- net /BNO085/HOST_SCLK: track 9.36 -> 31.2 mm
- net /MDBT50Q/BATT_SCL: track 12.8 -> 34.4 mm, vias 1 -> 2
- net /MDBT50Q/USBdata_P: track 9.12 -> 30.3 mm, vias 1 -> 2
- net /BNO085/HOST_INTN: track 13.8 -> 34.6 mm, vias 2 -> 4
- net /BNO085/BNO_WAKE: track 16.7 -> 36.5 mm
- net /MDBT50Q/GPOUT: track 6.10 -> 24.6 mm, vias 1 -> 4
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- added copper zone on In2.Cu, net Earth
- added copper zone on F.Cu, net GNDPWR
Other:
- board size 27 x 27 mm -> 39.6 x 28.6 mm

Commit message: 2022-11-01 2
Parts:
- moved R25 9.00 mm to (28.0, 22.0)
- moved R26 9.00 mm to (30.0, 22.0)
Routing:
- net /MDBT50Q/MCU_LED_G: track 3.96 -> 18.5 mm, vias 0 -> 2
- net /MDBT50Q/MCU_LED_R: track 12.8 -> 25.0 mm, vias 2 -> 4
- net Net-(LED2-Pad3): track 1.70 -> 12.9 mm, vias 0 -> 2
- net Net-(LED2-Pad2): track 1.91 -> 12.5 mm, vias 0 -> 2

Commit message: 20221115
Parts:
- S2: moved to F.Cu
- moved S2 13.7 mm to (45.5, 41.2)
Routing:
- net /MDBT50Q/MCU_RESET: track 41.2 -> 37.4 mm, vias 4 -> 5
